File: KiCad/C3Jr/c3jr-mech.sch (KiCad schematic (older format))
At the start: 18 parts

Commit message: 2011-04-25 : C3Jr : PCB update
Parts:
- removed BF1: BAFFLE, BAFFLE, symbol BAFFLE
- removed DF1: DIFFUSER, DIFFUSER, symbol DIFFUSER
- removed FC1: FRONT COVER, FrontCover, symbol DIFFUSER
- removed FP1: FACE PLATE, FrontCover, symbol DIFFUSER
- removed MP1: SCREW, MtgPost, symbol SCREW
- removed MT1, MT11, MT12, MT14, MT2, MT4, MT5, MT7, MT8: SCREW, VITE_CSK_3MM, symbol SCREW
- removed MT10, MT13, MT3, MT6: SCREW, vite_csk_3mm, symbol SCREW
Other:
- note removed: "DIFFUSER SCREWS\nCSK, 3mm"
- note removed: "MOUNTING POSTS\n14 nos, around the board\n3mm internal thread, 5mm OD"
Changed lines of the file:
@@
-EESchema Schematic File Version 2  date 04/25/11 15:56:13
+EESchema Schematic File Version 2  date 04/25/11 18:36:08
 LIBS:clock3
 LIBS:power
@@
 Sheet 3 4
 Title "ClockTHREE Junior aka C3Jr"
-Date "24 apr 2011"
+Date "25 apr 2011"
 Rev "A"
 Comp "an improved WordClock based on ClockTHREE"
@@
 Comment4 ""
 $EndDescr
-$Comp
-L SCREW MT13
-U 1 1 4D286CFF
-P 3250 3800
-F 0 "MT13" H 3250 3700 40  0000 C CNN
-F 1 "SCREW" H 3250 3900 40  0001 C CNN
-F 2 "vite_csk_3mm" H 3250 3800 60  0001 C CNN
-	1    3250 3800
-	1    0    0    -1
-$EndComp
-$Comp
-L SCREW MT10
-U 1 1 4D286CFA
-P 3250 5500
-F 0 "MT10" H 3250 5400 40  0000 C CNN
-F 1 "SCREW" H 3250 5600 40  0001 C CNN
-F 2 "vite_csk_3mm" H 3250 5500 60  0001 C CNN
-	1    3250 5500
-	1    0    0    -1
-$EndComp
-$Comp
-L SCREW MT6
-U 1 1 4D286CF6
-P 5050 5500
-F 0 "MT6" H 5050 5400 40  0000 C CNN
-F 1 "SCREW" H 5050 5600 40  0001 C CNN
-F 2 "vite_csk_3mm" H 5050 5500 60  0001 C CNN
-	1    5050 5500
-	1    0    0    -1
-$EndComp
-$Comp
-L SCREW MT3
-U 1 1 4D286CF3
-P 5050 3800
-F 0 "MT3" H 5050 3700 40  0000 C CNN
-F 1 "SCREW" H 5050 3900 40  0001 C CNN
-F 2 "vite_csk_3mm" H 5050 3800 60  0001 C CNN
-	1    5050 3800
-	1    0    0    -1
-$EndComp
-$Comp
-L SCREW MP1
-U 1 1 4D283F93
-P 1825 5600
-F 0 "MP1" H 1825 5500 40  0000 C CNN
-F 1 "SCREW" H 1825 5700 40  0001 C CNN
-F 2 "MtgPost" H 1825 5600 60  0001 C CNN
-	1    1825 5600
-	1    0    0    -1
-$EndComp
-$Comp
-L SCREW MT4
-U 1 1 4D283CE6
-P 5200 4400
-F 0 "MT4" H 5200 4300 40  0000 C CNN
-F 1 "SCREW" H 5200 4500 40  0001 C CNN
-F 2 "VITE_CSK_3MM" H 5200 4400 60  0001 C CNN
-	1    5200 4400
-	1    0    0    -1
-$EndComp
-$Comp
-L SCREW MT5
-U 1 1 4D283CDD
-P 5200 4900
-F 0 "MT5" H 5200 4800 40  0000 C CNN
-F 1 "SCREW" H 5200 5000 40  0001 C CNN
-F 2 "VITE_CSK_3MM" H 5200 4900 60  0001 C CNN
-	1    5200 4900
-	1    0    0    -1
-$EndComp
-$Comp
-L SCREW MT7
-U 1 1 4D283CC9
-P 4550 5500
-F 0 "MT7" H 4550 5400 40  0000 C CNN
-F 1 "SCREW" H 4550 5600 40  0001 C CNN
-F 2 "VITE_CSK_3MM" H 4550 5500 60  0001 C CNN
-	1    4550 5500
-	1    0    0    -1
-$EndComp
-$Comp
-L SCREW MT8
-U 1 1 4D283CC6
-P 4150 5500
-F 0 "MT8" H 4150 5400 40  0000 C CNN
-F 1 "SCREW" H 4150 5600 40  0001 C CNN
-F 2 "VITE_CSK_3MM" H 4150 5500 60  0001 C CNN
-	1    4150 5500
-	1    0    0    -1
-$EndComp
-$Comp
-L SCREW MT11
-U 1 1 4D283CC3
-P 3100 4900
-F 0 "MT11" H 3100 4800 40  0000 C CNN
-F 1 "SCREW" H 3100 5000 40  0001 C CNN
-F 2 "VITE_CSK_3MM" H 3100 4900 60  0001 C CNN
-	1    3100 4900
-	1    0    0    -1
-$EndComp
-$Comp
-L SCREW MT12
-U 1 1 4D283CBF
-P 3100 4400
-F 0 "MT12" H 3100 4300 40  0000 C CNN
-F 1 "SCREW" H 3100 4500 40  0001 C CNN
-F 2 "VITE_CSK_3MM" H 3100 4400 60  0001 C CNN
-	1    3100 4400
-	1    0    0    -1
-$EndComp
-$Comp
-L SCREW MT14
-U 1 1 4D283CB9
-P 3750 3800
-F 0 "MT14" H 3750 3700 40  0000 C CNN
-F 1 "SCREW" H 3750 3900 40  0001 C CNN
-F 2 "VITE_CSK_3MM" H 3750 3800 60  0001 C CNN
-	1    3750 3800
-	1    0    0    -1
-$EndComp
-$Comp
-L SCREW MT2
-U 1 1 4D283CB1
-P 4550 3800
-F 0 "MT2" H 4550 3700 40  0000 C CNN
-F 1 "SCREW" H 4550 3900 40  0001 C CNN
-F 2 "VITE_CSK_3MM" H 4550 3800 60  0001 C CNN
-	1    4550 3800
-	1    0    0    -1
-$EndComp
-$Comp
-L SCREW MT1
-U 1 1 4D283C9E
-P 4150 3800
-F 0 "MT1" H 4150 3700 40  0000 C CNN
-F 1 "SCREW" H 4150 3900 40  0001 C CNN
-F 2 "VITE_CSK_3MM" H 4150 3800 60  0001 C CNN
-	1    4150 3800
-	1    0    0    -1
-$EndComp
-$Comp
-L DIFFUSER FC1
-U 1 1 4D2828D4
-P 9900 1650
-F 0 "FC1" H 9900 1500 60  0000 C CNN
-F 1 "FRONT COVER" H 9900 1800 60  0000 C CNN
-F 2 "FrontCover" H 9900 1650 60  0001 C CNN
-	1    9900 1650
-	1    0    0    -1
-$EndComp
-$Comp
-L DIFFUSER FP1
-U 1 1 4D2828B9
-P 7000 3100
-F 0 "FP1" H 7000 2950 60  0000 C CNN
-F 1 "FACE PLATE" H 7000 3250 60  0000 C CNN
-F 2 "FrontCover" H 7000 3100 60  0001 C CNN
-	1    7000 3100
-	1    0    0    -1
-$EndComp
-Text Notes 2000 5600 0    40   ~ 0
-MOUNTING POSTS\n14 nos, around the board\n3mm internal thread, 5mm OD
-Text Notes 5100 4650 0    40   ~ 0
-DIFFUSER SCREWS\nCSK, 3mm
-$Comp
-L DIFFUSER DF1
-U 1 1 4D28255F
-P 4150 4650
-F 0 "DF1" H 4150 4500 60  0000 C CNN
-F 1 "DIFFUSER" H 4150 4800 60  0000 C CNN
-F 2 "DIFFUSER" H 4150 4650 60  0001 C CNN
-	1    4150 4650
-	1    0    0    -1
-$EndComp
-$Comp
-L BAFFLE BF1
-U 1 1 4D282455
-P 1800 6600
-F 0 "BF1" H 1400 7250 60  0000 C CNN
-F 1 "BAFFLE" H 2200 7250 60  0000 C CNN
-F 2 "BAFFLE" H 1800 6600 60  0001 C CNN
-	1    1800 6600
-	1    0    0    -1
-$EndComp
 $EndSCHEMATC

Commit message: 
Parts:
- added BF1: BAFFLE, Baffle, symbol BAFFLE
- added BP1: BackPlate, BackPlate, symbol DIFFUSER
- added FM1: FRAME, symbol FRAME
- added FP1: FacePlate, FacePlate, symbol DIFFUSER
Changed lines of the file:
@@
-EESchema Schematic File Version 2  date 05/03/11 17:26:50
+EESchema Schematic File Version 2  date 05/04/11 19:11:25
 LIBS:clock3
 LIBS:power
 LIBS:c3jr-cache
-LIBS:usb-b
 LIBS:c3jr-cache
 EELAYER 25  0
@@
 Sheet 3 4
 Title "ClockTHREE Junior aka C3Jr"
-Date "3 may 2011"
+Date "4 may 2011"
 Rev "A"
 Comp "an improved WordClock based on ClockTHREE"
@@
 Comment4 ""
 $EndDescr
+$Comp
+L FRAME FM1
+U 1 1 4DC15770
+P 6350 2100
+F 0 "FM1" H 6350 1950 60  0000 C CNN
+F 1 "FRAME" H 6350 2250 60  0000 C CNN
+	1    6350 2100
+	1    0    0    -1
+$EndComp
+$Comp
+L DIFFUSER BP1
+U 1 1 4DC14DC7
+P 8950 3850
+F 0 "BP1" H 8950 3700 60  0000 C CNN
+F 1 "BackPlate" H 8950 4000 60  0000 C CNN
+F 2 "BackPlate" H 8950 3850 60  0001 C CNN
+	1    8950 3850
+	1    0    0    -1
+$EndComp
+$Comp
+L DIFFUSER FP1
+U 1 1 4DC14DC3
+P 3450 3850
+F 0 "FP1" H 3450 3700 60  0000 C CNN
+F 1 "FacePlate" H 3450 4000 60  0000 C CNN
+F 2 "FacePlate" H 3450 3850 60  0001 C CNN
+	1    3450 3850
+	1    0    0    -1
+$EndComp
+$Comp
+L BAFFLE BF1
+U 1 1 4DC14DAD
+P 6300 3800
+F 0 "BF1" H 6350 3100 60  0000 C CNN
+F 1 "BAFFLE" H 6300 4450 60  0000 C CNN
+F 2 "Baffle" H 6300 3800 60  0001 C CNN
+	1    6300 3800
+	1    0    0    -1
+$EndComp
 $EndSCHEMATC
