File: KiCad/C3v2/C3v2-Aux.sch (KiCad schematic (older format))
At the start: 63 parts, among them IC1 DS1307, J1 V_IN, J2 V_IN, J3 V_IN, K1 PWR SEL, P10 CONN_1, P11 CONN_1, P12 V_OUT, P13 ISP, P14 CONN_1, P15 CONN_1, P16 CONN_1, P17 CONN_1, P18 CONN_1, P19 CONN_1, P20 CONN_1, P21 CONN_1, P22 CONN_1, P23 CONN_1, P24 DIL6, P25 DIL6, P26 DIL6, P27 DIL6, P28 DIL6, P29 DIL6, P30 DIL6, P31 DIL6, P32 DIL6, P33 DIL6, P34 DIL6, P35 DIL6, P36 DIL6, P37 DIL6, P38 DIL6, P39 DIL6, P41 STACK-L, P42 STACK-R, P48 7SegDisp, P49 CONN_1, P50 CONN_1, P51 CONN_1, P52 CONN_1, P7 FTDI, P8 CONN_1, P9 CONN_1, U1 DS3231, U5 7805, X2 32.768kHz

Commit message: C3v2 KiCad SCH / PCB update
Parts:
- BT1: footprint (none) -> CR2032
- C1: footprint (none) -> C2
- C10, C8: footprint CP_5x11mm -> CP_5X11MM
- IC1: footprint ds1307_pcf8583-DIL08 -> ds1307_SO8+SOIC8
- R24, R27, R28: footprint (none) -> RC03
- U1: footprint (none) -> DS3231
- X2: footprint (none) -> XTAL
Changed lines of the file:
@@
-EESchema Schematic File Version 2  date 06/02/11 15:47:38
+EESchema Schematic File Version 2  date 06/04/11 11:28:25
 LIBS:C3v2
 LIBS:power
@@
 Sheet 4 4
 Title "ClockTHREE"
-Date "2 jun 2011"
+Date "4 jun 2011"
 Rev "A"
 Comp "An Arduino friendly RGB LED Array"
@@
 F 0 "BT1" H 3150 1750 50  0000 C CNN
 F 1 "BATT_RTC" H 3550 1750 50  0000 C CNN
+F 2 "CR2032" H 3350 1850 60  0001 C CNN
 	1    3350 1850
 	0    1    1    0
@@
 F 0 "U1" H 5200 2350 60  0000 C CNN
 F 1 "DS3231" H 4600 1400 60  0000 C CNN
+F 2 "DS3231" H 4900 1800 60  0001 C CNN
 	1    4900 1800
 	1    0    0    -1
@@
 F 0 "IC1" H 7250 2450 50  0000 L BNN
 F 1 "DS1307" H 7250 1500 50  0000 L BNN
-F 2 "ds1307_pcf8583-DIL08" H 7550 2150 50  0001 C CNN
+F 2 "ds1307_SO8+SOIC8" H 7550 2150 50  0001 C CNN
 	1    7550 2000
 	1    0    0    -1
@@
 F 0 "X2" H 6750 2150 60  0000 C CNN
 F 1 "32.768kHz" H 6750 1850 60  0000 C CNN
+F 2 "XTAL" H 6750 2000 60  0001 C CNN
 	1    6750 2000
 	0    1    1    0
@@
 F 0 "R24" V 5930 1150 50  0000 C CNN
 F 1 "R" V 5850 1150 50  0000 C CNN
+F 2 "RC03" H 5850 1150 60  0001 C CNN
 	1    5850 1150
 	1    0    0    -1
@@
 F 0 "R27" V 6080 1150 50  0000 C CNN
 F 1 "R" V 6000 1150 50  0000 C CNN
+F 2 "RC03" H 6000 1150 60  0001 C CNN
 	1    6000 1150
 	1    0    0    -1
@@
 F 0 "R28" V 6230 1150 50  0000 C CNN
 F 1 "R" V 6150 1150 50  0000 C CNN
+F 2 "RC03" H 6150 1150 60  0001 C CNN
 	1    6150 1150
 	1    0    0    -1
@@
 F 0 "C1" V 3550 1600 50  0000 L CNN
 F 1 "100n" V 3650 1600 50  0000 L CNN
+F 2 "C2" H 3600 1800 60  0001 C CNN
 	1    3600 1800
 	1    0    0    -1
@@
 F 0 "C10" V 3200 4250 50  0000 L CNN
 F 1 "100u" V 3300 4250 50  0000 L CNN
-F 2 "CP_5x11mm" H 3400 4450 60  0001 C CNN
+F 2 "CP_5X11MM" H 3400 4450 60  0001 C CNN
 	1    3400 4450
 	1    0    0    -1
@@
 F 0 "C8" V 2100 4250 50  0000 L CNN
 F 1 "100u" V 2200 4250 50  0000 L CNN
-F 2 "CP_5x11mm" H 2150 4450 60  0001 C CNN
+F 2 "CP_5X11MM" H 2150 4450 60  0001 C CNN
 	1    2150 4450
 	1    0    0    -1

Commit message: C3 v2 KiCad design files
Parts:
- removed CD3: CDOT3, pin_strip_4, symbol CONN_4
- removed P20: CONN_1, vite_4mm, symbol CONN_1
- BT1: footprint CR2032 -> CR2032_SMD
- C10, C8: footprint CP_5X11MM -> CP_5x11mm
- J1, J2, J3: footprint JACK_ALIM -> JACK_ALIM_2
- P10, P11, P14, P15, P16, P17, P18, P19, P21, P22, P23, P8, P9: footprint vite_4mm -> vite_3mm
- P13: footprint PIN_STRIP_3X2 -> pin_strip_3x2
- P42: footprint PIN_STRIP_4-90 -> pin_strip_4-90
- P7: footprint PIN_STRIP_6-90 -> pin_strip_6-90
- U5: footprint VOLT_REG_78XX -> Volt_Reg_78xx
Connections:
- wire segments 266 -> 265
Other:
- note removed: "Add rtc chip on board, like in clockTWO"
