File: KiCad/C3v2/C3v2-LED.sch (KiCad schematic (older format))
At the start: 225 parts, among them K2 LED_ENABLE, Q1 2N5401, Q10 2N5401, Q11 2N5401, Q12 2N5401, Q13 2N5401, Q14 2N5401, Q15 2N5401, Q16 2N5401, Q2 2N5401, Q3 2N5401, Q4 2N5401, Q5 2N5401, Q6 2N5401, Q7 2N5401, Q8 2N5401, Q9 2N5401

Commit message: C3 v2 KiCad design files
Parts:
- 01D1, 01D10, 01D11, 01D12, 01D13, 01D14, 01D15, 01D16, 01D2, 01D3, 01D4, 01D5, 01D6, 01D7, 01D8, 01D9, 02D1, 02D10, 02D11, 02D12, 02D13, 02D14, 02D15, 02D16, 02D2, 02D3, 02D4, 02D5, 02D6, 02D7, 02D8, 02D9, 03D1, 03D10, 03D11, 03D12, 03D13, 03D14, 03D15, 03D16, 03D2, 03D3, 03D4, 03D5, 03D6, 03D7, 03D8, 03D9, 04D1, 04D10, 04D11, 04D12, 04D13, 04D14, 04D15, 04D16, 04D2, 04D3, 04D4, 04D5, 04D6, 04D7, 04D8, 04D9, 05D1, 05D10, 05D11, 05D12, 05D13, 05D14, 05D15, 05D16, 05D2, 05D3, 05D4, 05D5, 05D6, 05D7, 05D8, 05D9, 06D1, 06D10, 06D11, 06D12, 06D13, 06D14, 06D15, 06D16, 06D2, 06D3, 06D4, 06D5, 06D6, 06D7, 06D8, 06D9, 07D1, 07D10, 07D11, 07D12, 07D13, 07D14, 07D15, 07D16, 07D2, 07D3, 07D4, 07D5, 07D6, 07D7, 07D8, 07D9, 08D1, 08D10, 08D11, 08D12, 08D13, 08D14, 08D15, 08D16, 08D2, 08D3, 08D4, 08D5, 08D6, 08D7, 08D8, 08D9, 09D1, 09D10, 09D11, 09D12, 09D13, 09D14, 09D15, 09D16, 09D2, 09D3, 09D4, 09D5, 09D6, 09D7, 09D8, 09D9, 10D1, 10D10, 10D11, 10D12, 10D13, 10D14, 10D15, 10D16, 10D2, 10D3, 10D4, 10D5, 10D6, 10D7, 10D8, 10D9: footprint 01D01 -> LED_RGB_10
- 11D1, 11D10, 11D11, 11D12, 11D13, 11D14, 11D15, 11D16, 11D2, 11D3, 11D4, 11D5, 11D6, 11D7, 11D8, 11D9, 12D1, 12D10, 12D11, 12D12, 12D13, 12D14, 12D15, 12D16, 12D2, 12D3, 12D4, 12D5, 12D6, 12D7, 12D8, 12D9: footprint LED_10MM_BLUE -> led_10mm_blue
- K2: footprint pin_strip_3 -> LED_Enable_pin3
Other:
- note removed: "ISSUE 7 : DONE"
