File: KiCad/C3v2/C3v2-mech.sch (KiCad schematic (older format))
At the start: 18 parts

Commit message: C3v2 KiCad SCH / PCB update
Parts:
- removed MT1, MT11, MT12, MT14, MT2, MT4, MT5, MT7, MT8: SCREW, VITE_CSK_3MM, symbol SCREW
- FP1: footprint FrontCover -> FacePlate
Changed lines of the file:
@@
-EESchema Schematic File Version 2  date 06/02/11 15:47:38
+EESchema Schematic File Version 2  date 06/04/11 11:28:25
 LIBS:C3v2
 LIBS:power
@@
 Sheet 2 4
 Title "ClockTHREE"
-Date "2 jun 2011"
+Date "4 jun 2011"
 Rev "A"
 Comp "An Arduino friendly RGB LED Array"
@@
 $EndComp
 $Comp
-L SCREW MT4
-U 1 1 4D283CE6
-P 5200 4400
-F 0 "MT4" H 5200 4300 40  0000 C CNN
-F 1 "SCREW" H 5200 4500 40  0001 C CNN
-F 2 "VITE_CSK_3MM" H 5200 4400 60  0001 C CNN
-	1    5200 4400
-	1    0    0    -1
-$EndComp
-$Comp
-L SCREW MT5
-U 1 1 4D283CDD
-P 5200 4900
-F 0 "MT5" H 5200 4800 40  0000 C CNN
-F 1 "SCREW" H 5200 5000 40  0001 C CNN
-F 2 "VITE_CSK_3MM" H 5200 4900 60  0001 C CNN
-	1    5200 4900
-	1    0    0    -1
-$EndComp
-$Comp
-L SCREW MT7
-U 1 1 4D283CC9
-P 4550 5500
-F 0 "MT7" H 4550 5400 40  0000 C CNN
-F 1 "SCREW" H 4550 5600 40  0001 C CNN
-F 2 "VITE_CSK_3MM" H 4550 5500 60  0001 C CNN
-	1    4550 5500
-	1    0    0    -1
-$EndComp
-$Comp
-L SCREW MT8
-U 1 1 4D283CC6
-P 4150 5500
-F 0 "MT8" H 4150 5400 40  0000 C CNN
-F 1 "SCREW" H 4150 5600 40  0001 C CNN
-F 2 "VITE_CSK_3MM" H 4150 5500 60  0001 C CNN
-	1    4150 5500
-	1    0    0    -1
-$EndComp
-$Comp
-L SCREW MT11
-U 1 1 4D283CC3
-P 3100 4900
-F 0 "MT11" H 3100 4800 40  0000 C CNN
-F 1 "SCREW" H 3100 5000 40  0001 C CNN
-F 2 "VITE_CSK_3MM" H 3100 4900 60  0001 C CNN
-	1    3100 4900
-	1    0    0    -1
-$EndComp
-$Comp
-L SCREW MT12
-U 1 1 4D283CBF
-P 3100 4400
-F 0 "MT12" H 3100 4300 40  0000 C CNN
-F 1 "SCREW" H 3100 4500 40  0001 C CNN
-F 2 "VITE_CSK_3MM" H 3100 4400 60  0001 C CNN
-	1    3100 4400
-	1    0    0    -1
-$EndComp
-$Comp
-L SCREW MT14
-U 1 1 4D283CB9
-P 3750 3800
-F 0 "MT14" H 3750 3700 40  0000 C CNN
-F 1 "SCREW" H 3750 3900 40  0001 C CNN
-F 2 "VITE_CSK_3MM" H 3750 3800 60  0001 C CNN
-	1    3750 3800
-	1    0    0    -1
-$EndComp
-$Comp
-L SCREW MT2
-U 1 1 4D283CB1
-P 4550 3800
-F 0 "MT2" H 4550 3700 40  0000 C CNN
-F 1 "SCREW" H 4550 3900 40  0001 C CNN
-F 2 "VITE_CSK_3MM" H 4550 3800 60  0001 C CNN
-	1    4550 3800
-	1    0    0    -1
-$EndComp
-$Comp
-L SCREW MT1
-U 1 1 4D283C9E
-P 4150 3800
-F 0 "MT1" H 4150 3700 40  0000 C CNN
-F 1 "SCREW" H 4150 3900 40  0001 C CNN
-F 2 "VITE_CSK_3MM" H 4150 3800 60  0001 C CNN
-	1    4150 3800
-	1    0    0    -1
-$EndComp
-$Comp
 L DIFFUSER FC1
 U 1 1 4D2828D4
@@
 F 0 "FP1" H 7000 2950 60  0000 C CNN
 F 1 "FACE PLATE" H 7000 3250 60  0000 C CNN
-F 2 "FrontCover" H 7000 3100 60  0001 C CNN
+F 2 "FacePlate" H 7000 3100 60  0001 C CNN
 	1    7000 3100
 	1    0    0    -1

Commit message: C3 v2 KiCad design files
Parts:
- BF1: footprint BAFFLE -> Baffle
- DF1: footprint DIFFUSER -> Diffuser
Changed lines of the file:
@@
-EESchema Schematic File Version 2  date 06/04/11 11:28:25
+EESchema Schematic File Version 2  date 07/29/11 13:59:18
 LIBS:C3v2
 LIBS:power
@@
 encoding utf-8
 Sheet 2 4
-Title "ClockTHREE"
-Date "4 jun 2011"
+Title "ClockTHREE Version 2"
+Date "29 jul 2011"
 Rev "A"
 Comp "An Arduino friendly RGB LED Array"
-Comment1 "Wyo Innovations      :: Lumetronics"
+Comment1 "www.wyolum.com"
 Comment2 "wyojustin@gmail.com :: anool.m@gmail.com"
-Comment3 "wyoinnovation.blogspot.com"
-Comment4 "part of the project inspired from : http://www.evilmadscientist.com/article.php/peggy2"
+Comment3 ""
+Comment4 ""
 $EndDescr
 $Comp
@@
 F 0 "DF1" H 4150 4500 60  0000 C CNN
 F 1 "DIFFUSER" H 4150 4800 60  0000 C CNN
-F 2 "DIFFUSER" H 4150 4650 60  0001 C CNN
+F 2 "Diffuser" H 4150 4650 60  0001 C CNN
 	1    4150 4650
 	1    0    0    -1
@@
 F 0 "BF1" H 1400 7250 60  0000 C CNN
 F 1 "BAFFLE" H 2200 7250 60  0000 C CNN
-F 2 "BAFFLE" H 1800 6600 60  0001 C CNN
+F 2 "Baffle" H 1800 6600 60  0001 C CNN
 	1    1800 6600
 	1    0    0    -1
