File: KiCad/C3v2/C3v2.sch (KiCad schematic (older format))
At the start: 31 parts, among them P43 CONN_1, Q17 2N5401, SW1 INC, SW2 DEC, SW3 MODE, SW4 RST, SW5 ENTER, U3 ATMEGA8-P, U4 74LS154, X1 16MHz

Commit message: C3v2 KiCad SCH / PCB update
Parts:
- R32: footprint (none) -> pin_strip_2
Changed lines of the file:
@@
-EESchema Schematic File Version 2  date 06/02/11 15:47:38
+EESchema Schematic File Version 2  date 06/04/11 11:28:25
 LIBS:C3v2
 LIBS:power
@@
 Sheet 1 4
 Title "ClockTHREE"
-Date "2 jun 2011"
+Date "4 jun 2011"
 Rev "A"
 Comp "An Arduino friendly RGB LED Array"
@@
 F 0 "R32" V 5655 7200 50  0000 C CNN
 F 1 "LDR" V 5575 7200 50  0000 C CNN
+F 2 "pin_strip_2" H 5575 7200 60  0001 C CNN
 	1    5575 7200
 	1    0    0    -1

Commit message: C3 v2 KiCad design files
Parts:
- removed D1: 1N4148, diode_do35, symbol DIODE
- SP1: footprint SPEAKER -> Speaker
Changed lines of the file:
@@
-EESchema Schematic File Version 2  date 06/04/11 11:28:25
+EESchema Schematic File Version 2  date 07/29/11 13:59:18
 LIBS:C3v2
 LIBS:power
@@
 encoding utf-8
 Sheet 1 4
-Title "ClockTHREE"
-Date "4 jun 2011"
+Title "ClockTHREE Version 2"
+Date "29 jul 2011"
 Rev "A"
 Comp "An Arduino friendly RGB LED Array"
-Comment1 "Wyo Innovations      :: Lumetronics"
+Comment1 "www.wyolum.com"
 Comment2 "wyojustin@gmail.com :: anool.m@gmail.com"
-Comment3 "wyoinnovation.blogspot.com"
-Comment4 "part of the project inspired from : http://www.evilmadscientist.com/article.php/peggy2"
+Comment3 ""
+Comment4 ""
 $EndDescr
 $Comp
@@
 	8875 5400 8875 5550
 Connection ~ 5575 7500
-Connection ~ 3500 5550
-Wire Wire Line
-	3500 5550 3500 5850
-Wire Wire Line
-	3500 5850 3675 5850
 Connection ~ 4175 3450
 Wire Wire Line
@@
 Wire Wire Line
 	3350 5450 3500 5450
-Wire Wire Line
-	4075 5850 4175 5850
-Connection ~ 4175 5850
 Wire Wire Line
 	8625 5125 8625 5275
@@
 F1 "C3v2-mech.sch" 60
 $EndSheet
-$Comp
-L DIODE D1
-U 1 1 4D25BDEF
-P 3875 5850
-F 0 "D1" H 3875 5950 40  0000 C CNN
-F 1 "1N4148" H 3875 5750 40  0000 C CNN
-F 2 "diode_do35" H 3875 5850 60  0001 C CNN
-	1    3875 5850
-	1    0    0    -1
-$EndComp
 Text Notes 8250 1700 0    40   ~ 0
 Mounting Hole for rowBoB
@@
 F 0 "SP1" H 5175 7000 70  0000 C CNN
 F 1 "SPEAKER" H 5275 7400 70  0000 C CNN
-F 2 "SPEAKER" H 5200 7200 60  0001 C CNN
+F 2 "Speaker" H 5200 7200 60  0001 C CNN
 F 3 "http://products.cui.com/GetSpecForDigiKey.aspx?MFGNum=CEM-14R06CT" H 5200 7200 60  0001 C CNN
 F 4 "102-1169-ND" H 5200 7200 60  0001 C CNN "DigiKey"
