File: KiCad/Nb_v1/Nb_v1-mech.sch (KiCad schematic (older format))
At the start: 4 parts

Commit message: Nachbau, started initial spade work on PCB
Parts:
- FM1: footprint (none) -> Frame
Changed lines of the file:
@@
-EESchema Schematic File Version 2  date 11/25/2011 1:26:45 PM
+EESchema Schematic File Version 2  date 11/25/2011 7:19:25 PM
 LIBS:Nb_v1
 LIBS:power
+LIBS:conn
 LIBS:Nb_v1-cache
 EELAYER 25  0
@@
 F 0 "FM1" H 6350 1950 60  0000 C CNN
 F 1 "FRAME" H 6350 2250 60  0000 C CNN
+F 2 "Frame" H 6350 2100 60  0001 C CNN
 	1    6350 2100
 	1    0    0    -1

Commit message: Nachbau Schematic almost final, working on PCB component layout first
Parts:
- removed BF1: BAFFLE, Baffle, symbol BAFFLE
- removed BP1: BackPlate, BackPlate, symbol DIFFUSER
- removed FM1: FRAME, Frame, symbol FRAME
- removed FP1: FacePlate, FacePlate, symbol DIFFUSER
Changed lines of the file:
@@
-EESchema Schematic File Version 2  date Fri 25 Nov 2011 10:46:27 PM IST
+EESchema Schematic File Version 2  date 11/26/2011 1:49:00 PM
 LIBS:Nb_v1
 LIBS:power
-LIBS:conn
 LIBS:Nb_v1-cache
 EELAYER 25  0
@@
 Sheet 3 4
 Title "NachBau - WordClock"
-Date "25 nov 2011"
+Date "26 nov 2011"
 Rev "A"
 Comp ""
@@
 Comment4 ""
 $EndDescr
-$Comp
-L FRAME FM1
-U 1 1 4DC15770
-P 6350 2100
-F 0 "FM1" H 6350 1950 60  0000 C CNN
-F 1 "FRAME" H 6350 2250 60  0000 C CNN
-F 2 "Frame" H 6350 2100 60  0001 C CNN
-	1    6350 2100
-	1    0    0    -1
-$EndComp
-$Comp
-L DIFFUSER BP1
-U 1 1 4DC14DC7
-P 8950 3850
-F 0 "BP1" H 8950 3700 60  0000 C CNN
-F 1 "BackPlate" H 8950 4000 60  0000 C CNN
-F 2 "BackPlate" H 8950 3850 60  0001 C CNN
-	1    8950 3850
-	1    0    0    -1
-$EndComp
-$Comp
-L DIFFUSER FP1
-U 1 1 4DC14DC3
-P 3450 3850
-F 0 "FP1" H 3450 3700 60  0000 C CNN
-F 1 "FacePlate" H 3450 4000 60  0000 C CNN
-F 2 "FacePlate" H 3450 3850 60  0001 C CNN
-	1    3450 3850
-	1    0    0    -1
-$EndComp
-$Comp
-L BAFFLE BF1
-U 1 1 4DC14DAD
-P 6300 3800
-F 0 "BF1" H 6350 3100 60  0000 C CNN
-F 1 "BAFFLE" H 6300 4450 60  0000 C CNN
-F 2 "Baffle" H 6300 3800 60  0001 C CNN
-	1    6300 3800
-	1    0    0    -1
-$EndComp
 $EndSCHEMATC
