File: KiCad/C3Jr_v2/c3jr_v2-Aux.sch (KiCad schematic (older format))
At the start: 53 parts, among them J1 V_IN, J2 V_IN, J3 V_IN, K1 PWR SEL, K3 7Seg_Sel, P1 7SegDisp, P10 CONN_1, P11 CONN_1, P12 V_OUT, P13 ISP, P14 CONN_1, P15 CONN_1, P24 DIL6, P25 DIL6, P26 DIL6, P27 DIL6, P28 DIL6, P29 DIL6, P30 DIL6, P31 DIL6, P32 DIL6, P33 DIL6, P34 DIL6, P35 DIL6, P36 DIL6, P37 DIL6, P38 DIL6, P39 DIL6, P41 STACK-L, P42 STACK-R, P49 CONN_1, P50 CONN_1, P51 CONN_1, P52 CONN_1, P53 CONN_1, P54 CONN_1, P7 FTDI, P8 CONN_1, P9 CONN_1, U6 DS3231N

Commit message: C3jr_v2-Added extra buttons for rear side. Some track clean up. Added OSHW and WyoLum Logos. Final for Production.
Parts:
- J1: footprint (none) -> con-hirose-UX60-MB-5S8
- J3: footprint (none) -> JACK_ALIM
- K3: footprint (none) -> 7Seg_Sel
Changed lines of the file:
@@
-EESchema Schematic File Version 2  date Sunday 18 December 2011 08:43:59 PM IST
+EESchema Schematic File Version 2  date 1/5/2012 2:50:43 PM
 LIBS:C3Jr_v2
 LIBS:power
@@
 Sheet 4 4
 Title "ClockTHREE Junior aka C3Jr_v2 , with stackable board"
-Date "18 dec 2011"
+Date "4 jan 2012"
 Rev "A"
 Comp "an improved WordClock based on ClockTHREE"
@@
 F 0 "K3" V 5650 6050 50  0000 C CNN
 F 1 "7Seg_Sel" V 5750 6050 40  0000 C CNN
+F 2 "7Seg_Sel" H 5700 6050 60  0001 C CNN
 	1    5700 6050
 	1    0    0    -1
@@
 BAT
 $Comp
-L VCC #PWR017
+L VCC #PWR016
 U 1 1 4EDA2127
 P 4150 5800
-F 0 "#PWR017" H 4150 5900 30  0001 C CNN
+F 0 "#PWR016" H 4150 5900 30  0001 C CNN
 F 1 "VCC" H 4150 5900 30  0000 C CNN
 	1    4150 5800
@@
 $EndComp
 $Comp
-L GND #PWR018
+L GND #PWR017
 U 1 1 4EDA2121
 P 3350 7250
-F 0 "#PWR018" H 3350 7250 30  0001 C CNN
+F 0 "#PWR017" H 3350 7250 30  0001 C CNN
 F 1 "GND" H 3350 7180 30  0001 C CNN
 	1    3350 7250
@@
 $EndComp
 $Comp
-L PWR_FLAG #FLG019
+L PWR_FLAG #FLG018
 U 1 1 4EDA10E3
 P 3350 1000
-F 0 "#FLG019" H 3350 1270 30  0001 C CNN
+F 0 "#FLG018" H 3350 1270 30  0001 C CNN
 F 1 "PWR_FLAG" H 3350 1230 30  0000 C CNN
 	1    3350 1000
@@
 $EndComp
 $Comp
-L PWR_FLAG #FLG020
+L PWR_FLAG #FLG019
 U 1 1 4EDA108C
 P 9950 1300
-F 0 "#FLG020" H 9950 1570 30  0001 C CNN
+F 0 "#FLG019" H 9950 1570 30  0001 C CNN
 F 1 "PWR_FLAG" H 9950 1530 30  0000 C CNN
 	1    9950 1300
@@
 F 0 "J3" V 1000 5025 40  0000 C CNN
 F 1 "V_IN" V 1100 5025 40  0000 C CNN
+F 2 "JACK_ALIM" H 1050 5025 60  0001 C CNN
 	1    1050 5025
 	-1   0    0    -1
@@
 F 0 "J1" V 1025 4000 50  0000 L BNN
 F 1 "V_IN" V 1025 3475 50  0000 L BNN
+F 2 "con-hirose-UX60-MB-5S8" H 1100 3800 60  0001 C CNN
 F 3 "H2959CT-ND" H 1100 3800 60  0001 C CNN
 F 4 "http://search.digikey.com/us/en/products/UX60-MB-5ST/H2959CT-ND/597538" V 1100 3800 60  0001 C CNN "Link"
@@
 7Seg_Data
 $Comp
-L VCC #PWR021
+L VCC #PWR020
 U 1 1 4DBD205C
 P 5050 6550
-F 0 "#PWR021" H 5050 6650 30  0001 C CNN
+F 0 "#PWR020" H 5050 6650 30  0001 C CNN
 F 1 "VCC" H 5050 6650 30  0000 C CNN
 	1    5050 6550
@@
 $EndComp
 $Comp
-L GND #PWR022
+L GND #PWR021
 U 1 1 4DBD204B
 P 5050 6850
-F 0 "#PWR022" H 5050 6850 30  0001 C CNN
+F 0 "#PWR021" H 5050 6850 30  0001 C CNN
 F 1 "GND" H 5050 6780 30  0001 C CNN
 	1    5050 6850
@@
 VCC
 $Comp
-L GND #PWR023
+L GND #PWR022
 U 1 1 4DBAC297
 P 3775 3025
-F 0 "#PWR023" H 3775 3025 30  0001 C CNN
+F 0 "#PWR022" H 3775 3025 30  0001 C CNN
 F 1 "GND" H 3775 2955 30  0001 C CNN
 	1    3775 3025
@@
 $EndComp
 $Comp
-L VCC #PWR024
+L VCC #PWR023
 U 1 1 4DBAC28D
 P 3775 825
-F 0 "#PWR024" H 3775 925 30  0001 C CNN
+F 0 "#PWR023" H 3775 925 30  0001 C CNN
 F 1 "VCC" H 3775 925 30  0000 C CNN
 	1    3775 825
@@
 $EndComp
 $Comp
-L VCC #PWR025
+L VCC #PWR024
 U 1 1 4C109AAB
 P 9400 1150
-F 0 "#PWR025" H 9400 1250 30  0001 C CNN
+F 0 "#PWR024" H 9400 1250 30  0001 C CNN
 F 1 "VCC" H 9400 1250 30  0000 C CNN
 	1    9400 1150
@@
 $EndComp
 $Comp
-L GND #PWR026
+L GND #PWR025
 U 1 1 4C109AAA
 P 9450 2350
-F 0 "#PWR026" H 9450 2350 30  0001 C CNN
+F 0 "#PWR025" H 9450 2350 30  0001 C CNN
 F 1 "GND" H 9450 2280 30  0001 C CNN
 	1    9450 2350
@@
 USB5V
 $Comp
-L VDD #PWR027
+L VDD #PWR026
 U 1 1 4C109AA4
 P 9600 1150
-F 0 "#PWR027" H 9600 1250 30  0001 C CNN
+F 0 "#PWR026" H 9600 1250 30  0001 C CNN
 F 1 "VDD" H 9600 1260 30  0000 C CNN
 	1    9600 1150
@@
 $EndComp
 $Comp
-L VSS #PWR028
+L VSS #PWR027
 U 1 1 4B3F12CE
 P 3050 5300
-F 0 "#PWR028" H 3050 5300 30  0001 C CNN
+F 0 "#PWR027" H 3050 5300 30  0001 C CNN
 F 1 "VSS" H 3150 5350 30  0000 C CNN
 	1    3050 5300
@@
 $EndComp
 $Comp
-L GND #PWR029
+L GND #PWR028
 U 1 1 4B3F12CB
 P 2600 5300
-F 0 "#PWR029" H 2600 5300 30  0001 C CNN
+F 0 "#PWR028" H 2600 5300 30  0001 C CNN
 F 1 "GND" H 2600 5230 30  0001 C CNN
 F 4 "GND" H 2500 5350 60  0000 C CNN "Field1"

Commit message: c3jr_v2 user guide
Connections:
- net labels removed: VRAW
- wire segments 254 -> 253

Commit message: C3Jr_v2 Switches moved 0.6" to left (for i2sd). Added C1 and C2 (100uF) for C3SB filtering
Parts:
- added C1, C2: 100u, CP_5x11mm, symbol CP1
Connections:
- net labels added: VRAW
- wire segments 253 -> 260
Other:
- note added: "C3SB (i2c bus)"
- note removed: "STACK COMM"
- moved on the sheet: P41
Changed lines of the file:
@@
-EESchema Schematic File Version 2  date Sunday 22 January 2012 12:19:31 PM IST
+EESchema Schematic File Version 2  date 1/23/2012 5:52:41 PM
 LIBS:C3Jr_v2
 LIBS:power
@@
 Sheet 4 4
 Title "ClockTHREE Junior aka C3Jr_v2 , with stackable board"
-Date "22 jan 2012"
+Date "23 jan 2012"
 Rev "A"
 Comp "an improved WordClock based on ClockTHREE"
@@
 Comment4 ""
 $EndDescr
-Wire Wire Line
-	1800 4100 1800 4250
+Wire Notes Line
+	10700 5875 10700 4700
+Wire Notes Line
+	10700 5875 8600 5875
+Wire Notes Line
+	8600 5875 8600 4700
+Wire Notes Line
+	8600 4700 10700 4700
+Connection ~ 9500 5225
+Wire Wire Line
+	9500 5225 9500 5750
+Wire Wire Line
+	9750 5675 9750 5750
+Connection ~ 9300 4925
+Wire Wire Line
+	9300 4925 9300 5275
 Wire Wire Line
 	5800 5750 5250 5750
@@
 Connection ~ 5975 2400
 Wire Wire Line
-	5975 2400 5850 2400
+	5850 2400 5975 2400
 Connection ~ 5975 2200
 Wire Wire Line
@@
 	2600 5200 2600 5300
 Wire Wire Line
-	9400 4925 9900 4925
+	9900 4925 9175 4925
 Wire Notes Line
 	6050 3500 6050 5400
@@
 Wire Notes Line
 	8600 4550 8600 850
-Wire Notes Line
-	8600 5425 8600 4725
-Wire Notes Line
-	8600 5425 10700 5425
-Wire Notes Line
-	10700 5425 10700 4725
 Wire Wire Line
 	1000 7500 950  7500
 Wire Wire Line
-	9400 5125 9900 5125
+	9175 5125 9900 5125
 Wire Notes Line
 	750  7700 750  5500
@@
 Wire Wire Line
 	3600 4000 3450 4000
+Wire Wire Line
+	1800 4250 1800 3650
+Wire Wire Line
+	1800 3650 4500 3650
 Connection ~ 10150 1400
 Wire Wire Line
@@
 	750  5400 6050 5400
 Wire Wire Line
-	9900 5225 9400 5225
-Wire Wire Line
-	9900 5025 9400 5025
-Wire Notes Line
-	10700 4725 8600 4725
+	9175 5225 9900 5225
+Wire Wire Line
+	9900 5025 9175 5025
 Wire Wire Line
 	2900 7500 2950 7500
@@
 Wire Wire Line
 	5250 6350 5800 6350
+Wire Wire Line
+	9750 5275 9750 4925
+Connection ~ 9750 4925
+Wire Wire Line
+	9300 5675 9300 5750
+Wire Wire Line
+	9300 5750 9750 5750
+Connection ~ 9500 5750
+$Comp
+L CP1 C2
+U 1 1 4F1D4EB4
+P 9750 5475
+F 0 "C2" V 9700 5275 50  0000 L CNN
+F 1 "100u" V 9800 5275 50  0000 L CNN
+F 2 "CP_5x11mm" H 9750 5475 60  0001 C CNN
+	1    9750 5475
+	1    0    0    -1
+$EndComp
+$Comp
+L CP1 C1
+U 1 1 4F1D4E51
+P 9300 5475
+F 0 "C1" V 9250 5275 50  0000 L CNN
+F 1 "100u" V 9350 5275 50  0000 L CNN
+F 2 "CP_5x11mm" H 9300 5475 60  0001 C CNN
+	1    9300 5475
+	1    0    0    -1
+$EndComp
 Text HLabel 5800 5750 2    40   Input ~ 0
 DBG
@@
 	0    -1   -1   0
 $EndComp
-Text Notes 8600 5525 0    40   ~ 0
+Text Notes 8600 5975 0    40   ~ 0
 Stack-L and Stack-R have inverted pin nos\nsince one is facing Left and other is facing right.\nWhen mounted this way on the board,\ntracks from one to the other will be parallel - no cross over.
 Text HLabel 2550 2550 2    40   Input ~ 0
@@
 	1    0    0    -1
 $EndComp
-Text Notes 10100 5425 0    60   ~ 0
-STACK COMM
+Text Notes 10000 4800 0    60   ~ 0
+C3SB (i2c bus)
 Text Label 9550 5225 0    40   ~ 0
 GND
@@
 L CONN_4 P41
 U 1 1 4C9A16BC
-P 9050 5075
-F 0 "P41" V 9000 5075 50  0000 C CNN
-F 1 "STACK-L" V 9100 5075 50  0000 C CNN
-F 2 "pin_sck_4-90" H 9050 5075 60  0001 C CNN
-	1    9050 5075
+P 8825 5075
+F 0 "P41" V 8775 5075 50  0000 C CNN
+F 1 "STACK-L" V 8875 5075 50  0000 C CNN
+F 2 "pin_sck_4-90" H 8825 5075 60  0001 C CNN
+	1    8825 5075
 	-1   0    0    -1
 $EndComp
@@
 	1    0    0    -1
 $EndComp
+Text Label 3800 3650 0    40   ~ 0
+VRAW
 Text Label 9800 1400 2    40   ~ 0
 VCC
@@
 Text HLabel 4500 5000 2    47   Input ~ 0
 VSS
+Text HLabel 4500 3650 2    47   Input ~ 0
+VRAW
 Text Notes 5300 5350 0    60   ~ 0
 POWER SUPPLY

Commit message: C3jr_v2 : added jumper selector for RTC select, 2 pin headers for Switches, cleaned top Silk, Mini_USB error rectified. Gerber plots ready for a pre-production trial.
Parts:
- added K4: SCL, pin_strip_3, symbol CONN_3
- added K5: SDA, pin_strip_3, symbol CONN_3
Connections:
- net labels added: SCL_EXT, SCL_INT, SDA_EXT, SDA_INT
- wire segments 260 -> 264
- no-connect marks 12 -> 14
Other:
- note added: "EXTERNAL RTC\nI2SD\nrtcBoB\nChronoDOT"
- note added: "INTERNAL RTC\nDS3231"
- note added: "Jumpers, to select\nINT or EXT RTC Chip"
- note added: "Mounting Holes for\nrtcBoB / ChronoDOT"
- note removed: "Mounting Holes for rtcBoB"

Commit message: C3jr_v2 Modified SCL and SDA selection jumpers K4 and K5. Need to get a few sample boards before KS production run.
Parts:
- removed K4: SCL, pin_strip_3, symbol CONN_3
- removed K5: SDA, pin_strip_3, symbol CONN_3
- added K4: SCL, pin_strip_2, symbol CONN_2
- added K5: SDA, pin_strip_2, symbol CONN_2
Connections:
- net labels removed: SCL_EXT, SDA_EXT
- wire segments 264 -> 262
Changed lines of the file:
@@
-EESchema Schematic File Version 2  date 2/11/2012 5:26:33 PM
+EESchema Schematic File Version 2  date 2/13/2012 3:14:02 PM
 LIBS:C3Jr_v2
 LIBS:power
@@
 Sheet 4 4
 Title "ClockTHREE Junior aka C3Jr_v2 , with stackable board"
-Date "11 feb 2012"
+Date "13 feb 2012"
 Rev "A"
 Comp "an improved WordClock based on ClockTHREE"
@@
 Comment4 ""
 $EndDescr
+$Comp
+L CONN_2 K5
+U 1 1 4F38DADB
+P 1200 1400
+F 0 "K5" V 1150 1400 40  0000 C CNN
+F 1 "SDA" V 1250 1400 40  0000 C CNN
+F 2 "pin_strip_2" V 1350 1400 40  0001 C CNN
+	1    1200 1400
+	-1   0    0    1
+$EndComp
+$Comp
+L CONN_2 K4
+U 1 1 4F38DAA4
+P 1200 1000
+F 0 "K4" V 1150 1000 40  0000 C CNN
+F 1 "SCL" V 1250 1000 40  0000 C CNN
+F 2 "pin_strip_2" V 1350 1000 40  0001 C CNN
+	1    1200 1000
+	-1   0    0    1
+$EndComp
 NoConn ~ 1150 4000
 NoConn ~ 1100 4000
@@
 Text Label 1950 1500 2    40   ~ 0
 SDA_INT
-Text Label 1950 1300 2    40   ~ 0
-SDA_EXT
 Text Label 1950 1100 2    40   ~ 0
 SCL_INT
-Text Label 1950 900  2    40   ~ 0
-SCL_EXT
 Text Label 2950 2550 0    40   ~ 0
 SDA_INT
@@
 	1550 1500 1950 1500
 Wire Wire Line
-	1550 1300 1950 1300
-Wire Wire Line
-	1550 1000 2100 1000
+	1550 900  2100 900
 Wire Notes Line
 	10700 5875 10700 4700
@@
 Connection ~ 9500 5750
 Wire Wire Line
-	1550 900  1950 900
-Wire Wire Line
 	1550 1100 1950 1100
 Wire Wire Line
-	1550 1400 2100 1400
+	1550 1300 2100 1300
 Wire Wire Line
 	3950 2450 2950 2450
-$Comp
-L CONN_3 K5
-U 1 1 4F3608CC
-P 1200 1400
-F 0 "K5" V 1150 1400 50  0000 C CNN
-F 1 "SDA" V 1250 1400 40  0000 C CNN
-F 2 "pin_strip_3" V 1350 1400 40  0001 C CNN
-	1    1200 1400
-	-1   0    0    1
-$EndComp
-$Comp
-L CONN_3 K4
-U 1 1 4F36082E
-P 1200 1000
-F 0 "K4" V 1150 1000 50  0000 C CNN
-F 1 "SCL" V 1250 1000 40  0000 C CNN
-F 2 "pin_strip_3" V 1350 1000 40  0001 C CNN
-	1    1200 1000
-	-1   0    0    1
-$EndComp
 $Comp
 L CP1 C2
@@
 Text Notes 8600 5975 0    40   Italic 8
 Stack-L and Stack-R have inverted pin nos\nsince one is facing Left and other is facing right.\nWhen mounted this way on the board,\ntracks from one to the other will be parallel - no cross over.
-Text HLabel 2100 1400 2    40   Input ~ 0
+Text HLabel 2100 1300 2    40   Input ~ 0
 SDA
-Text HLabel 2100 1000 2    40   Input ~ 0
+Text HLabel 2100 900  2    40   Input ~ 0
 SCL
 Text Notes 6575 3300 0    60   ~ 0
@@
 $EndComp
 Text Label 2700 2550 2    40   ~ 0
-SDA_EXT
+SDA
 Text Label 2700 2450 2    40   ~ 0
-SCL_EXT
+SCL
 Text Label 2450 2350 0    40   ~ 0
 VCC

Commit message: C3jr_v2 : removed V_OUT (P12) header. Added 7805 Volt Reg (TO-220 horizontal) and 100nF Cap "C4" on output of V. Reg. Final Gerbers for trial boards from seeed.
Parts:
- removed P12: V_OUT, pin_strip_3, symbol CONN_3
- added C4: 100n, C2, symbol C
- added U2: 7805, symbol 7805
Connections:
- wire segments 262 -> 260
