File: KiCad/C3Jr_v2/c3jr_v2-LED.sch (KiCad schematic (older format))
At the start: 161 parts, among them K2 LED_ENABLE, Q1 2N5401, Q10 2N5401, Q11 2N5401, Q12 2N5401, Q13 2N5401, Q14 2N5401, Q15 2N5401, Q16 2N5401, Q2 2N5401, Q3 2N5401, Q4 2N5401, Q5 2N5401, Q6 2N5401, Q7 2N5401, Q8 2N5401, Q9 2N5401

Commit message: C3jr_v2-Added extra buttons for rear side. Some track clean up. Added OSHW and WyoLum Logos. Final for Production.
Parts:
- R1, R10, R11, R12, R13, R14, R15, R16, R2, R3, R4, R5, R6, R7, R8, R9: footprint RC03 -> rc03_vert
Changed lines of the file:
@@
-EESchema Schematic File Version 2  date Sunday 18 December 2011 08:43:59 PM IST
+EESchema Schematic File Version 2  date 1/5/2012 2:50:43 PM
 LIBS:C3Jr_v2
 LIBS:power
@@
 Sheet 2 4
 Title "ClockTHREE Junior aka C3Jr_v2 , with stackable board"
-Date "18 dec 2011"
+Date "15 dec 2011"
 Rev "A"
 Comp "an improved WordClock based on ClockTHREE"
@@
 F 0 "R16" V 2330 950 50  0000 C CNN
 F 1 "100" V 2250 950 50  0000 C CNN
-F 2 "RC03" H 2250 950 60  0001 C CNN
+F 2 "rc03_vert" H 2250 950 60  0001 C CNN
 	1    2250 950
 	1    0    0    -1
@@
 F 0 "R15" V 3130 950 50  0000 C CNN
 F 1 "100" V 3050 950 50  0000 C CNN
-F 2 "RC03" H 3050 950 60  0001 C CNN
+F 2 "rc03_vert" H 3050 950 60  0001 C CNN
 	1    3050 950
 	1    0    0    -1
@@
 F 0 "R14" V 3930 950 50  0000 C CNN
 F 1 "100" V 3850 950 50  0000 C CNN
-F 2 "RC03" H 3850 950 60  0001 C CNN
+F 2 "rc03_vert" H 3850 950 60  0001 C CNN
 	1    3850 950
 	1    0    0    -1
@@
 F 0 "R13" V 4730 950 50  0000 C CNN
 F 1 "100" V 4650 950 50  0000 C CNN
-F 2 "RC03" H 4650 950 60  0001 C CNN
+F 2 "rc03_vert" H 4650 950 60  0001 C CNN
 	1    4650 950
 	1    0    0    -1
@@
 F 0 "R12" V 5530 950 50  0000 C CNN
 F 1 "100" V 5450 950 50  0000 C CNN
-F 2 "RC03" H 5450 950 60  0001 C CNN
+F 2 "rc03_vert" H 5450 950 60  0001 C CNN
 	1    5450 950
 	1    0    0    -1
@@
 F 0 "R11" V 6330 950 50  0000 C CNN
 F 1 "100" V 6250 950 50  0000 C CNN
-F 2 "RC03" H 6250 950 60  0001 C CNN
+F 2 "rc03_vert" H 6250 950 60  0001 C CNN
 	1    6250 950
 	1    0    0    -1
@@
 F 0 "R10" V 7130 950 50  0000 C CNN
 F 1 "100" V 7050 950 50  0000 C CNN
-F 2 "RC03" H 7050 950 60  0001 C CNN
+F 2 "rc03_vert" H 7050 950 60  0001 C CNN
 	1    7050 950
 	1    0    0    -1
@@
 F 0 "R9" V 7930 950 50  0000 C CNN
 F 1 "100" V 7850 950 50  0000 C CNN
-F 2 "RC03" H 7850 950 60  0001 C CNN
+F 2 "rc03_vert" H 7850 950 60  0001 C CNN
 	1    7850 950
 	1    0    0    -1
@@
 F 0 "R8" V 8730 950 50  0000 C CNN
 F 1 "100" V 8650 950 50  0000 C CNN
-F 2 "RC03" H 8650 950 60  0001 C CNN
+F 2 "rc03_vert" H 8650 950 60  0001 C CNN
 	1    8650 950
 	1    0    0    -1
@@
 F 0 "R7" V 9530 950 50  0000 C CNN
 F 1 "100" V 9450 950 50  0000 C CNN
-F 2 "RC03" H 9450 950 60  0001 C CNN
+F 2 "rc03_vert" H 9450 950 60  0001 C CNN
 	1    9450 950
 	1    0    0    -1
@@
 F 0 "R6" V 10330 950 50  0000 C CNN
 F 1 "100" V 10250 950 50  0000 C CNN
-F 2 "RC03" H 10250 950 60  0001 C CNN
+F 2 "rc03_vert" H 10250 950 60  0001 C CNN
 	1    10250 950
 	1    0    0    -1
@@
 F 0 "R5" V 11130 950 50  0000 C CNN
 F 1 "100" V 11050 950 50  0000 C CNN
-F 2 "RC03" H 11050 950 60  0001 C CNN
+F 2 "rc03_vert" H 11050 950 60  0001 C CNN
 	1    11050 950
 	1    0    0    -1
@@
 F 0 "R4" V 11930 950 50  0000 C CNN
 F 1 "100" V 11850 950 50  0000 C CNN
-F 2 "RC03" H 11850 950 60  0001 C CNN
+F 2 "rc03_vert" H 11850 950 60  0001 C CNN
 	1    11850 950
 	1    0    0    -1
@@
 F 0 "R3" V 12730 950 50  0000 C CNN
 F 1 "100" V 12650 950 50  0000 C CNN
-F 2 "RC03" H 12650 950 60  0001 C CNN
+F 2 "rc03_vert" H 12650 950 60  0001 C CNN
 	1    12650 950
 	1    0    0    -1
@@
 F 0 "R2" V 13530 950 50  0000 C CNN
 F 1 "100" V 13450 950 50  0000 C CNN
-F 2 "RC03" H 13450 950 60  0001 C CNN
+F 2 "rc03_vert" H 13450 950 60  0001 C CNN
 	1    13450 950
 	1    0    0    -1
@@
 F 0 "R1" V 14330 950 50  0000 C CNN
 F 1 "100" V 14250 950 50  0000 C CNN
-F 2 "RC03" H 14250 950 60  0001 C CNN
+F 2 "rc03_vert" H 14250 950 60  0001 C CNN
 	1    14250 950
 	1    0    0    -1
