File: KiCad/C3Jr_v2/c3jr_v2-mech.sch (KiCad schematic (older format))
At the start: 4 parts

Commit message: C3jr_v2-Added extra buttons for rear side. Some track clean up. Added OSHW and WyoLum Logos. Final for Production.
Parts:
- FM1: footprint (none) -> Frame
Changed lines of the file:
@@
-EESchema Schematic File Version 2  date Sunday 18 December 2011 08:43:59 PM IST
+EESchema Schematic File Version 2  date 1/5/2012 2:50:43 PM
 LIBS:C3Jr_v2
 LIBS:power
@@
 F 0 "FM1" H 6350 1950 60  0000 C CNN
 F 1 "FRAME" H 6350 2250 60  0000 C CNN
+F 2 "Frame" H 6350 2100 60  0001 C CNN
 	1    6350 2100
 	1    0    0    -1
