File: KiCad/i2sd_v3/i2sd_v3.sch (KiCad schematic (older format))
At the start: 57 parts, among them IC1 ATMEGA8-AI, P1 I/O, P10 CD2, P11 CD2, P12 CD1, P13 CD1, P2 COMM_R, P3 BootDrive, P4 CONN_6, P5 CONN_6, P6 CONN_2, P8 FTDI, P9 ISP, SW1 SW_PUSH, U1 MCP1700T-3302E/TT, U2 74HC125, U3 MIC5219-5.0BM5, X1 CRYSTAL_2

Commit message: i2sd_v3 : legend clean up, DRC. PDF files added - SCH and PCB
Parts:
- C1, C2, C8: footprint c_0805 -> CP_5x11mm
- C10, C3, C4, C7: footprint c_0805 -> C2
- C11: footprint c_0805 -> cnp_3mm_disc
- C6: footprint C_ELCO_SMD -> C2
- D1, D2: footprint d_0805 -> led_5mm_clear
- P1: footprint I/O -> pin_strip_8
- P10, P11: footprint Sck-04-F-SMT -> vite_4mm
- P13: footprint Sck-04-F-SMT -> pin_strip_3x2
- P8: footprint pin_strip_6-90 -> vite_4mm
- P9: footprint ISP -> vite_4mm
- R1, R2, R3, R4, R5, R6, R7, R8: footprint r_0805 -> rc03_vert_LED
- SW1: footprint SW_SMD -> SW_PB_V
- U1: footprint SOT23-3 -> dil_16-300_socket
- U2: footprint SO14E -> TO-220_Horizontal
- U3: footprint SOT23-5 -> dil_28-300_socket
- X1: footprint Xtal_SMD2 -> XTAL
Changed lines of the file:
@@
-EESchema Schematic File Version 2  date Sunday 19 February 2012 12:02:41 AM IST
+EESchema Schematic File Version 2  date 2/20/2012 3:18:37 PM
 LIBS:i2sd_v3
 LIBS:power
@@
 F 0 "X1" V 950 3300 60  0000 C CNN
 F 1 "CRYSTAL_2" V 850 3450 60  0000 C CNN
-F 2 "Xtal_SMD2" H 900 3050 60  0001 C CNN
+F 2 "XTAL" H 900 3050 60  0001 C CNN
 	1    900  3050
 	0    1    1    0
@@
 F 0 "C11" H 725 3225 50  0000 L CNN
 F 1 "22p" H 725 3425 50  0000 L CNN
-F 2 "c_0805" H 700 3325 60  0001 C CNN
+F 2 "cnp_3mm_disc" H 700 3325 60  0001 C CNN
 F 4 "490-1734-1-ND" H 700 3525 60  0001 C CNN "Digikey"
 	1    700  3325
@@
 F 0 "C10" H 725 2875 50  0000 L CNN
 F 1 "22p" H 725 2675 50  0000 L CNN
-F 2 "c_0805" H 700 2775 60  0001 C CNN
+F 2 "C2" H 700 2775 60  0001 C CNN
 F 4 "490-1734-1-ND" H 700 2975 60  0001 C CNN "Digikey"
 	1    700  2775
@@
 F 0 "P1" H 6630 7000 40  0000 L CNN
 F 1 "I/O" H 6550 7055 30  0001 C CNN
-F 2 "I/O" H 6550 7000 60  0001 C CNN
+F 2 "pin_strip_8" H 6550 7000 60  0001 C CNN
 	1    6550 7000
 	1    0    0    -1
@@
 F 0 "C4" H 9375 1300 50  0000 L CNN
 F 1 "100n" H 9375 1150 50  0000 L CNN
-F 2 "c_0805" H 9350 1225 60  0001 C CNN
+F 2 "C2" H 9350 1225 60  0001 C CNN
 	1    9350 1225
 	1    0    0    -1
@@
 F 0 "U3" H 9875 650 60  0000 C CNN
 F 1 "MIC5219-5.0BM5" H 9875 1150 60  0000 C CNN
-F 2 "SOT23-5" H 9875 850 60  0001 C CNN
+F 2 "dil_28-300_socket" H 9875 850 60  0001 C CNN
 	1    9875 850
 	-1   0    0    -1
@@
 F 0 "C8" H 10550 1225 50  0000 L CNN
 F 1 "100n" H 10450 1075 50  0000 L CNN
-F 2 "c_0805" H 10650 1150 60  0001 C CNN
+F 2 "CP_5x11mm" H 10650 1150 60  0001 C CNN
 	1    10650 1150
 	1    0    0    -1
@@
 F 0 "C3" H 8775 1150 50  0000 L CNN
 F 1 "2u2 Tant" H 8875 900 50  0000 L CNN
-F 2 "c_0805" H 8875 1050 60  0001 C CNN
+F 2 "C2" H 8875 1050 60  0001 C CNN
 	1    8875 1050
 	1    0    0    -1
@@
 F 0 "P11" V 10625 5000 50  0000 C CNN
 F 1 "CD2" V 10725 5000 50  0000 C CNN
-F 2 "Sck-04-F-SMT" H 10675 5000 60  0001 C CNN
+F 2 "vite_4mm" H 10675 5000 60  0001 C CNN
 	1    10675 5000
 	1    0    0    1
@@
 F 0 "P13" V 9800 5450 50  0000 C CNN
 F 1 "CD1" V 9900 5450 50  0000 C CNN
-F 2 "Sck-04-F-SMT" H 9850 5450 60  0001 C CNN
+F 2 "pin_strip_3x2" H 9850 5450 60  0001 C CNN
 	1    9850 5450
 	1    0    0    1
@@
 F 0 "P10" V 9800 5000 50  0000 C CNN
 F 1 "CD2" V 9900 5000 50  0000 C CNN
-F 2 "Sck-04-F-SMT" H 9850 5000 60  0001 C CNN
+F 2 "vite_4mm" H 9850 5000 60  0001 C CNN
 	1    9850 5000
 	1    0    0    1
@@
 F 0 "R8" V 5330 6750 50  0000 C CNN
 F 1 "470E" V 5250 6750 50  0000 C CNN
-F 2 "r_0805" H 5250 6750 60  0001 C CNN
+F 2 "rc03_vert_LED" H 5250 6750 60  0001 C CNN
 	1    5250 6750
 	1    0    0    -1
@@
 F 0 "R5" V 5030 6750 50  0000 C CNN
 F 1 "470E" V 4950 6750 50  0000 C CNN
-F 2 "r_0805" H 4950 6750 60  0001 C CNN
+F 2 "rc03_vert_LED" H 4950 6750 60  0001 C CNN
 	1    4950 6750
 	1    0    0    -1
@@
 F 0 "D2" H 5250 7350 50  0000 C CNN
 F 1 "LED" H 5250 7150 50  0000 C CNN
-F 2 "d_0805" H 5250 7250 60  0001 C CNN
+F 2 "led_5mm_clear" H 5250 7250 60  0001 C CNN
 	1    5250 7250
 	0    1    1    0
@@
 F 0 "D1" H 4950 7350 50  0000 C CNN
 F 1 "LED" H 4950 7150 50  0000 C CNN
-F 2 "d_0805" H 4950 7250 60  0001 C CNN
+F 2 "led_5mm_clear" H 4950 7250 60  0001 C CNN
 	1    4950 7250
 	0    1    1    0
@@
 F 0 "P9" V 1450 7050 60  0000 C CNN
 F 1 "ISP" V 1550 7050 60  0000 C CNN
-F 2 "ISP" H 1500 7050 60  0001 C CNN
+F 2 "vite_4mm" H 1500 7050 60  0001 C CNN
 	1    1500 7050
 	1    0    0    -1
@@
 F 0 "C7" V 2500 6875 50  0000 L CNN
 F 1 "100n" V 2500 6575 50  0000 L CNN
-F 2 "c_0805" H 2600 6750 60  0001 C CNN
+F 2 "C2" H 2600 6750 60  0001 C CNN
 	1    2600 6750
 	0    1    1    0
@@
 F 0 "P8" V 3200 7050 60  0000 C CNN
 F 1 "FTDI" V 3300 7050 60  0000 C CNN
-F 2 "pin_strip_6-90" H 3250 7050 60  0001 C CNN
+F 2 "vite_4mm" H 3250 7050 60  0001 C CNN
 	1    3250 7050
 	1    0    0    1
@@
 F 0 "C6" H 10825 1200 50  0000 L CNN
 F 1 "47u,10V" V 10950 825 50  0000 L CNN
-F 2 "C_ELCO_SMD" H 10925 1100 60  0001 C CNN
+F 2 "C2" H 10925 1100 60  0001 C CNN
 	1    10925 1100
 	1    0    0    -1
@@
 F 0 "U2" H 6300 4400 50  0000 L BNN
 F 1 "74HC125" H 6350 4150 40  0000 L TNN
-F 2 "SO14E" H 6300 4300 60  0001 C CNN
+F 2 "TO-220_Horizontal" H 6300 4300 60  0001 C CNN
 	4    6300 4300
 	-1   0    0    -1
@@
 F 0 "U2" H 6300 2200 50  0000 L BNN
 F 1 "74HC125" H 6350 1950 40  0000 L TNN
-F 2 "SO14E" H 6300 2100 60  0001 C CNN
+F 2 "TO-220_Horizontal" H 6300 2100 60  0001 C CNN
 	1    6300 2100
 	1    0    0    -1
@@
 F 0 "U2" H 6300 3400 50  0000 L BNN
 F 1 "74HC125" H 6350 3150 40  0000 L TNN
-F 2 "SO14E" H 6300 3300 60  0001 C CNN
+F 2 "TO-220_Horizontal" H 6300 3300 60  0001 C CNN
 	3    6300 3300
 	1    0    0    -1
@@
 F 0 "U2" H 6300 2800 50  0000 L BNN
 F 1 "74HC125" H 6350 2550 40  0000 L TNN
-F 2 "SO14E" H 6300 2700 60  0001 C CNN
+F 2 "TO-220_Horizontal" H 6300 2700 60  0001 C CNN
 	2    6300 2700
 	1    0    0    -1
@@
 F 0 "U1" H 9750 2250 60  0000 C CNN
 F 1 "MCP1700T-3302E/TT" H 9950 2650 60  0000 C CNN
-F 2 "SOT23-3" H 9950 2400 60  0001 C CNN
+F 2 "dil_16-300_socket" H 9950 2400 60  0001 C CNN
 	1    9950 2400
 	-1   0    0    -1
@@
 F 0 "R2" V 5080 1450 50  0000 C CNN
 F 1 "10k" V 5000 1450 50  0000 C CNN
-F 2 "r_0805" H 5000 1450 60  0001 C CNN
+F 2 "rc03_vert_LED" H 5000 1450 60  0001 C CNN
 	1    5000 1450
 	1    0    0    -1
@@
 F 0 "R1" V 4875 1450 50  0000 C CNN
 F 1 "10k" V 4800 1450 50  0000 C CNN
-F 2 "r_0805" H 4800 1450 60  0001 C CNN
+F 2 "rc03_vert_LED" H 4800 1450 60  0001 C CNN
 	1    4800 1450
 	1    0    0    -1
@@
 F 0 "SW1" H 1225 5310 50  0000 C CNN
 F 1 "SW_PUSH" H 1075 5120 50  0000 C CNN
-F 2 "SW_SMD" H 1075 5200 60  0001 C CNN
+F 2 "SW_PB_V" H 1075 5200 60  0001 C CNN
 F 4 "" H 1325 5410 60  0001 C CNN "DigiKey"
 	1    1075 5200
@@
 F 0 "R7" H 1125 1900 50  0000 C CNN
 F 1 "10k" V 1075 1700 50  0000 C CNN
-F 2 "r_0805" H 1075 1700 60  0001 C CNN
+F 2 "rc03_vert_LED" H 1075 1700 60  0001 C CNN
 	1    1075 1700
 	1    0    0    -1
@@
 F 0 "C1" H 1300 1325 50  0000 L CNN
 F 1 "100n" H 1300 1125 50  0000 L CNN
-F 2 "c_0805" H 1250 1225 60  0001 C CNN
+F 2 "CP_5x11mm" H 1250 1225 60  0001 C CNN
 	1    1250 1225
 	1    0    0    -1
@@
 F 0 "R3" V 5280 1450 50  0000 C CNN
 F 1 "10k" V 5200 1450 50  0000 C CNN
-F 2 "r_0805" H 5200 1450 60  0001 C CNN
+F 2 "rc03_vert_LED" H 5200 1450 60  0001 C CNN
 	1    5200 1450
 	1    0    0    -1
@@
 F 0 "R4" V 5480 1450 50  0000 C CNN
 F 1 "10k" V 5400 1450 50  0000 C CNN
-F 2 "r_0805" H 5400 1450 60  0001 C CNN
+F 2 "rc03_vert_LED" H 5400 1450 60  0001 C CNN
 	1    5400 1450
 	1    0    0    -1
@@
 F 0 "R6" V 5680 1450 50  0000 C CNN
 F 1 "10k" V 5600 1450 50  0000 C CNN
-F 2 "r_0805" H 5600 1450 60  0001 C CNN
+F 2 "rc03_vert_LED" H 5600 1450 60  0001 C CNN
 	1    5600 1450
 	1    0    0    -1
@@
 F 0 "C2" H 10650 2700 50  0000 L CNN
 F 1 "1u" H 10650 2500 50  0000 L CNN
-F 2 "c_0805" H 10600 2600 60  0001 C CNN
+F 2 "CP_5x11mm" H 10600 2600 60  0001 C CNN
 	1    10600 2600
 	1    0    0    -1
