File: KiCad/Gemini_v1/Gemini_Host.sch (KiCad schematic (older format))
At the start: 42 parts

Commit message: added Uno for Target and i2gps for Host.
Parts:
- removed B? (x12): I/O, I/O, symbol I/O
- removed B? (x4): I/O, I/O_ADR, symbol I/O
- removed C? (x2): 1u, c_0805, symbol C
- removed C? (x3): 100n, c_0805, symbol C
- removed C?: 47u,10V, C_ELCO_SMD, symbol C_POL
- removed C?: 2u2 Tant, c_0805, symbol C_POL
- removed C? (x2): 22p, c_0805, symbol C
- removed P?: CONN_2, pin_strip_2, symbol CONN_2
- removed R? (x6): 10k, r_0805, symbol R
- removed SD?: SD_CARD_MICRO, SD_Micro, symbol SD_CARD_MICRO
- removed SW?: SW_PUSH, SW_SMD, symbol SW_PUSH
- removed U?: ATMEGA8-AI, TQFP32, symbol ATMEGA8-AI
- removed U?: MCP1700T-3302E/TT, SOT23-3, symbol MCP_1700
- removed U? (x4): 74HC125, SO14E, symbol 74LS125
- removed U?: MIC5219-5.0BM5, SOT23-5, symbol MIC5219-5.0
- removed X?: CRYSTAL_2, Xtal_SMD2, symbol CRYSTAL_2
- added B1, B12, B13, B14, B18, B19, B4, B5, B6, B7, B8, B9, P1: I/O, I/O, symbol I/O
- added B10, B11, B16, B17: I/O, I/O_ADR, symbol I/O
- added C1, C4, C7, C8: 100n, c_0805, symbol C
- added C10, C11: 22p, c_0805, symbol C
- added C2, C5: 1u, c_0805, symbol C
- added C3: 2u2 Tant, c_0805, symbol C_POL
- added C6: 47u,10V, C_ELCO_SMD, symbol C_POL
- added D1, D2: LED, d_0805, symbol LED
- added IC1: ATMEGA8-AI, TQFP32, symbol ATMEGA8-AI
- added P10, P11: CD2, Sck-04-F-SMT, symbol CONN_4
- added P12, P13: CD1, Sck-04-F-SMT, symbol CONN_4
- added P3: BootDrive, PIN_ARRAY-6X1, symbol CONN_6
- added P4, P5: CONN_6, PIN_ARRAY-6X1, symbol CONN_6
- added P6: CONN_2, pin_strip_2, symbol CONN_2
- added P7: GPS_UP501, PIN_ARRAY-6X1, symbol CONN_6
- added P8: FTDI, PIN_ARRAY-6X1, symbol CONN_6
- added P9: ISP, ISP, symbol ISP
- added PCB1: PCB, PCB, symbol PCB
- added R1, R2, R3, R4, R6, R7: 10k, r_0805, symbol R
- added R5, R8: 470E, r_0805, symbol R
- added SC1: SCREW, vite_3mm, symbol SCREW
- added SD1: SD_CARD_MICRO, SD_Micro, symbol SD_CARD_MICRO
- added SW1: SW_PUSH, SW_SMD, symbol SW_PUSH
- added U1: MCP1700T-3302E/TT, SOT23-3, symbol MCP_1700
- added U2: 74HC125, SO14E, symbol 74LS125
- added U3: MIC5219-5.0BM5, SOT23-5, symbol MIC5219-5.0
- added X1: CRYSTAL_2, Xtal_SMD2, symbol CRYSTAL_2
Connections:
- net labels added: 32k, BAT, RST
- wire segments 156 -> 226
- no-connect marks 7 -> 13
Other:
- note added: "Additional SMD headers for\nrtcBoB/ChronoDot compatibility"
- note added: "BUCKLER Interface"
- note added: "BootDrive Header"
- note added: "FTDI Header"
- note added: "GPS Breakout"
- note added: "INDICATORS"
- note added: "ISP/PROG Header"
- note added: "Mounting Hole"
