File: KiCad/Gemini_v1/Gemini_Target.sch (KiCad schematic (older format))
At the start: 0 parts

Commit message: added Uno for Target and i2gps for Host.
Parts:
- added C1: 0.1uF, SM0805, symbol C
- added C10, C6: 0.1uF, 0805, symbol C
- added C11: 0.01Uf, 0805, symbol C
- added C12, C8: 0.01uF, 0805, symbol C
- added C13, C14, C2, C3: 22pF, 0805, symbol C
- added C4: 47uF/25V, 1206, symbol CAPAPOL
- added C5: 1uF, 1206, symbol C
- added C7: 47uF/12V, 1206, symbol CAPAPOL
- added C9: 1uF/9V, 1206, symbol CAPAPOL
- added D1: DIODE, DO214AA, symbol DIODE
- added D2: CD1206-S01575, 1206, symbol DIODE
- added D3: LED YELLOW, 0805, symbol LED
- added D4: LED YELLOW (TX), 0805, symbol LED
- added D5: LED YELLOW (RX), 0805, symbol LED
- added D6: LED GREEN, 0805, symbol LED
- added D7: CD1206, 1206, symbol DIODE
- added F1: MF-MSMF050-2 500mA, symbol FUSE
- added IC1: ATMEGA16U2, symbol ATMEGA16U2
- added IC2: ATMEGA328-P, symbol ATMEGA328-P
- added J1: USB, symbol USB
- added J2: JACK_2P, symbol JACK_2P
- added JP1: JUMPER, symbol JUMPER
- added JP2: CONN_2X2, symbol CONN_2X2
- added L1: BLM21, symbol FERRITE
- added P1, P3: CONN_3X2, symbol CONN_3X2
- added P2, P6: CONN_8, symbol CONN_8
- added P4: CONN_10, symbol CONN_10
- added P5: CONN_6, symbol CONN_6
- added Q1: FDN340P, symbol FDN340P
- added R1, R16, R2, R6: 10K, 0805, symbol R
- added R10, R11, R12, R13, R14, R15, R8: 1K, 0805, symbol R
- added R17, R5: 1M, 0805, symbol R
- added R3, R4: 22E, 0805, symbol R
- added R7: 333E, 0805, symbol R
- added R9: 220E, 0805, symbol R
- added SW1: SW_PUSH, symbol SW_PUSH
- added U1: LM358, symbol LM358
- added U2: 7805, symbol 7805
- added U3: LM317_SOT223, symbol LM317_SOT223
- added VR1, VR2: CG0603MLC-05E, symbol VR
- added X1, X2: 16MHz, symbol CRYSTAL
Connections:
- new net: F1.1 (A), J1.1 (Vbus)
- new net: J1.2 (D-), R4.1, VR1.1 (A)
- new net: J1.3 (D+), R3.1, VR2.1 (A)
- new net: L1.1 (A), VR1.2 (B), VR2.2 (B)
- new net: IC1.30 (D-), R3.2
- new net: IC1.29 (D+), R4.2
- new net: C3.2, IC1.1 (XTAL1), R5.2, X1.1
- new net: D5.2 (K), IC1.10 ((INT5/AIN3)PD4)
- new net: D4.2 (K), IC1.11 ((XCK/AIN4/PCINT12)PD5)
- new net: C11.1, IC1.13 ((CTS/HWB/AINR/TO/INT7)PD7), R12.1
- new net: IC1.18 ((T1/PCINT4)PB4), JP2.1
- new net: IC1.19 ((PCINT5/PB5)PB5), JP2.3
- new net: C2.2, IC1.2 (XTAL2), R5.1, X1.2
- new net: IC1.20 ((PCINT6)PB6), JP2.2
- new net: IC1.21 ((PCINT7/OC0A/OC1C)PB7), JP2.4
- new net: D2.1 (A), IC1.24 (~RESET), P1.5, R6.2
- new net: C5.1, IC1.27 (VCAP)
- new net: IC1.8 ((RXD1/AIN1/INT2)PD2), R11.1
- new net: IC1.9 ((TXD1/INT3)PD3), R10.1
- new net: IC2.11 ((PCINT21/OC0B/T1)PD5), P6.6 (P6)
- new net: IC2.12 ((PCINT22/OC0A/AIN0)PD6), P6.7 (P7)
- new net: IC2.13 ((PCINT23/AIN1)PD7), P6.8 (P8)
- new net: IC2.14 ((PCINT0/CLKO/ICP1)PB0), P4.1 (P1)
- new net: IC2.15 ((PCINT1/OC1A)PB1), P4.2 (P2)
- new net: IC2.16 ((PCINT2/OC1B/~SS~)PB2), P4.3 (P3)
- new net: IC2.23 ((PCINT8/ADC0)PC0), P5.1
- new net: IC2.24 ((PCINT9/ADC1)PC1), P5.2
- new net: IC2.25 ((PCINT10/ADC2)PC2), P5.3
- new net: IC2.26 ((PCINT11/ADC3)PC3), P5.4
- new net: IC2.4 ((PCINT18/INT0)PD2), P6.3 (P3)
- new net: IC2.5 ((PCINT19/OC2B/INT1)PD3), P6.4 (P4)
- new net: IC2.6 ((PCINT20/XCK/T0)PD4), P6.5 (P5)
- new net: D5.1 (A), R14.1
- new net: D4.1 (A), R13.2
- new net: Q1.1 (G), U1.1
- new net: R1.1, R2.2, U1.3 (+)
- new net: R8.1, U1.6 (-), U1.7
- new net: D1.1 (A), J2.1
- new net: R7.1, R9.2, U3.1 (ADJ)
- new net: D3.1 (A), R8.2
- new net: D6.1 (A), R15.2
- new net +3V3: C9.1, P2.4 (P4), R9.1, U1.2 (-), U3.2 (OUT)
- new net +5V: C1.1, C10.1, C6.2, C7.1, C8.1, D2.2 (K), D7.2 (K), IC1.32 (AVCC), IC1.4 (VCC), IC2.20 (AVCC), IC2.7 (VCC), P1.2, P2.2 (P2), P2.5 (P5), P3.2, Q1.2 (S), R13.1, R14.2, R15.1, R16.1, R6.1, U1.8 (V+), U1.8 (V+), U2.VO, U3.3 (IN)
- new net AREF: C12.1, IC2.21 (AREF), P4.8 (P8)
- new net GND: C1.2, C10.2, C12.2, C13.1, C14.1, C2.1, C3.1, C4.2, C5.2, C6.1, C7.2, C8.2, C9.2, D3.2 (K), D6.2 (K), IC1.28 (UGND), IC1.3 (GND), IC2.22 (GND), IC2.8 (GND), J1.4 (GND), J1.5 (Shield_1), J1.6 (Shield_2), J2.2, J2.3, L1.2 (B), P1.6, P2.6 (P6), P2.7 (P7), P3.6, P4.7 (P7), R12.2, R2.1, R7.2, SW1.2, U1.4 (V-), U1.4 (V-), U2.GND
- new net MISO2: IC1.17 ((PDO/MISO/PCINT3)PB3), P1.1
- new net MOSI2: IC1.16 ((PDI/MOSI/PCINT2)PB2), P1.4
- new net OSC1: C13.2, IC2.9 ((PCINT6/XTAL1/TOSC1)PB6), R17.1, X2.2
- new net OSC2: C14.2, IC2.10 ((PCINT7/XTAL2/TOSC2)PB7), R17.2, X2.1
- new net PB3: IC2.17 ((PCINT3/OC2A/MOSI)PB3), P3.4, P4.4 (P4)
- new net PB4: IC2.18 ((PCINT4/MISO)PB4), P3.1, P4.5 (P5)
- new net PB5: IC2.19 ((PCINT5/SCK)PB5), P3.3, P4.6 (P6), U1.5 (+)
- new net RESET: C11.2, D7.1 (A), IC2.1 ((PCINT14/~RESET~)PC6), JP1.1, JP1.2, P2.3 (P3), P3.5, R16.2, SW1.1
- new net SCK2: IC1.15 ((SCLK/PCINT1)PB1), P1.3
- new net SCL: IC2.28 ((PCINT14/SCL/ADC5)PC5), P4.10 (P10), P5.6
- new net SDA: IC2.27 ((PCINT12/SDA/ADC4)PC4), P4.9 (P9), P5.5
- new net SERA: IC2.2 ((PCINT16/RXD)PD0), P6.1 (P1), R10.2
- new net SERB: IC2.3 ((PCINT17/TXD)PD1), P6.2 (P2), R11.2
- new net USBVCC: F1.2 (B), IC1.31 (UVCC), Q1.3 (D)
- new net VIN: C4.1, D1.2 (K), P2.8 (P8), R1.2, U2.VI
- no-connect marks 0 -> 10
Other:
- note added: "ICSP"
- note added: "License : CC BY-SA\nhttp://creativecommons.org/licenses/by-sa/3.0/\n\nBased on Arduino Uno R3 design from http://arduino.cc"
- note added: "POWER"
