File: KiCad/BatMon/BatMon_v1.sch (KiCad schematic (older format))
At the start: 39 parts, among them K1 BAT_MON, K2 LOAD, K3 FTDI, K4 ISP, P1 METER_H, P2 METER_L, P3 METER_H, P4 METER_L, P5 CONN_1, SW1 RST, U1 SSR, U2 7805, U3 ATMEGA328-P, U4 ULN2003, X1 16MHz

Commit message: BatMon - board layout
Parts:
- removed C10, C8, C9: 10n, C2, symbol C
- removed P5: CONN_1, symbol CONN_1
- added K5: OUTPUT, symbol CONN_3
- added U5: ATTINY85, DIL8, symbol ATTINY85
Connections:
- wire segments 175 -> 182
- no-connect marks 10 -> 11
Other:
- note removed: "INPUT"
- note removed: "OUTPUT"
- moved on the sheet: D1, D2, D3, K1, K2, P1, P2, R1, R2, R3, R4, R6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
