File: KiCad/BatMon/BatMon.sch (KiCad schematic (older format))
At the start: 33 parts, among them P43 CONN_1, Q17 2N5401, SW1 INC, SW12 INC, SW2 DEC, SW22 DEC, SW3 MODE, SW32 MODE, SW4 RST, SW42 RST, SW5 ENTER, SW52 ENTER, U3 ATMEGA8-P, X1 16MHz

Commit message: BatMon - initial schematic
Parts:
- removed P43: CONN_1, Pad01, symbol CONN_1
- removed Q17: 2N5401, to92_2N5401, symbol PNP
- removed R17, R18, R19, R23: 10k, RC03, symbol R
- removed R20, R21: 4k7, RC03, symbol R
- removed R24: 1k, RC03, symbol R
- removed R30: 100E, RC03, symbol R
- removed SP1: SPEAKER, Speaker, symbol SPEAKER
- removed SW1: INC, SW_PB_V, symbol SW_PUSH
- removed SW12: INC, SW-PB-MOD, symbol SW_PUSH
- removed SW2: DEC, SW_PB_V, symbol SW_PUSH
- removed SW22: DEC, SW-PB-MOD, symbol SW_PUSH
- removed SW3: MODE, SW_PB_V, symbol SW_PUSH
- removed SW32: MODE, SW-PB-MOD, symbol SW_PUSH
- removed SW42: RST, SW-PB-MOD, symbol SW_PUSH
- removed SW5: ENTER, SW_PB_V, symbol SW_PUSH
- removed SW52: ENTER, SW-PB-MOD, symbol SW_PUSH
- added D? (x2): DIODE_ZENER, symbol DIODE_ZENER
- added DP?: LED_4X7SEG, symbol LED_4X7SEG
- added K?: CONN_3, symbol CONN_3
- added P?: CONN_2, symbol CONN_2
- added R?: LDR, pin_strip_2, symbol R
- added R?: 10K, RC03, symbol R
- added U?: ULN2003, symbol ULN2003
- added U?: SSR, symbol SSR
- U3: value ATMEGA8-P -> ATMEGA328-P
Connections:
- net labels added: MOSI, OC1A, SCK, SS
- net labels removed: A0, A1, A2, A3, COL_DRIVER_ENABLE, DEC, ENTER, INC, LDR, MODE, OC1A-LE, SPEAKER
- wire segments 121 -> 129
- no-connect marks 0 -> 6
Other:
- note removed: "NOTE : Duplicate Switches\nto allow Vert. and \nHoriz. positions"
- moved on the sheet: D258, R25, R31, R32, R33, SW4

Commit message: BatMon schematic update
Parts:
- removed DP?: LED_4X7SEG, symbol LED_4X7SEG
- removed U?: ULN2003, symbol ULN2003
- added C4, C6, C7: 100n, C2, symbol C
- added C5: 100u, CP_5x11mm, symbol CP1
- added D4: PWR, led_5mm_blue, symbol LED
- added DP1: LED_4X7SEG, symbol LED_4X7SEG
- added K3: FTDI, pin_strip_6-90, symbol CONN_6
- added K4: ISP, pin_strip_3x2, symbol CONN_6
- added K5: OUTPUT, symbol CONN_3
- added P1, P3: METER_H, symbol CONN_7
- added P2, P4: METER_L, symbol CONN_7
- added R8: 1k, RC03, symbol R
- added U2: 7805, symbol 7805
- added U4: ULN2003, symbol ULN2003
- added U5: ATTINY85, DIL8, symbol ATTINY85
- D1, D2: renamed from D?; value DIODE_ZENER -> ZD_5V1
- K1: renamed from K?; value CONN_3 -> BAT_MON
- K2: renamed from P?; value CONN_2 -> LOAD
- R1: renamed from R31; value 10K -> 110k
- R2: renamed from R32; value LDR -> 40k
- R3: renamed from R?; value 10K -> 110k
- R4: renamed from R?; value LDR -> 40k
- R7: renamed from R33; value 680E -> 270E
- gave numbers to parts that had none: 1
- renumbered C11 to C1, C12 to C2, D258 to D3, R22 to R5, R25 to R6, SW4 to SW1
Connections:
- net labels added: LOAD, PB0, PB1, PD2, PD3, PD4, PD5, PD6, PD7, V_B, V_BAT, V_I, V_IGN, V_USB
- net labels removed: MOSI-SDI, OC1A, SCK-CLK
- wire segments 129 -> 182
- no-connect marks 6 -> 11
Other:
- note added: "FTDI"
- note added: "ISP"
- note added: "OPTIONAL - VOLTAGE DISPLAY"
- note added: "POWER SUPPLY"
- moved on the sheet: C1, C2, C3, D1, D2, D3, K1, K2, PCB1, R1, R2, R3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

Commit message: BatMon - board layout
Parts:
- removed K5: OUTPUT, symbol CONN_3
- removed U5: ATTINY85, DIL8, symbol ATTINY85
- added C10, C8, C9: 10n, C2, symbol C
- added P5: CONN_1, symbol CONN_1
Connections:
- net labels added: A, B, C, CC2, CC3, CC4, D, DP, E, F, G, d1, d2, d3, d4
- wire segments 182 -> 175
- no-connect marks 11 -> 10
Other:
- note added: "INPUT"
- note added: "OUTPUT"
- moved on the sheet: D1, D2, D3, K1, K2, P1, P2, R1, R2, R3, R4, R6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

Commit message: BatMon - board layout complete
Parts:
- added P10, P7, P8, P9: CONN_1, symbol CONN_1
- added P6: I2C, symbol CONN_4
Connections:
- net labels added: CC1, GND_M
- wire segments 175 -> 181
- no-connect marks 10 -> 8
Other:
- note added: "MOUNTING HOLES"
- moved on the sheet: C10, C5, C6, C7, C8, C9, D1, D2, D3, D4, K1, K2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

Commit message: BatMon - board modification
Parts:
- removed C1, C2: 22p, cnp_3mm_disc, symbol C
- removed R6: 1k, RC03, symbol R
- added K5: V_CUTOFF, symbol CONN_3X2
- added R10, R11: 53E, RC03, symbol R
- added R12: 3k1, RC03, symbol R
- added R9: 800E, RC03, symbol R
- R7: value 270E -> 150E
Connections:
- net labels added: HI, LOW, MID, V_CUTOFF
- net labels removed: DBG
- wire segments 181 -> 193
Other:
- note added: "3.10V (11.6V)"
- note added: "3.15V (11.8V)"
- note added: "3.20V (12.0V)"
- note added: "4V @15V"
- note added: "VOLTAGE CUTOFF SELECTOR"
- moved on the sheet: D3, K2, P7, P8, PCB1, R7, U1

Commit message: BatMon - board modification
Parts:
- added P11, P12: DIP_SW, symbol CONN_6
Connections:
- wire segments 193 -> 214
Other:
- note added: "3.10V(11.6V)"
- note added: "3.15V(11.8V)"
- note added: "3.20V(12.0V)"
- note removed: "3.10V (11.6V)"
- note removed: "3.15V (11.8V)"
- note removed: "3.20V (12.0V)"
- moved on the sheet: C10, D3, K2, P3, P4, P5, P7, P8, PCB1, R10, R11, R12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

Commit message: BatMon - libraries clean up. Added Zener across voltage regulator
Parts:
- removed R9: 800E, RC03, symbol R
- added D5: ZD_15V, d_0805, symbol DIODE_ZENER
- C10, C3, C4, C7, C9: footprint C2 -> c_0805
- C5: footprint CP_5x11mm -> c_0805
- C6: footprint C2 -> C_ELCO_SMD
- D1, D2: footprint (none) -> d_0805
- D3, D4: footprint led_5mm_blue -> d_VMD2
- P1: footprint (none) -> pin_array_13x2
- P10: footprint (none) -> JACK_ALIM
- P2: footprint (none) -> SIL-8
- P3: footprint (none) -> SIL-7
- P4, P5, P6: footprint (none) -> PIN_ARRAY-8X1
- P7, P8: footprint (none) -> PIN_ARRAY-6X1
- P9: footprint (none) -> ISP
- R1, R3, R5, R7, R8: footprint RC03 -> r_0805
- R10, R11: value 53E -> 1k5; footprint RC03 -> r_0805
- R12: value 3k1 -> 2k; footprint RC03 -> r_0805
- R2, R4: footprint pin_strip_2 -> r_0805
- SW1: footprint SW_PB_V -> SW_SMD
- U1: footprint (none) -> SOT23-5
- U2: footprint (none) -> SO14E
- U3: footprint dil_28-300_socket -> SOT223
- U4: footprint (none) -> DS3231
- X1: footprint XTAL -> Xtal_SMD2
Connections:
- net labels added: SSR
- wire segments 214 -> 215
Other:
- note added: "2.0V"
- note added: "3.5V"
- note added: "5.0V"
- note added: "5V"
- note removed: "3.10V(11.6V)"
- note removed: "3.15V(11.8V)"
- note removed: "3.20V(12.0V)"
- note removed: "4V @15V"

Commit message: BatMon - board modification
Parts:
- added K6: V_SEL, pin_strip_3, symbol CONN_3
- added SW2: RST, SW-PB-MOD, symbol SW_PUSH
- C10, C3, C4, C7, C9: footprint c_0805 -> C2
- C5: footprint c_0805 -> CP_5x11mm
- C6: footprint C_ELCO_SMD -> C2
- D1, D2: footprint d_0805 -> DO-35
- D3: footprint d_VMD2 -> led_5mm_clear
- D4: footprint d_VMD2 -> led_5mm_blue
- D5: footprint d_0805 -> DO-35_Vert
- DP1: footprint (none) -> LED_4x7Seg
- K1: footprint (none) -> bornier3
- K2: footprint (none) -> bornier2
- K3: footprint pin_strip_6-90 -> pin_strip_6
- K5: footprint (none) -> pin_strip_3x2
- P1: footprint pin_array_13x2 -> pin_strip_7
- P10: footprint JACK_ALIM -> vite_3mm
- P11, P12: footprint (none) -> pin_strip_6b
- P2: footprint SIL-8 -> pin_strip_7
- P3: footprint SIL-7 -> pin_strip_7
- P4: footprint PIN_ARRAY-8X1 -> pin_strip_7
- P5: footprint PIN_ARRAY-8X1 -> Pad01
- P6: footprint PIN_ARRAY-8X1 -> pin_strip_4
- P7, P8: footprint PIN_ARRAY-6X1 -> vite_3mm
- P9: footprint ISP -> vite_3mm
- R1, R2, R3, R4, R5, R7, R8: footprint r_0805 -> RC03
- R10, R11, R12: footprint r_0805 -> rc03_vert
- SW1: footprint SW_SMD -> SW_PB_V
- U1: footprint SOT23-5 -> DIP-8__300_ELL
- U2: footprint SO14E -> TO-220_Vertical
- U3: footprint SOT223 -> dil_28-300_socket
- U4: footprint DS3231 -> dil_16-300_socket
- X1: footprint Xtal_SMD2 -> XTAL
Connections:
- net labels added: V_REG
- wire segments 215 -> 228
- no-connect marks 8 -> 7
Other:
- note added: "Arduino breakout Pins\nUse Jumpers for \nMODE selection\nor as I/O pins\n"
- note added: "NOTE : \nSSR configuration (above) allows using either a \n8 pin device or a 6 pin device. \nA 6 pin device gets plugged in to pins 2,3,4 and 5,6,7 \nof the 8 pin DIP socket."
- moved on the sheet: C7, D4, P7, P8, PCB1, R8
