File: KiCad/BatMon/BatMon_v2.sch (KiCad schematic (older format))
At the start: 50 parts, among them K1 BAT_MON, K2 LOAD, K3 FTDI, K4 ISP, K5 V_CUTOFF, K6 V_SEL, P1 METER_H, P10 CONN_1, P11 DIP_SW, P12 DIP_SW, P2 METER_L, P3 METER_H, P4 METER_L, P5 CONN_1, P6 I2C, P7 CONN_1, P8 CONN_1, P9 CONN_1, SW1 RST, SW2 RST, U1 SSR, U2 7805, U3 ATMEGA328-P, U4 ULN2003, X1 16MHz

Commit message: BatMon - v2, revised board layout, moved some components around
Parts:
- removed DP1: LED_4X7SEG, LED_4x7Seg_2, symbol LED_4X7SEG
- added DP1: LTC4727JR, LED_4x7Seg_3, symbol LTC4727JR
- U4: footprint dil_16-300_socket -> SO16E
Connections:
- no-connect marks 7 -> 11
Changed lines of the file:
@@
-EESchema Schematic File Version 2  date 7/7/2012 2:35:45 PM
+EESchema Schematic File Version 2  date 7/7/2012 3:49:09 PM
 LIBS:BatMon
 LIBS:power
-LIBS:BatMon-cache
+LIBS:BatMon_v2-cache
 EELAYER 25  0
 EELAYER END
@@
 Sheet 1 1
 Title "BatMon - Car Battery Voltage Monitor"
-Date "11 jun 2012"
+Date "7 jul 2012"
 Rev "A"
 Comp "it's BatMon, not Bat Man"
@@
 Comment4 ""
 $EndDescr
+Wire Wire Line
+	9950 5600 10275 5600
+Wire Wire Line
+	10275 5600 10275 4775
+Wire Wire Line
+	9675 5125 10425 5125
+Wire Wire Line
+	9675 5125 9675 4775
+Wire Wire Line
+	10175 4775 10175 4975
+Wire Wire Line
+	10175 4975 8750 4975
+Wire Wire Line
+	9975 4775 9975 4825
+Wire Wire Line
+	9975 4825 8900 4825
+Wire Wire Line
+	9875 3225 9875 2950
+Wire Wire Line
+	9875 2950 8675 2950
+Wire Wire Line
+	8675 2950 8675 4200
+Wire Wire Line
+	9575 3225 9575 3025
+Wire Wire Line
+	9575 3025 8750 3025
 Connection ~ 10450 1500
 Wire Wire Line
@@
 	10550 1400 10650 1400
 Wire Wire Line
-	1250 2200 1250 2700
+	1250 2700 1250 2200
 Connection ~ 6225 5800
 Wire Wire Line
-	6225 5800 6225 6150
+	6225 6150 6225 5800
 Wire Wire Line
 	6225 6150 6125 6150
@@
 Connection ~ 7700 900
 Wire Wire Line
-	7700 900  7700 1050
+	7700 1050 7700 900
 Connection ~ 5100 3600
 Wire Wire Line
@@
 	8525 4400 7950 4400
 Wire Wire Line
-	8675 5050 9875 5050
-Wire Wire Line
-	8675 5050 8675 4200
-Wire Wire Line
 	8675 4200 7950 4200
 Wire Wire Line
-	9675 4775 9675 4900
-Wire Wire Line
-	9675 4900 8825 4900
-Wire Wire Line
-	8825 4900 8825 3900
+	8825 3900 8825 4900
 Wire Wire Line
 	8825 3900 7950 3900
@@
 	4475 6150 4475 2600
 Wire Wire Line
-	4475 5950 4425 5950
+	4425 5950 4475 5950
 Wire Wire Line
 	4475 6150 4425 6150
 Wire Wire Line
-	3250 6500 3525 6500
+	3525 6500 3250 6500
 Wire Wire Line
 	3525 6500 3525 6050
@@
 Connection ~ 3250 5950
 Wire Wire Line
-	3250 6475 3250 6525
+	3250 6525 3250 6475
 Wire Wire Line
 	3250 7575 3250 7650
@@
 	3350 2400 5700 2400
 Wire Wire Line
-	5700 2400 5700 1625
+	5700 1625 5700 2400
 Wire Wire Line
 	5700 1625 6275 1625
@@
 Wire Wire Line
 	3800 3100 3900 3100
-Wire Wire Line
-	10075 3225 10075 3025
-Wire Wire Line
-	9975 3175 10825 3175
-Wire Wire Line
-	9575 3225 9575 2950
 Connection ~ 6975 6675
 Wire Wire Line
-	6975 6675 6775 6675
+	6775 6675 6975 6675
 Wire Wire Line
 	6775 6675 6775 6550
 Wire Wire Line
-	6125 6300 6350 6300
+	6350 6300 6125 6300
 Wire Wire Line
 	6125 5800 6775 5800
@@
 Connection ~ 8350 900
 Wire Wire Line
-	9550 1000 9550 950
+	9550 950  9550 1000
 Wire Wire Line
 	9550 1500 9550 1550
@@
 	8000 900  8000 1050
 Wire Wire Line
-	8800 1200 8800 2100
-Wire Wire Line
-	9550 2100 9550 1950
-Wire Wire Line
-	8350 1050 8350 900
+	8800 2100 8800 1200
+Wire Wire Line
+	9550 1950 9550 2100
+Wire Wire Line
+	8350 900  8350 1050
 Wire Wire Line
 	9750 1050 9750 950
@@
 Connection ~ 8000 900
 Wire Wire Line
-	8400 900  7425 900
+	7425 900  8400 900
 Wire Notes Line
 	2000 6800 2925 6800
@@
 Connection ~ 1275 6950
 Wire Wire Line
-	1275 6950 1275 7050
+	1275 7050 1275 6950
 Wire Wire Line
 	1275 7050 1350 7050
@@
 	8650 5700 8450 5700
 Wire Wire Line
-	9950 5800 10925 5800
-Wire Wire Line
-	10925 5800 10925 3100
-Wire Wire Line
-	9875 3225 9875 3100
-Wire Wire Line
-	9950 5600 10075 5600
-Wire Wire Line
-	10075 5600 10075 4775
+	9950 5800 10425 5800
+Wire Wire Line
+	10425 5800 10425 5125
 Wire Wire Line
 	8825 3600 8825 3100
 Wire Wire Line
-	9775 3225 9775 3100
-Wire Wire Line
-	8900 3175 8900 3700
-Wire Wire Line
-	9875 5050 9875 4775
-Wire Wire Line
-	9975 4775 9975 5125
-Wire Wire Line
-	9675 3225 9675 3175
-Wire Wire Line
-	10075 3025 8750 3025
+	8900 3700 8900 3175
 Wire Wire Line
 	8750 3025 8750 3500
 Wire Wire Line
-	9975 3175 9975 3225
-Wire Wire Line
-	10825 3175 10825 5700
-Wire Wire Line
-	10825 5700 9950 5700
-Wire Wire Line
-	9575 2950 11025 2950
-Wire Wire Line
-	11025 2950 11025 5900
-Wire Wire Line
-	11025 5900 9950 5900
+	10350 5700 10350 5050
+Wire Wire Line
+	10350 5700 9950 5700
+Wire Wire Line
+	10500 5900 10500 5200
+Wire Wire Line
+	10500 5900 9950 5900
 Wire Wire Line
 	8375 5800 8650 5800
@@
 Connection ~ 6100 1625
 Wire Wire Line
-	6900 2275 6900 2175
-Wire Wire Line
-	6100 1575 6100 1675
+	6900 2175 6900 2275
+Wire Wire Line
+	6100 1675 6100 1575
 Wire Wire Line
 	3900 2900 3350 2900
@@
 	1050 3700 1050 3550
 Wire Wire Line
-	2650 1700 2650 1650
+	2650 1650 2650 1700
 Connection ~ 600  2400
 Wire Wire Line
-	650  2600 600  2600
+	600  2600 650  2600
 Wire Wire Line
 	600  2600 600  1650
@@
 	750  3300 700  3300
 Wire Wire Line
-	2350 2100 2350 1600
+	2350 1600 2350 2100
 Wire Wire Line
 	600  1650 750  1650
@@
 	2650 2100 2650 2150
 Wire Wire Line
-	600  2800 1450 2800
+	1450 2800 600  2800
 Wire Wire Line
 	1450 2700 1370 2700
@@
 	3350 3300 3500 3300
 Wire Wire Line
-	2650 1650 1250 1650
+	1250 1650 2650 1650
 Wire Wire Line
 	700  3300 700  3100
 Connection ~ 1250 2600
 Wire Wire Line
-	6900 1575 6900 1675
-Wire Wire Line
-	6100 2275 6100 2175
+	6900 1675 6900 1575
+Wire Wire Line
+	6100 2175 6100 2275
 Connection ~ 6900 1625
 Wire Wire Line
-	7075 1750 7075 1625
+	7075 1625 7075 1750
 Wire Wire Line
 	7075 1625 6525 1625
@@
 	11050 1200 11050 950
 Wire Wire Line
-	1350 6950 800  6950
+	800  6950 1350 6950
 Wire Wire Line
 	1350 7150 800  7150
@@
 Connection ~ 6675 1625
 Wire Wire Line
-	6975 6725 6975 5775
-Wire Wire Line
-	6775 5775 6775 6150
+	6975 5775 6975 6725
+Wire Wire Line
+	6775 6150 6775 5775
 Connection ~ 6775 5800
 Wire Notes Line
 	7300 5275 4600 5275
 Wire Wire Line
-	9675 3175 8900 3175
-Wire Wire Line
-	9875 3100 10925 3100
-Wire Wire Line
-	9775 3100 8825 3100
-Wire Wire Line
 	3900 3000 3700 3000
 Wire Wire Line
@@
 	10300 6550 10900 6550
 Wire Wire Line
-	700  5225 1050 5225
+	1050 5225 700  5225
 Wire Wire Line
 	875  5325 875  5225
@@
 	5200 6625 5200 6725
 Wire Wire Line
-	3250 7025 3250 7075
+	3250 7075 3250 7025
 Connection ~ 3250 6500
 Wire Wire Line
@@
 	3700 7050 3250 7050
 Wire Wire Line
-	4425 6050 4475 6050
+	4475 6050 4425 6050
 Connection ~ 4475 6050
 Wire Notes Line
@@
 	8900 3800 8900 4825
 Wire Wire Line
-	8900 4825 9575 4825
-Wire Wire Line
-	9575 4825 9575 4775
-Wire Wire Line
 	7950 4000 8750 4000
 Wire Wire Line
 	8750 4000 8750 4975
 Wire Wire Line
-	8750 4975 9775 4975
-Wire Wire Line
-	9775 4975 9775 4775
-Wire Wire Line
 	7950 4300 8600 4300
 Wire Wire Line
-	8600 4300 8600 5125
-Wire Wire Line
-	8600 5125 9975 5125
-Wire Wire Line
 	7950 4500 8450 4500
 Wire Wire Line
@@
 	8300 4700 8300 5900
 Wire Wire Line
-	5025 3500 5100 3500
-Wire Wire Line
-	5100 3500 5100 4850
+	5100 3500 5025 3500
+Wire Wire Line
+	5100 4850 5100 3500
 Wire Wire Line
 	5100 4600 5025 4600
@@
 Connection ~ 5100 3700
 Wire Wire Line
-	3250 5375 3250 5975
-Wire Wire Line
-	7700 1450 7700 2000
-Wire Wire Line
-	7700 2000 10000 2000
+	3250 5975 3250 5375
+Wire Wire Line
+	7700 2000 7700 1450
+Wire Wire Line
+	10000 2000 7700 2000
 Connection ~ 8000 2000
 Wire Wire Line
-	6350 6300 6350 5875
+	6350 5875 6350 6300
 Connection ~ 6350 5950
 Wire Wire Line
@@
 Wire Wire Line
 	10350 1350 10350 1250
+Wire Wire Line
+	8900 3175 9775 3175
+Wire Wire Line
+	9775 3175 9775 3225
+Wire Wire Line
+	8825 3100 10075 3100
+Wire Wire Line
+	10075 3100 10075 3225
+Wire Wire Line
+	8600 4300 8600 2875
+Wire Wire Line
+	8600 2875 9675 2875
+Wire Wire Line
+	9675 2875 9675 3225
+Wire Wire Line
+	8825 4900 9775 4900
+Wire Wire Line
+	9775 4900 9775 4775
+Wire Wire Line
+	9575 4775 9575 5200
+Wire Wire Line
+	9575 5200 10500 5200
+Wire Wire Line
+	10075 4775 10075 5050
+Wire Wire Line
+	10075 5050 10350 5050
+NoConn ~ 9875 4775
+NoConn ~ 10275 3225
+NoConn ~ 10175 3225
+NoConn ~ 9975 3225
+$Comp
+L LTC4727JR DP1
+U 1 1 4FF809B9
+P 9925 4025
+F 0 "DP1" H 9175 4575 60  0000 C CNN
+F 1 "LTC4727JR" H 9325 3525 60  0000 C CNN
+F 2 "LED_4x7Seg_3" H 9325 3625 60  0001 C CNN
+	1    9925 4025
+	1    0    0    -1
+$EndComp
 Text Label 10650 1400 0    40   ~ 0
 V_USB
@@
 Text Label 8125 3500 0    40   ~ 0
 B
-Text Label 10075 5375 0    40   ~ 0
+Text Label 10075 5600 0    40   ~ 0
 CC4
 Text Label 8125 4300 0    40   ~ 0
@@
 F 0 "U4" H 9300 6100 70  0000 C CNN
 F 1 "ULN2003" H 9300 5900 70  0000 C CNN
-F 2 "dil_16-300_socket" H 9300 6000 60  0001 C CNN
+F 2 "SO16E" H 9300 6000 60  0001 C CNN
 	1    9300 6000
 	1    0    0    -1
 $EndComp
-$Comp
-L LED_4X7SEG DP1
-U 1 1 4FC75ED5
-P 9825 4025
-F 0 "DP1" H 9075 4475 60  0000 C CNN
-F 1 "LED_4X7SEG" H 10400 3500 60  0000 C CNN
-F 2 "LED_4x7Seg_2" H 10400 3600 60  0001 C CNN
-F 3 "LDQ-N286RI" H 9825 4025 60  0001 C CNN
-F 4 "LDQ-N286RI" H 9825 4025 60  0001 C CNN "Field1"
-	1    9825 4025
-	1    0    0    -1
-$EndComp
