File: KiCad/aLaMode/aLaMode_pwr.sch (KiCad schematic (older format))
At the start: 20 parts, among them P10 V_IN, Q1 FDN340P, U1 LP2985-33DBVR, U3 NCP1117ST50T3G, U5 LM358N

Commit message: aLaMode - preliminary track layout complete
Parts:
- C3, C4: footprint c_0805 -> C2
- C5: footprint c_0805 -> CP_5x11mm
- C6: footprint C_ELCO_SMD -> C2
- D5: footprint (none) -> DO-35_Vert
- P10: footprint (none) -> vite_3mm
- PCB1: footprint (none) -> PCB
- R10, R11, R12: footprint (none) -> rc03_vert
- U1: footprint (none) -> DIP-8__300_ELL
- U3: footprint (none) -> dil_28-300_socket
Changed lines of the file:
@@
-EESchema Schematic File Version 2  date Monday 11 June 2012 11:32:55 PM IST
+EESchema Schematic File Version 2  date Tuesday 12 June 2012 11:26:21 PM IST
 LIBS:aLaMode
 LIBS:power
@@
 Sheet 2 4
 Title ""
-Date "11 jun 2012"
+Date "12 jun 2012"
 Rev ""
 Comp ""
@@
 F 0 "R12" V 8405 5975 50  0000 C CNN
 F 1 "1k" V 8325 5975 50  0000 C CNN
+F 2 "rc03_vert" H 8325 5975 60  0001 C CNN
 	1    8325 5975
 	1    0    0    -1
@@
 F 0 "U1" H 6800 4000 60  0000 C CNN
 F 1 "LP2985-33DBVR" H 7100 3900 60  0000 C CNN
+F 2 "DIP-8__300_ELL" H 7000 3600 60  0001 C CNN
 	1    7000 3600
 	1    0    0    -1
@@
 F 0 "R11" V 4480 5425 50  0000 C CNN
 F 1 "10k" V 4400 5425 50  0000 C CNN
+F 2 "rc03_vert" H 4400 5425 60  0001 C CNN
 	1    4400 5425
 	1    0    0    -1
@@
 F 0 "R10" V 4480 4825 50  0000 C CNN
 F 1 "10k" V 4400 4825 50  0000 C CNN
+F 2 "rc03_vert" H 4400 4825 60  0001 C CNN
 	1    4400 4825
 	1    0    0    -1
@@
 F 0 "U3" H 5175 2550 60  0000 C CNN
 F 1 "NCP1117ST50T3G" H 5325 2850 60  0000 C CNN
+F 2 "dil_28-300_socket" H 5325 2550 60  0001 C CNN
 	1    5325 2550
 	1    0    0    -1
@@
 F 0 "D5" H 4325 2500 40  0000 C CNN
 F 1 "DIODESCH" H 4325 2300 40  0000 C CNN
+F 2 "DO-35_Vert" H 4325 2400 60  0001 C CNN
 	1    4325 2400
 	1    0    0    -1
@@
 F 0 "C6" H 4900 2600 50  0000 L CNN
 F 1 "47u,10V" H 4800 2500 50  0000 L CNN
-F 2 "C_ELCO_SMD" H 4750 2700 60  0001 C CNN
+F 2 "C2" H 4750 2700 60  0001 C CNN
 	1    4750 2700
 	-1   0    0    -1
@@
 F 0 "C3" H 6050 2750 50  0000 L CNN
 F 1 "2u2 Tant" H 5800 2475 50  0000 L CNN
-F 2 "c_0805" H 6150 2650 60  0001 C CNN
+F 2 "C2" H 6150 2650 60  0001 C CNN
 	1    6150 2650
 	-1   0    0    -1
@@
 F 0 "C5" H 7725 3800 50  0000 L CNN
 F 1 "1u" H 7725 3600 50  0000 L CNN
-F 2 "c_0805" H 7675 3700 60  0001 C CNN
+F 2 "CP_5x11mm" H 7675 3700 60  0001 C CNN
 	1    7675 3700
 	-1   0    0    -1
@@
 F 0 "C4" H 5900 2900 50  0000 L CNN
 F 1 "100n" H 5900 2750 50  0000 L CNN
-F 2 "c_0805" H 5875 2825 60  0001 C CNN
+F 2 "C2" H 5875 2825 60  0001 C CNN
 	1    5875 2825
 	-1   0    0    -1
@@
 F 0 "P10" H 3650 2700 60  0000 C CNN
 F 1 "V_IN" H 3650 2250 60  0000 C CNN
+F 2 "vite_3mm" H 3650 2500 60  0001 C CNN
 	1    3650 2500
 	1    0    0    -1
@@
 F 0 "PCB1" H 10900 6550 60  0000 C CNN
 F 1 "PCB" H 10900 7150 60  0000 C CNN
+F 2 "PCB" H 10900 6850 60  0001 C CNN
 	1    10900 6850
 	1    0    0    -1

Commit message: aLaMode - some schematic and board changes based on email feedback
Parts:
- C3, C4: footprint C2 -> c_0805
- C5: footprint CP_5x11mm -> c_0805
- C6: footprint C2 -> C_ELCO_SMD
- D5: footprint DO-35_Vert -> d_0805
- D6: footprint (none) -> d_0805
- G1, G2: footprint (none) -> Logo-WL3
- G3, G4: footprint (none) -> OSHW_6mm
- P10: footprint vite_3mm -> JACK_ALIM
- Q1: footprint (none) -> SOT23-3
- R10, R11, R12: footprint rc03_vert -> r_0805
- U1: footprint DIP-8__300_ELL -> SOT23-5
- U3: footprint dil_28-300_socket -> SOT223
- U5: footprint (none) -> SO8E
Changed lines of the file:
@@
-EESchema Schematic File Version 2  date Tuesday 12 June 2012 11:26:21 PM IST
+EESchema Schematic File Version 2  date Wednesday 13 June 2012 10:25:36 PM IST
 LIBS:aLaMode
 LIBS:power
@@
 Sheet 2 4
 Title ""
-Date "12 jun 2012"
+Date "13 jun 2012"
 Rev ""
 Comp ""
@@
 F 0 "D6" H 8325 6575 50  0000 C CNN
 F 1 "LED" H 8325 6375 50  0000 C CNN
+F 2 "d_0805" H 8325 6475 60  0001 C CNN
 	1    8325 6475
 	0    1    1    0
@@
 F 0 "R12" V 8405 5975 50  0000 C CNN
 F 1 "1k" V 8325 5975 50  0000 C CNN
-F 2 "rc03_vert" H 8325 5975 60  0001 C CNN
+F 2 "r_0805" H 8325 5975 60  0001 C CNN
 	1    8325 5975
 	1    0    0    -1
@@
 F 0 "U5" H 7725 5425 60  0000 L CNN
 F 1 "LM358N" H 7725 4975 60  0000 L CNN
+F 2 "SO8E" H 7775 5225 60  0001 C CNN
 	2    7775 5225
 	1    0    0    -1
@@
 F 0 "U1" H 6800 4000 60  0000 C CNN
 F 1 "LP2985-33DBVR" H 7100 3900 60  0000 C CNN
-F 2 "DIP-8__300_ELL" H 7000 3600 60  0001 C CNN
+F 2 "SOT23-5" H 7000 3600 60  0001 C CNN
 	1    7000 3600
 	1    0    0    -1
@@
 F 0 "Q1" V 6425 5025 60  0000 R CNN
 F 1 "FDN340P" V 6525 5175 60  0000 R CNN
+F 2 "SOT23-3" H 6200 4975 60  0001 C CNN
 	1    6200 4975
 	0    -1   -1   0
@@
 F 0 "R11" V 4480 5425 50  0000 C CNN
 F 1 "10k" V 4400 5425 50  0000 C CNN
-F 2 "rc03_vert" H 4400 5425 60  0001 C CNN
+F 2 "r_0805" H 4400 5425 60  0001 C CNN
 	1    4400 5425
 	1    0    0    -1
@@
 F 0 "R10" V 4480 4825 50  0000 C CNN
 F 1 "10k" V 4400 4825 50  0000 C CNN
-F 2 "rc03_vert" H 4400 4825 60  0001 C CNN
+F 2 "r_0805" H 4400 4825 60  0001 C CNN
 	1    4400 4825
 	1    0    0    -1
@@
 F 0 "U5" H 5250 5425 60  0000 L CNN
 F 1 "LM358N" H 5250 4975 60  0000 L CNN
+F 2 "SO8E" H 5300 5225 60  0001 C CNN
 	1    5300 5225
 	1    0    0    -1
@@
 F 0 "U3" H 5175 2550 60  0000 C CNN
 F 1 "NCP1117ST50T3G" H 5325 2850 60  0000 C CNN
-F 2 "dil_28-300_socket" H 5325 2550 60  0001 C CNN
+F 2 "SOT223" H 5325 2550 60  0001 C CNN
 	1    5325 2550
 	1    0    0    -1
@@
 F 0 "D5" H 4325 2500 40  0000 C CNN
 F 1 "DIODESCH" H 4325 2300 40  0000 C CNN
-F 2 "DO-35_Vert" H 4325 2400 60  0001 C CNN
+F 2 "d_0805" H 4325 2400 60  0001 C CNN
 	1    4325 2400
 	1    0    0    -1
@@
 F 0 "C6" H 4900 2600 50  0000 L CNN
 F 1 "47u,10V" H 4800 2500 50  0000 L CNN
-F 2 "C2" H 4750 2700 60  0001 C CNN
+F 2 "C_ELCO_SMD" H 4750 2700 60  0001 C CNN
 	1    4750 2700
 	-1   0    0    -1
@@
 F 0 "C3" H 6050 2750 50  0000 L CNN
 F 1 "2u2 Tant" H 5800 2475 50  0000 L CNN
-F 2 "C2" H 6150 2650 60  0001 C CNN
+F 2 "c_0805" H 6150 2650 60  0001 C CNN
 	1    6150 2650
 	-1   0    0    -1
@@
 F 0 "C5" H 7725 3800 50  0000 L CNN
 F 1 "1u" H 7725 3600 50  0000 L CNN
-F 2 "CP_5x11mm" H 7675 3700 60  0001 C CNN
+F 2 "c_0805" H 7675 3700 60  0001 C CNN
 	1    7675 3700
 	-1   0    0    -1
@@
 F 0 "C4" H 5900 2900 50  0000 L CNN
 F 1 "100n" H 5900 2750 50  0000 L CNN
-F 2 "C2" H 5875 2825 60  0001 C CNN
+F 2 "c_0805" H 5875 2825 60  0001 C CNN
 	1    5875 2825
 	-1   0    0    -1
@@
 F 0 "P10" H 3650 2700 60  0000 C CNN
 F 1 "V_IN" H 3650 2250 60  0000 C CNN
-F 2 "vite_3mm" H 3650 2500 60  0001 C CNN
+F 2 "JACK_ALIM" H 3650 2500 60  0001 C CNN
 	1    3650 2500
 	1    0    0    -1
@@
 F 0 "G4" H 10900 5800 60  0000 C CNN
 F 1 "Logo_OH" H 10900 6400 60  0000 C CNN
+F 2 "OSHW_6mm" H 10900 6100 60  0001 C CNN
 	1    10900 6100
 	1    0    0    -1
@@
 F 0 "G3" H 10900 5100 60  0000 C CNN
 F 1 "Logo_OH" H 10900 5700 60  0000 C CNN
+F 2 "OSHW_6mm" H 10900 5400 60  0001 C CNN
 	1    10900 5400
 	1    0    0    -1
@@
 F 0 "G2" H 10900 4400 60  0000 C CNN
 F 1 "Logo_Wyolum" H 10900 5000 60  0000 C CNN
+F 2 "Logo-WL3" H 10900 4700 60  0001 C CNN
 	1    10900 4700
 	1    0    0    -1
@@
 F 0 "G1" H 10900 3700 60  0000 C CNN
 F 1 "Logo_Wyolum" H 10900 4300 60  0000 C CNN
+F 2 "Logo-WL3" H 10900 4000 60  0001 C CNN
 	1    10900 4000
 	1    0    0    -1

Commit message: aLaMode - track layout complete. Need to add USB Input circuit.
Parts:
- D6: footprint d_0805 -> led_0805
Changed lines of the file:
@@
-EESchema Schematic File Version 2  date Wednesday 13 June 2012 10:25:36 PM IST
+EESchema Schematic File Version 2  date 6/14/2012 6:53:41 PM
 LIBS:aLaMode
 LIBS:power
-LIBS:Conn-raspberry
 LIBS:aLaMode_v1-cache
 EELAYER 25  0
@@
 Sheet 2 4
 Title ""
-Date "13 jun 2012"
+Date "14 jun 2012"
 Rev ""
 Comp ""
@@
 F 0 "D6" H 8325 6575 50  0000 C CNN
 F 1 "LED" H 8325 6375 50  0000 C CNN
-F 2 "d_0805" H 8325 6475 60  0001 C CNN
+F 2 "led_0805" H 8325 6475 60  0001 C CNN
 	1    8325 6475
 	0    1    1    0

Commit message: aLaMode - added USB socket to schematic
Parts:
- added C15: 1n, c_0805, symbol C
- added D7: DIODE_TRANSIL, symbol DIODE_TRANSIL
- added P12: UUSB_B, symbol UUSB_B
- added U7: FUSE, symbol FUSE
- C6: value 47u,10V -> 100u,25V
Connections:
- net labels added: PWR_IN, USB_IN
- wire segments 60 -> 101
- no-connect marks 1 -> 4
Other:
- moved on the sheet: C2, C3, C4, C5, C6, D5, D6, P10, Q1, R10, R11, R12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

Commit message: aLaMode - added micro-USB B Power Input circuit.
Parts:
- added C16: 10n, c_0805, symbol C
- C5: value 1u -> 2u2
- D7: value DIODE_TRANSIL -> SMBJ5.0CA-TR; footprint (none) -> diode-DO214AA
- F1: renamed from U7; value FUSE -> miniSMDC100F; footprint (none) -> f_1812
- P12: footprint (none) -> USB_B_Micro
Connections:
- wire segments 101 -> 74
- no-connect marks 4 -> 3
Other:
- note added: "Bi-directional clamping\nDiode, 5V"
- note added: "Polyswitch resettable fuse\n1.1A Hold, 2.2A Trip 8V max."
- note added: "TE - 1981568-1\nor\nFCI - 10118193-0001LF"
- moved on the sheet: C15, C5, D7, P12, U1

Commit message: aLamode - track layout complete.
Other:
- note added: "If using Micro USB -B socket, \nDO NOT INSTALL :\nP10, D5, U3\nApply solder bridge between Pins 2 and 3 of U3\n\nIf using Barrel Socket,\nDO NOT INSTALL :\nP12, F1, D7, C15"
Changed lines of the file:
@@
-EESchema Schematic File Version 2  date 6/15/2012 5:59:12 PM
+EESchema Schematic File Version 2  date Friday 15 June 2012 09:02:44 PM IST
 LIBS:aLaMode
 LIBS:power
@@
 Comment4 ""
 $EndDescr
+Text Notes 5400 1200 0    60   ~ 12
+If using Micro USB -B socket, \nDO NOT INSTALL :\nP10, D5, U3\nApply solder bridge between Pins 2 and 3 of U3\n\nIf using Barrel Socket,\nDO NOT INSTALL :\nP12, F1, D7, C15
 Connection ~ 6525 5350
 Wire Wire Line
