File: KiCad/uControl/uControl_rtc.sch (KiCad schematic (older format))
At the start: 7 parts, among them U5 DS3231N

Commit message: uControl Board layout work in progress
Parts:
- BT1: footprint CR1632_2 -> CR2032
Changed lines of the file:
@@
-EESchema Schematic File Version 2  date 12/27/2012 6:53:46 PM
+EESchema Schematic File Version 2  date Thursday 27 December 2012 10:04:40 PM IST
 LIBS:uControl
 LIBS:Conn-raspberry
@@
 F 0 "BT1" H 3650 2600 50  0000 C CNN
 F 1 "BATT_RTC" H 3950 2610 50  0000 C CNN
-F 2 "CR1632_2" H 3950 2800 60  0001 C CNN
+F 2 "CR2032" H 3950 2800 60  0001 C CNN
 	1    3950 2800
 	0    1    1    0

Commit message: uControl changed to Thru Hole design. Basic parts laid out. No tracks yet.
Parts:
- C23: footprint c_0805 -> C2
- R11: footprint r_0805 -> rc03_vert
Changed lines of the file:
@@
-EESchema Schematic File Version 2  date Thursday 27 December 2012 10:04:40 PM IST
+EESchema Schematic File Version 2  date 12/28/2012 6:29:01 PM
 LIBS:uControl
 LIBS:Conn-raspberry
@@
 Sheet 4 5
 Title "uControl"
-Date "27 dec 2012"
+Date "28 dec 2012"
 Rev "1"
 Comp "WyoLum"
@@
 F 0 "R11" H 7225 2150 50  0000 C CNN
 F 1 "10k" V 7150 2000 50  0000 C CNN
-F 2 "r_0805" H 7150 2000 60  0001 C CNN
+F 2 "rc03_vert" H 7150 2000 60  0001 C CNN
 	1    7150 2000
 	1    0    0    -1
 $EndComp
 $Comp
-L +BATT #PWR021
+L +BATT #PWR18
 U 1 1 4EC101F0
 P 5300 1850
-F 0 "#PWR021" H 5300 1800 20  0001 C CNN
+F 0 "#PWR18" H 5300 1800 20  0001 C CNN
 F 1 "+BATT" H 5300 1950 30  0000 C CNN
 	1    5300 1850
@@
 F 0 "C23" H 4175 2850 50  0000 L CNN
 F 1 "100n" V 4225 2525 50  0000 L CNN
-F 2 "c_0805" H 4175 2775 60  0001 C CNN
+F 2 "C2" H 4175 2775 60  0001 C CNN
 	1    4175 2775
 	1    0    0    -1
