File: KiCad/RasPi_Epoch/RasPi_RTC_th.sch (KiCad schematic (older format))
At the start: 20 parts, among them P1 RasPi_GPIO, P2 CONN_1, P3 CONN_1, P4 CONN_1, P5 32k, P6 CONN_1, P7 CONN_1, P8 CONN_1, P9 SQW, U1 DS3231N, U2 DS1307, X1 CRYSTAL

Commit message: RasPi_EPOCH - Modified. DS1307 connected to 5V0. All pull up resistors connected to 3V3. Added filter cap for 3V3.
Parts:
- added C1: 100n, cnp_3mm_disc, symbol C
Connections:
- wire segments 75 -> 78
Other:
- note added: "DS1307 (Optional)\nVcc is tied to 5V0 on Ras-Pi, but SCL and SDA are pulled up to 3V3.\nNeed to verify if this works."
- moved on the sheet: C4, C5, P5, P6, P7, P8, P9, R2, R3, U2, X1
