File: KiCad/OHSBadge/repaper.sch (KiCad schematic (older format))
At the start: 62 parts, among them J1 HEADER1X10MS2.54, J2 HEADER1X10MS2.54, J3 HEADER2X10MS2.54, J4 ZIF-40-0.5, Q1 AP2305, Q2 2N7002KW, Q3 BSS84W, Q4 2N7002KW, Q5 2N7002KW, Q6 2N7002KW, Q7 BSS84W, U1 S-5813A/S-5814A, U3 TPS77030, U4 TXS0108

Commit message: OHSBadge - need to assign repaper signals to Arduino shield pin outs.
Parts:
- removed R13, R14, R6, R7, R8: 0R, R0402, symbol R
- removed R32, R33: 0R, R0603, symbol R
- removed R34: 0R(NC), R0603, symbol R
Connections:
- net labels added: RST
- net labels removed: BUSY_MCU, EPD_CS_MCU, FLASH_CS, FLASH_CS_MCU, FLASH_SCLK, FLASH_SI, FLASH_SO, RESET_MCU, SPI_CLK_MCU, SPI_MISO_MCU, SPI_MOSI_MCU, VTCON
- wire segments 280 -> 260
- no-connect marks 14 -> 22
Other:
- note added: "SIGNALS TO BE CONNECTED TO MICRO\nLED1\nUART_RX\nUART_RX\nSW2\nBUSY\nPWM\n/RESET\n/FLASH_CS\nTEST/SBWTCK\nRST/SBWTDIO\nBORDER_CONTROL\nDISCHARGE\nPANEL_ON"

Commit message: OHSBadge - Controller to EPD pin connections assigned. Need to check 5V out from Digital Port 10
Parts:
- removed J3: HEADER2X10MS2.54, HEADER2X10MS2.54, symbol CON20C
Connections:
- net labels added: ENABLE_5V, FLASH_CS
- net labels removed: /FLASH_CS, PB0, PB1, PD2, PD3, PD4, PD5, PD6, PD7
- wire segments 260 -> 258
- no-connect marks 22 -> 35
Other:
- note removed: "SIGNALS TO BE CONNECTED TO MICRO\nLED1\nUART_RX\nUART_RX\nSW2\nBUSY\nPWM\n/RESET\n/FLASH_CS\nTEST/SBWTCK\nRST/SBWTDIO\nBORDER_CONTROL\nDISCHARGE\nPANEL_ON"
Changed lines of the file:
@@
-EESchema Schematic File Version 2  date 29-Mar-13 11:55:17 AM
+EESchema Schematic File Version 2  date 29-Mar-13 5:39:17 PM
 LIBS:power
 LIBS:repaper_sym
@@
 	1350 700  2450 700
 Wire Wire Line
-	2750 6125 3200 6125
-Wire Wire Line
-	2750 6175 3200 6175
-Wire Wire Line
-	1900 6525 2300 6525
+	2825 6125 3200 6125
+Wire Wire Line
+	2825 6175 3200 6175
+Wire Wire Line
+	1900 6525 2200 6525
 Wire Wire Line
 	9300 3300 9950 3300
@@
 	6250 4300 8350 4300
 Wire Wire Line
-	2750 6425 3200 6425
-Wire Wire Line
-	1900 6425 2300 6425
+	2825 6425 3200 6425
+Wire Wire Line
+	1900 6425 2200 6425
 Wire Wire Line
 	6250 850  10100 850
@@
 	6250 3200 7450 3200
 Wire Wire Line
-	2750 6475 3200 6475
+	2825 6475 3200 6475
 Wire Wire Line
 	6250 800  10100 800
@@
 	1800 1300 1800 1350
 Wire Wire Line
-	2750 6075 3200 6075
-Wire Wire Line
-	1900 6125 2300 6125
+	2825 6075 3200 6075
+Wire Wire Line
+	1900 6125 2200 6125
 Wire Wire Line
 	8500 3950 8500 4150
@@
 	1350 1250 1650 1250
 Wire Wire Line
-	2750 6525 3200 6525
+	2825 6525 3200 6525
 Wire Wire Line
 	6250 3550 6925 3550
 Wire Wire Line
-	1900 6475 2300 6475
+	1900 6475 2200 6475
 Wire Wire Line
 	6250 1100 10100 1100
 Wire Wire Line
-	2750 6275 3200 6275
-Wire Wire Line
-	1900 6375 2300 6375
+	2825 6275 3200 6275
+Wire Wire Line
+	1900 6375 2200 6375
 Wire Wire Line
 	6250 950  10100 950
 Wire Wire Line
-	2750 6375 3200 6375
+	2825 6375 3200 6375
 Wire Wire Line
 	6250 1050 10100 1050
 Wire Wire Line
-	2750 6325 3200 6325
+	2825 6325 3200 6325
 Wire Wire Line
 	6250 1000 10100 1000
 Wire Wire Line
-	1900 6275 2300 6275
+	1900 6275 2200 6275
 Wire Wire Line
 	2825 1850 3275 1850
@@
 	3275 1850 3275 1950
 Wire Wire Line
-	1900 6325 2300 6325
-Wire Wire Line
-	2750 6225 3200 6225
-Wire Wire Line
-	1900 6175 2300 6175
-Wire Wire Line
-	1900 6225 2300 6225
-Wire Wire Line
-	1900 6075 2300 6075
-Wire Wire Line
-	1900 6850 3200 6850
+	1900 6325 2200 6325
+Wire Wire Line
+	2825 6225 3200 6225
+Wire Wire Line
+	1900 6175 2200 6175
+Wire Wire Line
+	1900 6225 2200 6225
+Wire Wire Line
+	1900 6075 2275 6075
 Wire Wire Line
 	10100 2300 9650 2300
 Wire Wire Line
-	9650 2500 9650 2300
+	9650 2300 9650 2500
 Wire Wire Line
 	8700 2500 8700 2600
@@
 	8500 4350 8500 4450
 Wire Wire Line
-	6250 2500 9650 2500
+	9650 2500 6250 2500
 Wire Wire Line
 	3125 700  3125 1100
@@
 $EndComp
 $Comp
-L CON20C J3
-U 1 1 514F454B
-P 2450 6025
-F 0 "J3" H 2500 6000 27  0000 L TNN
-F 1 "HEADER2X10MS2.54" V 2550 5500 27  0000 L TNN
-F 2 "HEADER2X10MS2.54" H 2500 6075 27  0001 L TNN
-F 3 "" H 2450 6025 60  0001 C CNN
-	1    2450 6025
-	1    0    0    -1
-$EndComp
-$Comp
 L N_MOSFET_3 Q2
 U 1 1 514F454D
@@
 	0    1    -1   0
 $EndComp
-Text Label 2800 6125 0    24   ~ 0
+Text Label 2825 6125 0    24   ~ 0
 /EPD_CS
 Text Label 2025 5025 2    24   ~ 0
 /EPD_CS
-Text Label 2800 6175 0    24   ~ 0
-/FLASH_CS
+Text Label 2825 6175 0    24   ~ 0
+FLASH_CS
 Text Label 2025 5125 2    24   ~ 0
-/FLASH_CS
-Text Label 1950 6525 0    24   ~ 0
+FLASH_CS
+Text Label 2200 6525 2    24   ~ 0
 /RESET
 Text Label 2025 5325 2    24   ~ 0
@@
 Text Label 6250 4300 0    24   ~ 0
 BORDER_CONTROL
-Text Label 2800 6425 0    24   ~ 0
+Text Label 2825 6425 0    24   ~ 0
 BORDER_CONTROL
-Text Label 1950 6425 0    24   ~ 0
+Text Label 2200 6425 2    24   ~ 0
 BUSY
 Text Label 2025 5225 2    24   ~ 0
@@
 Text Label 6250 3200 0    24   ~ 0
 DISCHARGE
-Text Label 2800 6475 0    24   ~ 0
+Text Label 2825 6475 0    24   ~ 0
 DISCHARGE
 Text Label 3025 5025 0    24   ~ 0
@@
 Text Label 3025 5125 0    24   ~ 0
 FLASH_CS_COG
-Text Label 2800 6075 0    24   ~ 0
+Text Label 2825 6075 0    24   ~ 0
 GND
-Text Label 1950 6125 0    24   ~ 0
+Text Label 2200 6125 2    24   ~ 0
 LED1
 Text Label 1350 1250 0    24   ~ 0
 PANEL_ON
-Text Label 2800 6525 0    24   ~ 0
+Text Label 2825 6525 0    24   ~ 0
 PANEL_ON
 Text Label 6250 3550 0    24   ~ 0
 PWM
-Text Label 1950 6475 0    24   ~ 0
+Text Label 2200 6475 2    24   ~ 0
 PWM
 Text Label 3025 5325 0    24   ~ 0
 RESET_COG
-Text Label 2800 6275 0    24   ~ 0
+Text Label 2825 6275 0    24   ~ 0
 RST/SBWTDIO
-Text Label 1950 6375 0    24   ~ 0
+Text Label 2200 6375 2    24   ~ 0
 SPI_CLK
 Text Label 2025 4725 2    24   ~ 0
@@
 Text Label 3025 4725 0    24   ~ 0
 SPI_CLK_COG
-Text Label 2800 6375 0    24   ~ 0
+Text Label 2825 6375 0    24   ~ 0
 SPI_MISO
 Text Label 2025 4925 2    24   ~ 0
@@
 Text Label 3025 4925 0    24   ~ 0
 SPI_MISO_COG
-Text Label 2800 6325 0    24   ~ 0
+Text Label 2825 6325 0    24   ~ 0
 SPI_MOSI
 Text Label 2025 4825 2    24   ~ 0
@@
 Text Label 3025 4825 0    24   ~ 0
 SPI_MOSI_COG
-Text Label 1950 6275 0    24   ~ 0
+Text Label 2200 6275 2    24   ~ 0
 SW2
 Text Label 3025 1850 0    24   ~ 0
 TEMPERATURE
-Text Label 1950 6325 0    24   ~ 0
+Text Label 2200 6325 2    24   ~ 0
 TEMPERATURE
-Text Label 2800 6225 0    24   ~ 0
+Text Label 2825 6225 0    24   ~ 0
 TEST/SBWTCK
-Text Label 1950 6175 0    24   ~ 0
+Text Label 2200 6175 2    24   ~ 0
 UART_RX
-Text Label 1950 6225 0    24   ~ 0
+Text Label 2200 6225 2    24   ~ 0
 UART_TX
 Text Label 1600 700  0    24   ~ 0
 VCC3V
-Text Label 1950 6075 0    24   ~ 0
+Text Label 2200 6075 2    24   ~ 0
 5V0
 Text Label 9300 2600 0    24   ~ 0
@@
 Text Label 925  1850 0    24   ~ 0
 VCC3V
-Text Label 1900 6850 0    24   ~ 0
-VCC5V
 Text Label 7650 6400 0    24   ~ 0
 VCC5V
@@
 Wire Wire Line
 	4250 6225 4000 6225
-Connection ~ 4200 6425
-Wire Wire Line
-	4200 6425 4200 6525
-Wire Wire Line
-	4200 6525 4250 6525
 Wire Wire Line
 	4250 7225 4000 7225
@@
 Wire Wire Line
 	4250 7325 4000 7325
-Wire Wire Line
-	4200 6325 4200 6025
-Wire Wire Line
-	4200 6025 4250 6025
-Connection ~ 4200 6325
 Wire Wire Line
 	6150 5525 6400 5525
@@
 PC0
 Text Label 6400 6325 0    40   ~ 0
-PB1
+FLASH_CS
 Text Label 6400 6425 0    40   ~ 0
-PB0
+/EPD_CS
 Text Label 6400 6625 0    40   ~ 0
-PD7
+BUSY
 Text Label 6400 6725 0    40   ~ 0
-PD6
+/RESET
 Text Label 6400 6825 0    40   ~ 0
-PD5
+PWM
 Text Label 6400 6925 0    40   ~ 0
-PD4
+DISCHARGE
 Text Label 6400 7025 0    40   ~ 0
-PD3
+BORDER_CONTROL
 Text Label 6400 7125 0    40   ~ 0
-PD2
+PANEL_ON
 Text Label 6400 7325 0    40   ~ 0
 RXD
@@
 TXD
 Text Label 6400 6225 0    40   ~ 0
-/EPD_CS
+ENABLE_5V
 Text Label 6400 6125 0    40   ~ 0
 SPI_MOSI
@@
 Text Label 4000 7325 0    40   ~ 0
 SCL
-Text Label 4000 7225 0    40   ~ 0
-SDA
-Text Label 4000 6425 0    40   ~ 0
-GND
 Text Label 4000 6125 0    40   ~ 0
 RST
-Text Label 4000 6325 0    40   ~ 0
-5V0
 $Comp
 L ARDUINO_SHIELD SHIELD1
@@
 	10475 6975 10475 6950
 Connection ~ 9550 6975
-Text Label 3200 6850 2    24   ~ 0
-5V0
 Wire Notes Line
 	3700 1550 3700 2425
 Wire Notes Line
 	600  2425 600  1550
-Text Notes 700  7025 0    30   ~ 0
-SIGNALS TO BE CONNECTED TO MICRO\nLED1\nUART_RX\nUART_RX\nSW2\nBUSY\nPWM\n/RESET\n/FLASH_CS\nTEST/SBWTCK\nRST/SBWTDIO\nBORDER_CONTROL\nDISCHARGE\nPANEL_ON
 NoConn ~ 4000 6825
 NoConn ~ 4000 6925
 NoConn ~ 4000 7025
 NoConn ~ 4000 7125
-NoConn ~ 4000 7225
 NoConn ~ 4000 7325
 NoConn ~ 4000 6625
 NoConn ~ 4000 6225
+$Comp
+L VCC_CIRCLE #PWR7
+U 1 1 51557DCF
+P 2275 5975
+F 0 "#PWR7" V 2275 5975 27  0001 L TNN
+F 1 "VCC5V" H 2325 5975 27  0000 L TNN
+F 2 "" H 2275 5975 60  0001 C CNN
+F 3 "" H 2275 5975 60  0001 C CNN
+	1    2275 5975
+	1    0    0    -1
+$EndComp
+Wire Wire Line
+	2275 6075 2275 6050
+NoConn ~ 2825 6225
+NoConn ~ 2825 6275
+NoConn ~ 2200 6125
+NoConn ~ 2200 6175
+NoConn ~ 2200 6225
+NoConn ~ 2200 6275
+NoConn ~ 4000 6125
+NoConn ~ 4000 6325
+NoConn ~ 6400 7225
+NoConn ~ 6400 7325
+NoConn ~ 4000 7225
+Wire Wire Line
+	4250 6025 4000 6025
+NoConn ~ 4000 6025
+Wire Wire Line
+	4250 6525 4000 6525
+NoConn ~ 4000 6425
+NoConn ~ 4000 6525
 $EndSCHEMATC

Commit message: Changed Temp sensor, removed 20pin Header, all buckler connections made except 5V
Parts:
- removed R4: 26.7K/1%, R0603, symbol R
- removed R5: 17.8K/1%, R0603, symbol R
- removed U1: S-5813A/S-5814A, SNT-4A, symbol LM3940_19
- added U1: MCP9700AT-E/TT, ~, symbol MCP9700AT-E/TT
- C7: value 0.1uF,16V -> 1uF,10V; footprint C0402 -> C0805; Field4 0402/0.1uF/16V/Y -> 1u/10V/X7R
Connections:
- wire segments 258 -> 254
- no-connect marks 35 -> 34
Changed lines of the file:
@@
-EESchema Schematic File Version 2  date 29-Mar-13 5:39:17 PM
+EESchema Schematic File Version 2  date Friday 29 March 2013 10:51:09 PM IST
 LIBS:power
 LIBS:repaper_sym
@@
 $EndDescr
 Wire Wire Line
-	2450 1850 2575 1850
-Wire Wire Line
 	1350 700  2450 700
 Wire Wire Line
@@
 	8300 2700 8400 2700
 Wire Wire Line
-	3275 2250 3275 2200
-Wire Wire Line
-	1900 2000 1950 2000
-Wire Wire Line
 	3125 1350 3125 1275
 Wire Wire Line
@@
 	1900 6275 2200 6275
 Wire Wire Line
-	2825 1850 3275 1850
-Wire Wire Line
-	3275 1850 3275 1950
+	2450 1850 2925 1850
 Wire Wire Line
 	1900 6325 2200 6325
@@
 	900  1850 1950 1850
 Wire Wire Line
-	2925 2025 2925 1850
-Connection ~ 2925 1850
-NoConn ~ 2450 2000
+	2925 1850 2925 2025
 $Comp
 L +3.3V #PWR01
@@
 P 1500 2100
 F 0 "C7" H 1575 2100 27  0000 L TNN
-F 1 "0.1uF,16V" H 1575 2150 27  0000 L TNN
-F 2 "C0402" H 1550 2150 27  0001 L TNN
+F 1 "1uF,10V" H 1575 2150 27  0000 L TNN
+F 2 "C0805" H 1550 2150 27  0001 L TNN
 F 3 "" H 1500 2100 60  0001 C CNN
-F 4 "0402/0.1uF/16V/Y" H 1500 2100 60  0001 C CNN "Field4"
+F 4 "1u/10V/X7R" H 1500 2100 60  0001 C CNN "Field4"
 	1    1500 2100
 	1    0    0    1
@@
 $EndComp
 $Comp
-L R R4
-U 1 1 514F45B1
-P 2700 1850
-F 0 "R4" V 2750 1825 27  0000 L TNN
-F 1 "26.7K/1%" V 2625 1750 27  0000 L TNN
-F 2 "R0603" H 2750 1900 27  0001 L TNN
-F 3 "" H 2700 1850 60  0001 C CNN
-F 4 "0603/26.7K/1%" V -2950 2950 60  0001 C CNN "Field4"
-	1    2700 1850
-	0    1    -1   0
-$EndComp
-$Comp
 L CAPACITOR_NON_POL_2 C3
 U 1 1 514F45AF
@@
 $EndComp
 $Comp
-L R R5
-U 1 1 514F4565
-P 3275 2075
-F 0 "R5" H 3175 2125 27  0000 L TNN
-F 1 "17.8K/1%" H 3025 2075 27  0000 L TNN
-F 2 "R0603" H 3325 2125 27  0001 L TNN
-F 3 "" H 3275 2075 60  0001 C CNN
-F 4 "0603/17.8K/1%" H -4575 -2675 60  0001 C CNN "Field4"
-	1    3275 2075
-	-1   0    0    -1
-$EndComp
-$Comp
 L R R12
 U 1 1 514F4567
@@
 	1    9575 1200
 	0    -1   1    0
-$EndComp
-$Comp
-L LM3940_19 U1
-U 1 1 514F4551
-P 2000 2050
-F 0 "U1" H 2000 2100 27  0000 L TNN
-F 1 "S-5813A/S-5814A" H 2000 1775 27  0000 L TNN
-F 2 "SNT-4A" H 2050 2100 27  0001 L TNN
-F 3 "" H 2000 2050 60  0001 C CNN
-	1    2000 2050
-	1    0    0    1
 $EndComp
 $Comp
@@
 Text Label 2200 6275 2    24   ~ 0
 SW2
-Text Label 3025 1850 0    24   ~ 0
+Text Label 2600 1850 0    24   ~ 0
 TEMPERATURE
 Text Label 2200 6325 2    24   ~ 0
@@
 Connection ~ 2775 1350
 Wire Wire Line
-	1500 2250 3275 2250
+	1500 2250 2925 2250
 Wire Wire Line
 	1500 2250 1500 2200
-Connection ~ 2925 2250
 Wire Wire Line
 	1500 2025 1500 1850
 Connection ~ 1500 1850
-Wire Wire Line
-	1900 2000 1900 2300
-Connection ~ 1900 2250
 Text Label 2000 2250 0    30   ~ 0
 GND
@@
 L GND #PWR09
 U 1 1 5151E3F1
-P 1900 2300
-F 0 "#PWR09" H 1900 2300 30  0001 C CNN
-F 1 "GND" H 1900 2370 30  0001 C CNN
-F 2 "" H 1900 2300 60  0000 C CNN
-F 3 "" H 1900 2300 60  0000 C CNN
-	1    1900 2300
+P 2200 2300
+F 0 "#PWR09" H 2200 2300 30  0001 C CNN
+F 1 "GND" H 2200 2370 30  0001 C CNN
+F 2 "" H 2200 2300 60  0000 C CNN
+F 3 "" H 2200 2300 60  0000 C CNN
+	1    2200 2300
 	1    0    0    -1
 $EndComp
@@
 NoConn ~ 4000 6425
 NoConn ~ 4000 6525
+$Comp
+L MCP9700AT-E/TT U1
+U 1 1 5155C609
+P 2000 1800
+F 0 "U1" H 2000 1850 30  0000 L CNN
+F 1 "MCP9700AT-E/TT" H 2000 1900 30  0000 L CNN
+F 2 "~" H 2000 1800 60  0000 C CNN
+F 3 "~" H 2000 1800 60  0000 C CNN
+	1    2000 1800
+	1    0    0    -1
+$EndComp
+Wire Wire Line
+	2200 2100 2200 2300
+Connection ~ 2200 2250
 $EndSCHEMATC

Commit message: OHSBadge - started basic PCB layout
Parts:
- added C5: 0.1u,16V, C0603, symbol CAPACITOR_NON_POL_2
- added R4, R5, R6: 10k, R0402, symbol R
- added SW1: SEL, ~, symbol SW_PUSH
- added SW2: UP, ~, symbol SW_PUSH
- added SW3: DOWN, ~, symbol SW_PUSH
- C1: value 2.2u,10V -> 2.2u,16V; Field4 0805/2.2u/10V/Y -> 0805/2.2u/10V/Y5V
- C2, C4, C8: value 0.1uF,16V -> 0.1u,16V
- C26: value 100n,16V -> 0.1u,16V
- C27, C29: value 0.1uF -> 0.1u,16V
- C28, C30: value 2.2uF,16V -> 2.2u,16V
- C3: value 0.1uF,16V -> 0.1u,16V; Field4 0402/0.1uF/16V/Y -> 0402/0.1uF/16V/Y5V
- C7: value 1uF,10V -> 1u,16V
Connections:
- net labels removed: 3V3, AREF, PC0, PC1, PC2, PC3, RST, SCL, V_IN
- wire segments 254 -> 255
- no-connect marks 34 -> 32
Other:
- moved on the sheet: C1, C2, C27, C28, C29, C3, C30, C4, C7, C8, J1, J2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

Commit message: OHSBadge - Track layout in progress (almost done).
Connections:
- net labels removed: 5V0, ENABLE_5V
- wire segments 255 -> 254
Changed lines of the file:
@@
-EESchema Schematic File Version 2  date 30-Mar-13 5:07:47 PM
+EESchema Schematic File Version 2  date Sunday 31 March 2013 11:53:46 PM IST
 LIBS:power
 LIBS:repaper_sym
@@
 Sheet 1 1
 Title ""
-Date "30 mar 2013"
+Date "31 mar 2013"
 Rev ""
 Comp ""
@@
 	900  6550 900  6900
 Wire Wire Line
-	750  6600 1250 6600
+	900  6600 1250 6600
 Wire Wire Line
 	2100 6600 2100 6900
@@
 Text Label 1900 5625 0    24   ~ 0
 /EPD_CS
-Text Label 1025 4525 2    24   ~ 0
+Text Label 1025 4625 2    24   ~ 0
 /EPD_CS
 Text Label 1900 5675 0    24   ~ 0
 FLASH_CS
-Text Label 1025 4625 2    24   ~ 0
+Text Label 1025 4525 2    24   ~ 0
 FLASH_CS
 Text Label 1275 6025 2    24   ~ 0
@@
 Text Label 1900 5975 0    24   ~ 0
 DISCHARGE
-Text Label 2025 4525 0    24   ~ 0
+Text Label 2025 4625 0    24   ~ 0
 EPD_CS_COG
 Text Label 1200 2775 0    30   ~ 0
 FLASH_CS_COG
-Text Label 2025 4625 0    24   ~ 0
+Text Label 2025 4525 0    24   ~ 0
 FLASH_CS_COG
 Text Label 1900 5575 0    24   ~ 0
@@
 Text Label 1900 5875 0    24   ~ 0
 SPI_MISO
-Text Label 1025 4425 2    24   ~ 0
+Text Label 1025 4325 2    24   ~ 0
 SPI_MISO
 Text Label 1200 3025 0    30   ~ 0
 SPI_MISO_COG
-Text Label 2025 4425 0    24   ~ 0
+Text Label 2025 4325 0    24   ~ 0
 SPI_MISO_COG
 Text Label 1900 5825 0    24   ~ 0
 SPI_MOSI
-Text Label 1025 4325 2    24   ~ 0
+Text Label 1025 4425 2    24   ~ 0
 SPI_MOSI
 Text Label 1200 2825 0    30   ~ 0
 SPI_MOSI_COG
-Text Label 2025 4325 0    24   ~ 0
+Text Label 2025 4425 0    24   ~ 0
 SPI_MOSI_COG
 Text Label 1275 5775 2    24   ~ 0
@@
 VCC3V
 Text Label 1275 5575 2    24   ~ 0
-5V0
+VCC5V
 Text Label 9300 2600 0    24   ~ 0
 VCC_T
@@
 	1    0    0    -1
 $EndComp
-Text Label 1850 3350 0    40   ~ 0
-GND
 $Comp
 L VCC_CIRCLE #PWR10
@@
 TXD
 Text Label 6175 5875 0    40   ~ 0
-ENABLE_5V
+VCC5V
 Text Label 6175 5775 0    40   ~ 0
 SPI_MOSI
@@
 	1    0    0    -1
 $EndComp
-$Comp
-L PWR_FLAG #FLG021
-U 1 1 51531060
-P 750 6550
-F 0 "#FLG021" H 750 6455 30  0001 C CNN
-F 1 "PWR_FLAG" H 750 6725 30  0000 C CNN
-F 2 "" H 750 6550 60  0000 C CNN
-F 3 "" H 750 6550 60  0000 C CNN
-	1    750  6550
-	1    0    0    -1
-$EndComp
-Wire Wire Line
-	750  6550 750  6600
 Wire Wire Line
 	2500 7175 2500 7150
@@
 Connection ~ 8950 6475
 $Comp
-L GND #PWR022
+L GND #PWR021
 U 1 1 5156E539
 P 8950 6750
-F 0 "#PWR022" H 8950 6750 30  0001 C CNN
+F 0 "#PWR021" H 8950 6750 30  0001 C CNN
 F 1 "GND" H 8950 6820 30  0001 C CNN
 F 2 "" H 8950 6750 60  0000 C CNN
@@
 Text Label 7325 4875 0    40   ~ 0
 VCC3V
+Text Label 1200 2700 0    30   ~ 0
+VCC3V
+Text Label 1600 1350 0    30   ~ 0
+GND
+Text Label 1200 3350 0    30   ~ 0
+GND
+Text Label 1700 5175 0    30   ~ 0
+GND
 $EndSCHEMATC

Commit message: OHSBadge - original design renamed as repaper_dumb. creating a new Schematic with ATMega included.
Parts:
- added IC?: ATMEGA328-AU-ND, TQFP32, symbol ATMEGA328-AU-ND
- added P1: PCB, symbol PCB
- added X?: CRYSTAL_2, symbol CRYSTAL_2
Connections:
- net labels removed: SDA
- wire segments 254 -> 301
Other:
- moved on the sheet: C10, C11, C12, C13, C14, C15, C16, C17, C18, C19, C20, C21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

Commit message: OHSBadge - check the revised schematic - includes 328P and headers for ISP, FTDI and C3SB
Parts:
- added B1, B2: I/O, ~, symbol I/O
- added C31: 0.1u,16V, C0603, symbol CAPACITOR_NON_POL_2
- added C6, C9: 22pF, C0603, symbol CAPACITOR_NON_POL_2
- added P2: ISP, symbol ISP
- added P3: FTDI, symbol ISP
- added P4: C3SB, symbol CONN_4
- added R7: 10k, R0402, symbol R
- added SW4: RST, ~, symbol SW_PUSH
- X1: renamed from X?; value CRYSTAL_2 -> CRYSTAL_16MHz
- gave numbers to parts that had none: 1
Connections:
- net labels added: AD6, AD7, RST, SCL, SDA, SPI_SS
- wire segments 301 -> 322
Other:
- note added: "Interfaces_Communication"
- moved on the sheet: C26, D1, P1, R4, R5, R6, SHIELD1, SW1, SW2, SW3, U2, X1

Commit message: OHSBadge : added 328P, and full Arduino shield. See Board outline for lanyard looping option.
Parts:
- removed J1, J2: HEADER1X10MS2.54, HEADER1X10MS2.54_SMD, symbol CON10
Connections:
- net labels removed: LED1, RST/SBWTDIO, SW2, TEST/SBWTCK, UART_RX, UART_TX
- wire segments 322 -> 307
- no-connect marks 32 -> 29
Other:
- note added: "TI Launchpad Interface - REMOVED"
- note removed: "Microcontroller Interface"
