File: KiCad/uControl_v2/interface.sch (KiCad schematic (older format))
At the start: 72 parts, among them M1 MANIFOLD, P10 C3SB, P11 VSel_Vlv, P12 Valve_Conn, P13 Valve_Conn_BO, P14 X_VALVE, P15 FLOW_CONN, P16 FLOWMETER, P17 Pump_Conn, P18 Pump_Conn_BO, P19 PUMP_CONN_FLEX, P20 Temp_Conn, P21 Temp_Conn_BO, P22 Temp, P23 PUMP, P28 VLV_90_M, P29 VLV_90_F, P30 X_VALVE_CONN, P31 FLOW_CONN_CABLE, P32 FLOWMETER, P6 Pulse, P7 GAGE_PR, P8 ABSO_PR, P9 C3SB, Q1 TIP112G, U1 TXB0104D, U2 TXS0102DCT

Commit message: uControl_v2 schematic more progress
Parts:
- removed D2: 1N5225B, diode_do35, symbol D_1N5225B
- removed P15: FLOW_CONN, Conn_Flow, symbol FLOW_CONN
- removed P31: FLOW_CONN_CABLE, symbol FLOW_CONN_CABLE
- added D2: 1N4001, diode_do41, symbol D_1N4001
- added P15: FLOW_CONN, FlowMeter, symbol FLOWMETER
- added P31: FLOW_CABLE, symbol FLOWMETER
- added Q?: TIP112G, TO220-3-V, symbol NPN_TIP112G
- P16, P32: footprint FlowMeter -> (none); Field10 EM1NR4R0V_1A -> (none); Field11 http://www.sensirion.com/en/products/mass-flow-meters-for-g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 -> (none); Field4 Mass Flow Meter for Gases -> (none); Field5 CMOSens EM1 -> (none); Field6 G3/8 thread (BSPP -> (none); Field7 Sensirion -> (none); Field8 EM1NR4R0V_1A -> (none); Field9 Sensirion -> (none)
- P23: footprint Pump -> (none); Field10 P200_GAS -> (none); Field4 Intelligent Pump -> (none); Field5 P200/P1500 -> (none); Field6 X-Life Motor -> (none); Field7 XAVITECH -> (none); Field8 P200_GAS -> (none); Field9 XAVITECH -> (none)
Connections:
- net labels removed: PB0_IO_R, PD2_Flow_Tx, PD4_Flow_Rx, PD7_IO_X
- wire segments 200 -> 195
- no-connect marks 39 -> 31
Other:
- note added: "Absolute Pressure Sensor #2 on I2C Bus [HDIB002AUY8H5]"
- note added: "Additional footprint for\nalternate mounting position\n(not used)"
- note added: "Flow Meter on I2C : SFM3000\nAddress : 64 (h40)"
- note added: "Gage Sensor #1 on SPI Bus [HCEM500GUH9P3]"
- note added: "Pump cable assembly"
- note added: "Pump, 12V DC [P54E01R]\non digital port ~PB1"
- note added: "Symbol for FlowMeter\nConnector"
- note added: "Symbol for FlowMeter\nFootprint"
- note added: "Symbol for Pump\n[P54E01R]\nFootprint"
- note removed: "Absolute Pressure Sensor #2 on I2C Bus"
- note removed: "Additional footprint for\nalternate mounting position"
- note removed: "Flow Meter on Serial"
- note removed: "Gage Sensor #1 on SPI Bus"
- note removed: "P200"
- note removed: "Pump on digital port\nV_IN = 12V DC\nIO_X = 3V3 for pump control"
- moved on the sheet: C27

Commit message: uControl_v2 : schematic work in progress
Parts:
- removed P17: Pump_Conn, Header_FTDI, symbol CONN_6
- removed P18: Pump_Conn_BO, Header_FTDI, symbol CONN_6
- removed P19: PUMP_CONN_FLEX, Conn_Pump_Flex, symbol PUMP_CONN_FLEX
- added P17: Pump_Conn, Header_5V_Link, symbol CONN_2
- added P18, P19: Pump_Cable, Header_5V_Link, symbol CONN_2
Connections:
- net labels removed: IO_R, IO_X, ~PB1_IO_T
- wire segments 195 -> 240

Commit message: uControl_v2 schematic progression
Parts:
- removed C16: 100n, c_0805, symbol C2
- removed C6: 100n, C2, symbol C
- removed D3: 1N5225B, diode_do35, symbol D_1N5225B
- removed P20: Temp_Conn, SIL-4, symbol CONN_4
- removed P21: Temp_Conn_BO, SIL-4, symbol CONN_4
- removed P22: Temp, STS21, symbol STS21
- removed P28: VLV_90_M, 2X06/90, symbol CONN_12
- removed P29: VLV_90_F, Header_F_6x2, symbol CONN_12
- removed P6: Pulse, pin_strip_3-90, symbol CONN_3
- removed R5, R6: 47E, rc03_vert, symbol R_47E
- removed SC21, SC22, SC23, SC24: SCREW, vite_3mm, symbol SCREW
- removed U2: TXS0102DCT, TXS0102DCTR, symbol TXS0102DCT
- added B4, B5: I/O, symbol I/O
- added C16, C31: 100n, C2, symbol C
- added C6: 100u,16V, CP_6.3x7mm, symbol C_POL_1
- added D3, D9: 1N4001, diode_do41, symbol D_1N4001
- added P34: VSel_Vlv2, SIL-3, symbol CONN_3
- added P35: Valve2, Header_5V_Link, symbol CONN_2
- added P36: Valve2_Conn_BO, Header_5V_Link, symbol CONN_2
- added P37: X_VALVE2_CONN, Valve_Conn, symbol X_VALVE_CONN
- added P38: X_VALVE2, Valve, symbol X_VALVE
- added PCB4: PCB_Vlv2, PCB_Vlv, symbol PCB
- added Q3, Q4: TIP112G, TO220-3-V, symbol NPN_TIP112G
- added R14: 8k2, rc03_vert, symbol R_10K
- added R5, R6: 1k, rc03_vert, symbol R_10K
- added SC27, SC28, SC29, SC30: SCREW, vite_3mm, symbol SCREW
- added SP1: BUZZER, symbol BUZZER
- added U2: ADXL345, symbol ADXL345
- P12: value Valve_Conn -> Valve1
- R7: value 10K -> 16k
- gave numbers to parts that had none: 1
Connections:
- net labels added: +Vlv2, -Vlv2, PB0_ACL, PB0_ACL_3V, PD4_Valve2, ~PB1_Pump, ~PD6_Spk
- net labels removed: PC1_Pulse, TSCL, TSDA
- wire segments 240 -> 176
- no-connect marks 31 -> 34
Other:
- note added: "Accelerometer, 3V3\non 3V3 SPI (share with Pr. Sensor)\nLevel shifter for CS"
- note added: "Flow Meter on I2C\nSFM3000\nAddress : 64 (h40)"
- note added: "Pressure Sensor #1, Gage, SPI Bus [HCEM500GUH9P3]"
- note added: "Pressure Sensor #2, Absolute, I2C Bus [HDIB002AUY8H5]"
- note added: "Spare I2C on C3SB Bus"
- note added: "Speaker, 12V DC\ndigital PWM port ~PD6"
- note added: "Valve #1 on digital PWM port\neither 12V (V_IN) or 5V0"
- note added: "Valve #2 on digital port PD4\neither 12V (V_IN) or 5V0"
- note removed: "Absolute Pressure Sensor #2 on I2C Bus [HDIB002AUY8H5]"
- note removed: "Dummy Mounting Headers\nfor Valve Board, 2 x 6 way"
- note removed: "Flow Meter on I2C : SFM3000\nAddress : 64 (h40)"
- note removed: "Gage Sensor #1 on SPI Bus [HCEM500GUH9P3]"
- note removed: "Pulse Sensor\nAnalog + I2C on C3SB Bus"
- note removed: "SPARE"
- note removed: "Temp Sensor on I2C\nwith 3V3<>5V0 translator"
- note removed: "Valve on digital PWM port\neither 12V (V_IN) or 5V0"
- moved on the sheet: C11, C12, C5, C9, M1, P10, P9, PCB2, PCB3, PCB6, SC1, SC13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

Commit message: uControl_v2 : Schematic DRC passes. Most component footprints done. Using old PCB layout to begin with
Parts:
- removed P19: Pump_Cable, Header_5V_Link, symbol CONN_2
- removed P30: X_VALVE_CONN, Valve_Conn, symbol X_VALVE_CONN
- removed P32: FLOWMETER, symbol FLOWMETER
- removed P37: X_VALVE2_CONN, Valve_Conn, symbol X_VALVE_CONN
- removed R14: 8k2, rc03_vert, symbol R_10K
- removed R7: 16k, rc03_vert, symbol R_10K
- added B6: I/O, I/O, symbol I/O
- added C28, C29: 100n, c_0805, symbol C
- added U8: TXB0104D, TXB0104D, symbol TXB0104D
- B4, B5: footprint (none) -> I/O
- C10, C11, C12, C13, C14, C15, C16, C17, C31, C5, C7, C8, C9: footprint C2 -> c_0805
- C27, C6: footprint CP_6.3x7mm -> C_ELCO_SMD
- D1, D2, D3, D9: footprint diode_do41 -> d_0805
- P11, P34: footprint SIL-3 -> Header_3
- P12, P13, P17, P18, P35, P36: footprint Header_5V_Link -> Header_2
- P15: value FLOW_CONN -> Flow_Conn; footprint FlowMeter -> Header_4
- P16: footprint (none) -> FlowMeter
- P23: footprint (none) -> Pump
- P31: footprint (none) -> Header_4
- Q1, Q2, Q3, Q4: footprint TO220-3-V -> DPAK_3
- R4, R6: footprint rc03_vert -> r_0805
- R5: value 1k -> 10K; footprint rc03_vert -> r_0805
- SP1: footprint (none) -> Speaker
- U2: footprint (none) -> ADXL345
Connections:
- net labels added: A_SCL, A_SDA, A_SDO, Pump, Spk
- wire segments 176 -> 187
- no-connect marks 34 -> 30
Other:
- note added: "Accelerometer, 3V3 I2C"
- note added: "Connector at Flow Meter"
- note added: "Connector at Pump"
- note added: "Connector at Valve"
- note added: "Connector at uC_v2"
- note added: "Flow Meter, I2C , SFM3000\nAddress : 64 (h40)"
- note added: "FlowMeter Footprint"
- note added: "Pump [P54E01R]\nFootprint"
- note added: "Speaker, 5V DC\ndigital PWM port ~PD6"
- note added: "Valve Footprint"
- note removed: "Accelerometer, 3V3\non 3V3 SPI (share with Pr. Sensor)\nLevel shifter for CS"
- note removed: "Additional footprint for\nalternate mounting position\n(not used)"
- note removed: "Flow Meter on I2C\nSFM3000\nAddress : 64 (h40)"
- note removed: "Flow Sensor cable assembly"
- note removed: "Pump cable assembly"
- note removed: "Speaker, 12V DC\ndigital PWM port ~PD6"
- note removed: "Symbol for FlowMeter\nConnector"
- note removed: "Symbol for FlowMeter\nFootprint"
- note removed: "Symbol for Pump\n[P54E01R]\nFootprint"
- moved on the sheet: B4, B5, C12, C13, C14, C15, C16, C27, C31, C5, C6, D1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

Commit message: uControl_v2 : Moved Accel to Ras-Pi side. Added 2 buttons to Atmega. Working on new footprints (flow, pump)
Parts:
- removed B4, B5, B6: I/O, I/O, symbol I/O
- removed C15, C16, C28, C29: 100n, c_0805, symbol C
- removed C6: 100u,16V, C_ELCO_SMD, symbol C_POL_1
- removed R5: 10K, r_0805, symbol R_10K
- removed U2: ADXL345, ADXL345, symbol ADXL345
- removed U8: TXB0104D, TXB0104D, symbol TXB0104D
- R4: value 10K -> 10k
Connections:
- net labels removed: A_SCL, A_SDA, A_SDO, PB0_ACL, PB0_ACL_3V
- wire segments 187 -> 148
- no-connect marks 30 -> 26
Other:
- note removed: "Accelerometer, 3V3 I2C"

Commit message: 
Parts:
- P15: footprint Header_4 -> Conn_Flow_SFM3000_Male
- P31: footprint Header_4 -> (none)
Changed lines of the file:
@@
-EESchema Schematic File Version 2  date 16-Aug-13 2:36:23 PM
+EESchema Schematic File Version 2
 LIBS:Conn-raspberry
 LIBS:power
 LIBS:uControl
 LIBS:uControl_v2-cache
-EELAYER 27 0
+EELAYER 24 0
 EELAYER END
 $Descr A4 11693 8268
@@
 F 0 "P15" V 6150 2100 50  0000 C CNN
 F 1 "Flow_Conn" V 6250 2100 40  0000 C CNN
-F 2 "Header_4" V 6350 2100 40  0001 C CNN
+F 2 "Conn_Flow_SFM3000_Male" V 6350 2100 40  0001 C CNN
 F 3 "" H 6200 2100 60  0001 C CNN
 F 4 "Mass Flow Meter for Gases" H 6200 2200 60  0001 L CNN "Field4"
@@
 F 0 "P31" V 7000 2100 50  0000 C CNN
 F 1 "FLOW_CABLE" V 7100 2100 40  0000 C CNN
-F 2 "Header_4" V 7200 2100 40  0001 C CNN
+F 2 "" V 7200 2100 40  0001 C CNN
 F 3 "" H 7050 2100 60  0001 C CNN
 F 4 "http://www.sensirion.com/en/products/mass-flow-meters-for-gases/mass-flow-meter-em1/" H 7050 2900 60  0001 L CNN "Field11"

Commit message: uControl_v2 : Components selected and footprints done. Ready to start layout
Parts:
- removed P13: Valve_Conn_BO, Header_2, symbol CONN_2
- removed P36: Valve2_Conn_BO, Header_2, symbol CONN_2
- removed PCB2: PCB_Pump, PCB_Pump, symbol PCB
- removed PCB3: PCB_Flow, PCB_Flow, symbol PCB
- removed PCB4: PCB_Vlv2, PCB_Vlv, symbol PCB
- removed PCB5: PCB_Vlv, PCB_Vlv, symbol PCB
- removed PCB6: PCB_MFold, PCB_Mfold, symbol PCB
- C10, C11, C12, C13, C14, C17, C31, C5, C7, C8, C9: footprint c_0805 -> c_0603
- D1, D2, D3, D9: value 1N4001 -> 1N4007; footprint d_0805 -> diode-DO214AC
- P14, P38: footprint Valve -> X_Valve_2
- P16: footprint FlowMeter -> FlowMeter_CFM3000
- P18: footprint Header_2 -> (none)
- P23: footprint Pump -> Pump_P54E01R
- Q1, Q2, Q3, Q4: value TIP112G -> BCP5416TA; footprint DPAK_3 -> SOT223
- R4, R6: footprint r_0805 -> r_0603
Connections:
- no-connect marks 26 -> 22
Other:
- note added: "Flow Meter cable"
- note added: "Pump cable"
- note removed: "Connector at Flow Meter"
- note removed: "Connector at Pump"
- note removed: "Connector at Valve"
- moved on the sheet: P14, P38
