File: KiCad/uControl_v2/uControl_RPi.sch (KiCad schematic (older format))
At the start: 9 parts, among them P25 U6_OE, P26 5V_LINK, P27 BCM2835_GPIO, U6 TSX0108

Commit message: uControl_v2 : Schematic DRC passes. Most component footprints done. Using old PCB layout to begin with
Parts:
- C24, C25: footprint C2 -> c_0805
- P25: footprint pin_strip_3-90 -> ShortLink2
- P26: footprint Header_U6OE -> ShortLink2
- R12: footprint rc03_vert -> r_0805
Changed lines of the file:
@@
 F 0 "R12" H 5525 1775 50  0000 C CNN
 F 1 "10K" V 5630 1625 50  0000 C CNN
-F 2 "rc03_vert" V 5730 1625 50  0001 C CNN
+F 2 "r_0805" V 5730 1625 50  0001 C CNN
 F 3 "" H 5625 1625 60  0001 C CNN
 F 4 "RES 10K OHM 1/8W 5% CF AXIAL" H 5625 1725 60  0001 L CNN "Field4"
@@
 F 0 "C25" H 2300 1950 50  0000 L CNN
 F 1 "100n" H 2300 1750 50  0000 L CNN
-F 2 "C2" H 2300 1850 50  0001 C CNN
+F 2 "c_0805" H 2300 1850 50  0001 C CNN
 F 3 "" H 2300 1850 60  0001 C CNN
 F 4 "CAP FILM 0.1UF 63VDC RADIAL" H 2300 2050 60  0001 L CNN "Field4"
@@
 F 0 "C24" H 1925 1950 50  0000 L CNN
 F 1 "100n" H 1925 1750 50  0000 L CNN
-F 2 "C2" H 1925 1850 50  0001 C CNN
+F 2 "c_0805" H 1925 1850 50  0001 C CNN
 F 3 "" H 1925 1850 60  0001 C CNN
 F 4 "CAP FILM 0.1UF 63VDC RADIAL" H 1925 2050 60  0001 L CNN "Field4"
@@
 	2125 3600 2125 3500
 Wire Wire Line
-	2300 2050 2300 2125
-Wire Wire Line
-	2300 2125 1925 2125
-Wire Wire Line
-	1925 2125 1925 2050
+	2300 2125 2300 1975
+Wire Wire Line
+	1925 2125 2300 2125
+Wire Wire Line
+	1925 2125 1925 1975
 Connection ~ 1925 1575
 Wire Wire Line
-	1925 1650 1925 1575
+	1925 1725 1925 1575
 Wire Wire Line
 	3750 1475 2300 1475
@@
 	3250 2375 1500 2375
 Wire Wire Line
-	3450 1875 3450 1575
+	3450 1575 3450 1875
 Wire Wire Line
 	1500 3075 3250 3075
@@
 	3250 2475 1500 2475
 Wire Wire Line
-	3450 1575 1500 1575
-Wire Wire Line
-	2300 1475 2300 1650
+	1500 1575 3450 1575
+Wire Wire Line
+	2300 1475 2300 1725
 Wire Wire Line
 	2125 2175 2125 2125
@@
 	5850 1425 5850 2050
 Wire Wire Line
-	5950 1325 5225 1325
+	5225 1325 5950 1325
 Wire Wire Line
 	5225 1325 5225 2175
@@
 	5950 1225 5525 1225
 $Comp
-L PWR_FLAG #FLG025
+L PWR_FLAG #FLG029
 U 1 1 50E00A24
 P 6300 4000
-F 0 "#FLG025" H 6300 4270 30  0001 C CNN
+F 0 "#FLG029" H 6300 4270 30  0001 C CNN
 F 1 "PWR_FLAG" H 6300 4230 30  0000 C CNN
 F 2 "" H 6300 4000 60  0001 C CNN
@@
 F 0 "P26" V 7450 3650 50  0000 C CNN
 F 1 "5V_LINK" V 7550 3650 50  0000 C CNN
-F 2 "Header_U6OE" H 7350 3850 50  0001 C CNN
+F 2 "ShortLink2" H 7350 3850 50  0001 C CNN
 F 3 "" H 7500 3650 60  0001 C CNN
 	1    7500 3650
@@
 Rpi_OE
 $Comp
-L GND #PWR026
+L GND #PWR030
 U 1 1 4FD8C28A
 P 5850 2050
-F 0 "#PWR026" H 5850 2050 30  0001 C CNN
+F 0 "#PWR030" H 5850 2050 30  0001 C CNN
 F 1 "GND" H 5850 1980 30  0001 C CNN
 F 2 "" H 5850 2050 60  0001 C CNN
@@
 F 0 "P25" V 6250 1325 50  0000 C CNN
 F 1 "U6_OE" V 6350 1325 50  0000 C CNN
-F 2 "pin_strip_3-90" H 6300 1275 60  0001 C CNN
+F 2 "ShortLink2" H 6300 1275 60  0001 C CNN
 F 3 "" H 6300 1325 60  0001 C CNN
 	1    6300 1325
@@
 Rpi_3V3
 $Comp
-L GND #PWR027
+L GND #PWR031
 U 1 1 4FD62C0F
 P 2125 2175
-F 0 "#PWR027" H 2125 2175 30  0001 C CNN
+F 0 "#PWR031" H 2125 2175 30  0001 C CNN
 F 1 "GND" H 2125 2105 30  0001 C CNN
 F 2 "" H 2125 2175 60  0001 C CNN
@@
 $EndComp
 $Comp
-L GND #PWR028
+L GND #PWR032
 U 1 1 4FD62BFD
 P 2125 3600
-F 0 "#PWR028" H 2125 3600 30  0001 C CNN
+F 0 "#PWR032" H 2125 3600 30  0001 C CNN
 F 1 "GND" H 2125 3530 30  0001 C CNN
 F 2 "" H 2125 3600 60  0001 C CNN

Commit message: uControl_v2 : Moved Accel to Ras-Pi side. Added 2 buttons to Atmega. Working on new footprints (flow, pump)
Parts:
- added B4: A_INT1, I/O, symbol I/O
- added B5: A_INT2, I/O, symbol I/O
- added B6: A_SDO, I/O, symbol I/O
- added B7: A_CS, I/O, symbol I/O
- added C15, C16: 100n, c_0805, symbol C
- added C6: 100u,16V, C_ELCO_SMD, symbol C_POL_1
- added R14, R15, R16, R5: 8k, r_0805, symbol R_10K
- added R17, R18, R19, R20: 16k, r_0805, symbol R_10K
- added U2: ADXL345, ADXL345, symbol ADXL345
- R12: value 10K -> 10k
Connections:
- net labels added: 3V3, ACL_CS, ACL_INT1, ACL_INT2, ACL_SDO
- wire segments 63 -> 100
- no-connect marks 16 -> 18
Other:
- note added: "Accelerometer, 3V3 I2C"
- note added: "Enable/Disable Voltage Translator U6,\nAllow/Dis-allow comm betn\nRasp-Pi and AlaMode"
- note removed: "this jumper enables/disables the Voltage Translator U6, \nthereby allowing/dis-allowing communication \nbetween the Raspberry-Pi and a La Mode\nEDIT:Permanenty shorted(23-08-2012)"
- moved on the sheet: C24, C25, P25, P26, P27, SC25, SC26, U6

Commit message: uControl_v2 : Components selected and footprints done. Ready to start layout
Parts:
- C15, C16, C24, C25: footprint c_0805 -> c_0603
- R12, R14, R15, R16, R17, R18, R19, R20, R5: footprint r_0805 -> r_0603
Changed lines of the file:
@@
-EESchema Schematic File Version 2
+EESchema Schematic File Version 2  date 17-Aug-13 4:16:47 PM
 LIBS:Conn-raspberry
 LIBS:power
 LIBS:uControl
 LIBS:uControl_v2-cache
-EELAYER 24 0
+EELAYER 27 0
 EELAYER END
 $Descr A4 11693 8268
@@
 Sheet 5 5
 Title "uControl"
-Date "16 aug 2013"
+Date "17 aug 2013"
 Rev "1"
 Comp "WyoLum"
@@
 F 0 "R12" H 3300 1775 50  0000 C CNN
 F 1 "10k" V 3405 1625 50  0000 C CNN
-F 2 "r_0805" V 3505 1625 50  0001 C CNN
+F 2 "r_0603" V 3505 1625 50  0001 C CNN
 F 3 "" H 3400 1625 60  0001 C CNN
 F 4 "RES 10K OHM 1/8W 5% CF AXIAL" H 3400 1725 60  0001 L CNN "Field4"
@@
 F 0 "C25" H 1400 1950 50  0000 L CNN
 F 1 "100n" H 1400 1750 50  0000 L CNN
-F 2 "c_0805" H 1400 1850 50  0001 C CNN
+F 2 "c_0603" H 1400 1850 50  0001 C CNN
 F 3 "" H 1400 1850 60  0001 C CNN
 F 4 "CAP FILM 0.1UF 63VDC RADIAL" H 1400 2050 60  0001 L CNN "Field4"
@@
 F 0 "C24" H 1125 1950 50  0000 L CNN
 F 1 "100n" H 1125 1750 50  0000 L CNN
-F 2 "c_0805" H 1125 1850 50  0001 C CNN
+F 2 "c_0603" H 1125 1850 50  0001 C CNN
 F 3 "" H 1125 1850 60  0001 C CNN
 F 4 "CAP FILM 0.1UF 63VDC RADIAL" H 1125 2050 60  0001 L CNN "Field4"
@@
 F 0 "C15" V 10875 1900 50  0000 L CNN
 F 1 "100n" V 10875 1600 50  0000 L CNN
-F 2 "c_0805" H 10825 1850 50  0001 C CNN
+F 2 "c_0603" H 10825 1850 50  0001 C CNN
 F 3 "" H 10825 1850 60  0001 C CNN
 F 4 "CAP FILM 0.1UF 63VDC RADIAL" H 10825 2050 60  0001 L CNN "Field4"
@@
 F 0 "C16" V 11075 1900 50  0000 L CNN
 F 1 "100n" V 11075 1600 50  0000 L CNN
-F 2 "c_0805" H 11025 1850 50  0001 C CNN
+F 2 "c_0603" H 11025 1850 50  0001 C CNN
 F 3 "" H 11025 1850 60  0001 C CNN
 F 4 "CAP FILM 0.1UF 63VDC RADIAL" H 11025 2050 60  0001 L CNN "Field4"
@@
 F 0 "R5" V 8250 1825 50  0000 C CNN
 F 1 "8k" V 8205 1625 50  0000 C CNN
-F 2 "r_0805" V 8305 1625 50  0001 C CNN
+F 2 "r_0603" V 8305 1625 50  0001 C CNN
 F 3 "" H 8200 1625 60  0001 C CNN
 F 4 "RES 10K OHM 1/8W 5% CF AXIAL" H 8200 1725 60  0001 L CNN "Field4"
@@
 F 0 "R14" V 8250 1925 50  0000 C CNN
 F 1 "8k" V 8205 1725 50  0000 C CNN
-F 2 "r_0805" V 8305 1725 50  0001 C CNN
+F 2 "r_0603" V 8305 1725 50  0001 C CNN
 F 3 "" H 8200 1725 60  0001 C CNN
 F 4 "RES 10K OHM 1/8W 5% CF AXIAL" H 8200 1825 60  0001 L CNN "Field4"
@@
 F 0 "R15" V 8250 2325 50  0000 C CNN
 F 1 "8k" V 8205 2125 50  0000 C CNN
-F 2 "r_0805" V 8305 2125 50  0001 C CNN
+F 2 "r_0603" V 8305 2125 50  0001 C CNN
 F 3 "" H 8200 2125 60  0001 C CNN
 F 4 "RES 10K OHM 1/8W 5% CF AXIAL" H 8200 2225 60  0001 L CNN "Field4"
@@
 F 0 "R16" V 8250 2425 50  0000 C CNN
 F 1 "8k" V 8205 2225 50  0000 C CNN
-F 2 "r_0805" V 8305 2225 50  0001 C CNN
+F 2 "r_0603" V 8305 2225 50  0001 C CNN
 F 3 "" H 8200 2225 60  0001 C CNN
 F 4 "RES 10K OHM 1/8W 5% CF AXIAL" H 8200 2325 60  0001 L CNN "Field4"
@@
 F 0 "R17" V 8575 3100 50  0000 C CNN
 F 1 "16k" V 8530 2900 50  0000 C CNN
-F 2 "r_0805" V 8630 2900 50  0001 C CNN
+F 2 "r_0603" V 8630 2900 50  0001 C CNN
 F 3 "" H 8525 2900 60  0001 C CNN
 F 4 "RES 10K OHM 1/8W 5% CF AXIAL" H 8525 3000 60  0001 L CNN "Field4"
@@
 F 0 "R18" V 8675 3100 50  0000 C CNN
 F 1 "16k" V 8630 2900 50  0000 C CNN
-F 2 "r_0805" V 8730 2900 50  0001 C CNN
+F 2 "r_0603" V 8730 2900 50  0001 C CNN
 F 3 "" H 8625 2900 60  0001 C CNN
 F 4 "RES 10K OHM 1/8W 5% CF AXIAL" H 8625 3000 60  0001 L CNN "Field4"
@@
 F 0 "R19" V 8775 3100 50  0000 C CNN
 F 1 "16k" V 8730 2900 50  0000 C CNN
-F 2 "r_0805" V 8830 2900 50  0001 C CNN
+F 2 "r_0603" V 8830 2900 50  0001 C CNN
 F 3 "" H 8725 2900 60  0001 C CNN
 F 4 "RES 10K OHM 1/8W 5% CF AXIAL" H 8725 3000 60  0001 L CNN "Field4"
@@
 F 0 "R20" V 8875 3100 50  0000 C CNN
 F 1 "16k" V 8830 2900 50  0000 C CNN
-F 2 "r_0805" V 8930 2900 50  0001 C CNN
+F 2 "r_0603" V 8930 2900 50  0001 C CNN
 F 3 "" H 8825 2900 60  0001 C CNN
 F 4 "RES 10K OHM 1/8W 5% CF AXIAL" H 8825 3000 60  0001 L CNN "Field4"

Commit message: uControl_v2 progress : Pump 3d added
Parts:
- removed SC25, SC26: SCREW, vite_3mm, symbol SCREW
- B4, B5, B6, B7: footprint I/O -> I_O; symbol I/O -> I_O
Other:
- note removed: "Mounting Holes\nfor Raspberry-Pi"
Changed lines of the file:
@@
-EESchema Schematic File Version 2  date 17-Aug-13 4:16:47 PM
+EESchema Schematic File Version 2
 LIBS:Conn-raspberry
 LIBS:power
 LIBS:uControl
 LIBS:uControl_v2-cache
-EELAYER 27 0
+EELAYER 24 0
 EELAYER END
 $Descr A4 11693 8268
@@
 Text Label 3300 1225 0    40   ~ 0
 Rpi_3V3
-Text Notes 6100 7250 0    40   ~ 0
-Mounting Holes\nfor Raspberry-Pi
-$Comp
-L SCREW SC26
-U 1 1 50DD59EB
-P 6450 7450
-F 0 "SC26" H 6450 7350 40  0000 C CNN
-F 1 "SCREW" H 6450 7550 40  0001 C CNN
-F 2 "vite_3mm" H 6450 7650 40  0001 C CNN
-F 3 "" H 6450 7450 60  0001 C CNN
-	1    6450 7450
-	1    0    0    -1
-$EndComp
-$Comp
-L SCREW SC25
-U 1 1 50DD59E1
-P 6200 7450
-F 0 "SC25" H 6200 7350 40  0000 C CNN
-F 1 "SCREW" H 6200 7550 40  0001 C CNN
-F 2 "vite_3mm" H 6200 7650 40  0001 C CNN
-F 3 "" H 6200 7450 60  0001 C CNN
-	1    6200 7450
-	1    0    0    -1
-$EndComp
 NoConn ~ 4175 3750
 $Comp
@@
 Connection ~ 10825 1625
 $Comp
-L I/O B5
+L I_O B5
 U 1 1 520DE179
 P 7525 2225
 F 0 "B5" H 7550 2175 40  0000 L CNN
 F 1 "A_INT2" H 7525 2280 30  0001 C CNN
-F 2 "I/O" H 7525 2225 60  0001 C CNN
+F 2 "I_O" H 7525 2225 60  0001 C CNN
 F 3 "" H 7525 2225 60  0000 C CNN
 	1    7525 2225
@@
 $EndComp
 $Comp
-L I/O B4
+L I_O B4
 U 1 1 520DE17F
 P 7525 2125
 F 0 "B4" H 7550 2075 40  0000 L CNN
 F 1 "A_INT1" H 7525 2180 30  0001 C CNN
-F 2 "I/O" H 7525 2125 60  0001 C CNN
+F 2 "I_O" H 7525 2125 60  0001 C CNN
 F 3 "" H 7525 2125 60  0000 C CNN
 	1    7525 2125
@@
 	7675 1625 7950 1625
 $Comp
-L I/O B6
+L I_O B6
 U 1 1 520DE1FA
 P 7525 1725
 F 0 "B6" H 7575 1725 40  0000 L CNN
 F 1 "A_SDO" H 7525 1780 30  0001 C CNN
-F 2 "I/O" H 7525 1725 60  0001 C CNN
+F 2 "I_O" H 7525 1725 60  0001 C CNN
 F 3 "" H 7525 1725 60  0000 C CNN
 	1    7525 1725
@@
 ACL_INT2
 $Comp
-L I/O B7
+L I_O B7
 U 1 1 520DEC11
 P 7525 1625
 F 0 "B7" H 7575 1625 40  0000 L CNN
 F 1 "A_CS" H 7525 1680 30  0001 C CNN
-F 2 "I/O" H 7525 1625 60  0001 C CNN
+F 2 "I_O" H 7525 1625 60  0001 C CNN
 F 3 "" H 7525 1625 60  0000 C CNN
 	1    7525 1625
