File: KiCad/uControl_v2/uControl_v2.sch (KiCad schematic (older format))
At the start: 21 parts, among them P1 AREF, P2 ANALOG_5V0, P3 ANALOG_GND, P4 ICSP, P5 FTDI, SW1 Reset, U7 ATMEGA328P, X1 16MHz

Commit message: uControl_v2 schematic more progress
Parts:
- added U7: ATMEGA328-AU-ND, TQFP32, symbol ATMEGA328-AU-ND
Connections:
- net labels added: PB0, PD2, PD4, PD7, ~PB1
- wire segments 167 -> 171
Other:
- note added: "Blank (ex Flow_Rx)"
- note added: "Blank (ex Flow_Tx)"
- note added: "Blank (ex Pump PB0_IO_R)"
- note added: "Blank (ex Pump PD7_IO_X)"
- note added: "PUMP (ex Pump ~PB1_IO_T)"
- note removed: "Flow"
- note removed: "Pump"
Changed lines of the file:
@@
-EESchema Schematic File Version 2  date 13-Aug-13 5:34:33 PM
+EESchema Schematic File Version 2
 LIBS:Conn-raspberry
 LIBS:power
 LIBS:uControl
-EELAYER 27 0
+EELAYER 24 0
 EELAYER END
 $Descr A4 11693 8268
@@
 $EndComp
 Wire Wire Line
-	1250 3050 750  3050
+	750  3050 1250 3050
 Wire Notes Line
 	4675 7650 5650 7650
@@
 	6225 2725 6175 2725
 Wire Wire Line
-	6225 2950 6225 2325
+	6225 2325 6225 2950
 Wire Wire Line
 	6225 2325 6175 2325
@@
 	975  1675 975  2550
 Wire Wire Line
-	875  3300 825  3300
-Wire Wire Line
-	825  3300 825  2800
+	825  3300 875  3300
+Wire Wire Line
+	825  2800 825  3300
 Wire Wire Line
 	825  2800 875  2800
@@
 	6675 2525 6425 2525
 Wire Wire Line
-	2900 5100 2900 4850
+	2950 4850 2950 5100
 Wire Wire Line
 	8575 2825 8825 2825
@@
 Wire Wire Line
 	3900 4250 4125 4250
-Connection ~ 2900 4975
 Wire Wire Line
 	4125 4450 3900 4450
@@
 	6675 1625 6425 1625
 Wire Wire Line
-	6675 1925 6425 1925
+	6425 1925 6675 1925
 Wire Wire Line
 	9675 6350 10050 6350
@@
 	6675 2825 6425 2825
 Wire Wire Line
-	1575 4050 1575 1700
+	1575 1700 1575 4050
 Connection ~ 1575 2250
 Wire Wire Line
-	1925 3150 1925 3300
+	1925 3300 1925 3150
 Wire Wire Line
 	1925 3150 2000 3150
@@
 	975  2550 2000 2550
 Wire Wire Line
-	2900 800  2900 1950
+	2900 800  2900 1850
 Connection ~ 2900 800
 Wire Wire Line
@@
 Connection ~ 1800 2450
 Wire Wire Line
-	1925 3300 1275 3300
+	1275 3300 1925 3300
 Connection ~ 1400 3300
 Connection ~ 825  3050
@@
 	750  3050 750  4975
 Wire Wire Line
-	750  4975 2900 4975
+	750  4975 2950 4975
 Connection ~ 1575 4975
 Wire Wire Line
@@
 L ATMEGA8-P U7
 U 1 1 50E2C28A
-P 2900 3350
-F 0 "U7" H 2250 2900 50  0000 L BNN
-F 1 "ATMEGA328P" H 2275 2800 50  0000 L BNN
-F 2 "DIP-28__300_ELL" H 3400 1875 50  0001 C CNN
-F 3 "" H 2900 3350 60  0001 C CNN
-F 4 "IC MCU AVR 32K FLASH 28PDIP" H 2900 4700 60  0001 L CNN "Field4"
-F 5 "AVR ATMega 8 bit 20Mhz" H 2900 4800 60  0001 L CNN "Field5"
-F 6 "28-DIP (0.300\", 7.62mm)" H 2900 4900 60  0001 L CNN "Field6"
-F 7 "Atmel" H 2900 5000 60  0001 L CNN "Field7"
-F 8 "ATMEGA328-PU" H 2900 5100 60  0001 L CNN "Field8"
-F 9 "Digikey" H 2900 5200 60  0001 L CNN "Field9"
-F 10 "ATMEGA328-PU-ND" H 2900 5300 60  0001 L CNN "Field10"
-F 11 "http://www.digikey.com/product-detail/en/ATMEGA328-PU/ATMEGA328-PU-ND/2271026?cur=USD" H 2900 5400 60  0001 L CNN "Field11"
-	1    2900 3350
+P -3600 3300
+F 0 "U7" H -4250 2850 50  0000 L BNN
+F 1 "ATMEGA328P" H -4225 2750 50  0000 L BNN
+F 2 "DIP-28__300_ELL" H -3100 1825 50  0001 C CNN
+F 3 "" H -3600 3300 60  0001 C CNN
+F 4 "IC MCU AVR 32K FLASH 28PDIP" H -3600 4650 60  0001 L CNN "Field4"
+F 5 "AVR ATMega 8 bit 20Mhz" H -3600 4750 60  0001 L CNN "Field5"
+F 6 "28-DIP (0.300\", 7.62mm)" H -3600 4850 60  0001 L CNN "Field6"
+F 7 "Atmel" H -3600 4950 60  0001 L CNN "Field7"
+F 8 "ATMEGA328-PU" H -3600 5050 60  0001 L CNN "Field8"
+F 9 "Digikey" H -3600 5150 60  0001 L CNN "Field9"
+F 10 "ATMEGA328-PU-ND" H -3600 5250 60  0001 L CNN "Field10"
+F 11 "http://www.digikey.com/product-detail/en/ATMEGA328-PU/ATMEGA328-PU-ND/2271026?cur=USD" H -3600 5350 60  0001 L CNN "Field11"
+	1    -3600 3300
 	1    0    0    -1
 $EndComp
@@
 F9 "~SS" I L 10050 2225 40
 F10 "PC3_Pr1" I L 10050 2525 40
-F11 "PD7_IO_X" I L 10050 2825 40
-F12 "~PB1_IO_T" O L 10050 2925 40
-F13 "PB0_IO_R" I L 10050 3025 40
-F14 "3V3" B L 10050 2025 40
-F15 "SCL" I L 10050 3225 40
-F16 "SDA" I L 10050 3325 40
-F17 "PC1_Pulse" I L 10050 3425 40
-F18 "PC2_Pr2" I L 10050 3625 40
-F19 "PD4_Flow_Rx" I L 10050 2725 40
-F20 "PD2_Flow_Tx" O L 10050 2625 40
+F11 "3V3" B L 10050 2025 40
+F12 "SCL" I L 10050 3225 40
+F13 "SDA" I L 10050 3325 40
+F14 "PC1_Pulse" I L 10050 3425 40
+F15 "PC2_Pr2" I L 10050 3625 40
 $EndSheet
 NoConn ~ 6300 7175
@@
 Slave Sel #1 Pr Sensor
 Text Notes 4550 4150 0    40   ~ 0
-Pump
+PUMP (ex Pump ~PB1_IO_T)
 Text Notes 4550 4050 0    40   ~ 0
-Pump
+Blank (ex Pump PB0_IO_R)
 Text Notes 4550 3850 0    40   ~ 0
-Pump
+Blank (ex Pump PD7_IO_X)
 Text Notes 4550 3750 0    40   ~ 0
 Blank
@@
 Valve
 Text Notes 4550 3550 0    40   ~ 0
-Flow
+Blank (ex Flow_Rx)
 Text Notes 4550 3350 0    40   ~ 0
-Flow
+Blank (ex Flow_Tx)
 Text Label 9600 3025 0    40   ~ 0
 ~PB1_IO_T
@@
 L GND #PWR02
 U 1 1 4F5AFC62
-P 2900 5100
-F 0 "#PWR02" H 2900 5100 30  0001 C CNN
-F 1 "GND" H 2900 5030 30  0001 C CNN
-F 2 "" H 2900 5100 60  0001 C CNN
-F 3 "" H 2900 5100 60  0001 C CNN
-	1    2900 5100
+P 2950 5100
+F 0 "#PWR02" H 2950 5100 30  0001 C CNN
+F 1 "GND" H 2950 5030 30  0001 C CNN
+F 2 "" H 2950 5100 60  0001 C CNN
+F 3 "" H 2950 5100 60  0001 C CNN
+	1    2950 5100
 	1    0    0    -1
 $EndComp
@@
 ~PD3
 Text Label 4125 4050 0    40   ~ 0
-PB0_IO_R
+PB0
 Text Label 4125 4150 0    40   ~ 0
-~PB1_IO_T
+~PB1
 Text Label 4125 2250 0    40   ~ 0
 PC0
@@
 TXD
 Text Label 4125 3350 0    40   ~ 0
-PD2_Flow_Tx
+PD2
 Text Label 4125 3850 0    40   ~ 0
-PD7_IO_X
+PD7
 Text Label 4125 3550 0    40   ~ 0
-PD4_Flow_Rx
+PD4
 Text Label 4800 650  0    40   ~ 0
 5V0
@@
 Text Label 4125 4450 0    40   ~ 0
 MISO
+$Comp
+L ATMEGA328-AU-ND U7
+U 1 1 520A592B
+P 2900 3250
+F 0 "U7" H 2300 2650 50  0000 L BNN
+F 1 "ATMEGA328-AU-ND" H 2300 2500 50  0000 L BNN
+F 2 "TQFP32" H 3425 1675 50  0001 C CNN
+F 3 "" H 2900 3250 60  0000 C CNN
+	1    2900 3250
+	1    0    0    -1
+$EndComp
+Connection ~ 2950 4975
+Wire Wire Line
+	2850 4850 2850 4975
+Connection ~ 2850 4975
+Wire Wire Line
+	2950 1850 2950 1950
+Wire Wire Line
+	2850 1850 2950 1850
+Wire Wire Line
+	2850 1950 2850 1850
+Connection ~ 2900 1850
 $EndSCHEMATC

Commit message: uControl_v2 schematic progression
Parts:
- removed DIP1: SOCKET_28X0.3, symbol SOCKET_28X0.3
- removed P2: ANALOG_5V0, Header_6x1, symbol CONN_6
- removed P3: ANALOG_GND, Header_6x1, symbol CONN_6
- removed U7: ATMEGA328P, DIP-28__300_ELL, symbol ATMEGA8-P
Connections:
- net labels added: PB0_ACL, PC1, PD4_Valve2, ~PB1_Pump, ~PD6_Spk
- net labels removed: PB0, PB0_IO_R, PC1_Pulse, PD2_Flow_Tx, PD4, PD4_Flow_Rx, PD7_IO_X, ~PB1, ~PB1_IO_T, ~PD6
- wire segments 171 -> 120
- no-connect marks 2 -> 40
Other:
- note added: "Blank (ex Pulse)"
- note added: "PUMP PWM (ex Pump ~PB1_IO_T)"
- note added: "Slave Sel Accel ADXL345 (ex Pump PB0_IO_R)"
- note added: "Speaker PWM (ex Blank)"
- note added: "Valve #1 PWM"
- note added: "Valve #2 (ex Flow_Rx)"
- note removed: "Blank (ex Flow_Rx)"
- note removed: "Blank (ex Pump PB0_IO_R)"
- note removed: "PUMP (ex Pump ~PB1_IO_T)"
- note removed: "Valve"

Commit message: uControl_v2 : Schematic DRC passes. Most component footprints done. Using old PCB layout to begin with
Parts:
- added C30, C32, C33: 100n, c_0805, symbol C
- added R7: 10K, r_0805, symbol R_10K
- added SD1: SD_CARD_MICRO, SD_Micro_seeed, symbol SD_CARD_MICRO
- added U9: TXB0104D, TXB0104D, symbol TXB0104D
- C1, C4: footprint C2 -> c_0805
- C2, C3: footprint cnp_3mm_disc -> c_0603
- P1: footprint Header_A_REF -> Header_3
- P4: footprint Header_ICSP -> Header_ISP
- R1, R2, R3: footprint rc03_vert -> r_0805
- X1: footprint XTAL -> Xtal_SMD3
Connections:
- net labels added: PD7_SD, SD_CS_3V3, SPI_CLK_3V3, SPI_MISO_3V3, SPI_MOSI_3V3
- net labels removed: PD7
- wire segments 120 -> 149
- no-connect marks 40 -> 47
Other:
- note added: "CS #1 Pr Sensor"
- note added: "CS Accel ADXL345 (ex Pump PB0_IO_R)"
- note added: "CS SDCard (ex Pump PD7_IO_X)"
- note added: "Micro SD Card"
- note removed: "Blank (ex Pump PD7_IO_X)"
- note removed: "Slave Sel #1 Pr Sensor"
- note removed: "Slave Sel Accel ADXL345 (ex Pump PB0_IO_R)"
- moved on the sheet: C4, P4, P5, SC17, SC18, SC19, SC20

Commit message: uControl_v2 : Moved Accel to Ras-Pi side. Added 2 buttons to Atmega. Working on new footprints (flow, pump)
Parts:
- added B10: PC6, I/O, symbol I/O
- added B11: PC7, I/O, symbol I/O
- added B12: PB0, I/O, symbol I/O
- added B8: PC0, I/O, symbol I/O
- added B9: PC1, I/O, symbol I/O
- added C28: 100n, c_0805, symbol C
- added R21, R22: 10k, r_0805, symbol R_10K
- added SW2: INT0, SW_PB_V_H, symbol SW_PUSH
- added SW3: INT1, SW_PB_V_H, symbol SW_PUSH
- R1, R2, R3, R7: value 10K -> 10k
Connections:
- net labels added: PB0, PC6, PC7
- net labels removed: PB0_ACL
- wire segments 149 -> 164
- no-connect marks 47 -> 41
Other:
- note added: "Analog, from Absolute Pr Sensor"
- note added: "Analog, from Gage Pr Sensor"
- note added: "Blank (ex Pump PB0_IO_R)"
- note added: "SW INT0 (ex Flow_Tx)"
- note added: "SW INT1 (ex Blank)"
- note removed: "Blank (ex Flow_Tx)"
- note removed: "CS Accel ADXL345 (ex Pump PB0_IO_R)"
- moved on the sheet: C30, C32, C33, C4, P4, P5, SC17, SC18, SC19, SC20, SHIELD1, U9

Commit message: uControl_v2 : Components selected and footprints done. Ready to start layout
Parts:
- C1, C28, C30, C32, C33, C4: footprint c_0805 -> c_0603
- R1, R2, R21, R22, R3, R7: footprint r_0805 -> r_0603
Changed lines of the file:
@@
-EESchema Schematic File Version 2
+EESchema Schematic File Version 2  date 17-Aug-13 4:16:42 PM
 LIBS:Conn-raspberry
 LIBS:power
 LIBS:uControl
 LIBS:uControl_v2-cache
-EELAYER 24 0
+EELAYER 27 0
 EELAYER END
 $Descr A4 11693 8268
@@
 Sheet 1 5
 Title "uControl"
-Date "16 aug 2013"
+Date "17 aug 2013"
 Rev "1"
 Comp "WyoLum"
@@
 F 0 "R3" H 4750 1600 50  0000 C CNN
 F 1 "10k" V 4805 1450 50  0000 C CNN
-F 2 "r_0805" V 4905 1450 50  0001 C CNN
+F 2 "r_0603" V 4905 1450 50  0001 C CNN
 F 3 "" H 4800 1450 60  0001 C CNN
 F 4 "RES 10K OHM 1/8W 5% CF AXIAL" H 4800 1550 60  0001 L CNN "Field4"
@@
 F 0 "R2" H 4550 1600 50  0000 C CNN
 F 1 "10k" V 4605 1450 50  0000 C CNN
-F 2 "r_0805" V 4705 1450 50  0001 C CNN
+F 2 "r_0603" V 4705 1450 50  0001 C CNN
 F 3 "" H 4600 1450 60  0001 C CNN
 F 4 "RES 10K OHM 1/8W 5% CF AXIAL" H 4600 1550 60  0001 L CNN "Field4"
@@
 F 0 "R1" H 1525 1600 50  0000 C CNN
 F 1 "10k" V 1580 1450 50  0000 C CNN
-F 2 "r_0805" V 1680 1450 50  0001 C CNN
+F 2 "r_0603" V 1680 1450 50  0001 C CNN
 F 3 "" H 1575 1450 60  0001 C CNN
 F 4 "RES 10K OHM 1/8W 5% CF AXIAL" H 1575 1550 60  0001 L CNN "Field4"
@@
 F 0 "C4" H 8850 6200 50  0000 L CNN
 F 1 "100n" H 8750 6025 50  0000 L CNN
-F 2 "c_0805" H 8950 6125 50  0001 C CNN
+F 2 "c_0603" H 8950 6125 50  0001 C CNN
 F 3 "" H 8950 6125 60  0001 C CNN
 F 4 "CAP FILM 0.1UF 63VDC RADIAL" H 8950 6325 60  0001 L CNN "Field4"
@@
 F 0 "C1" H 1800 1550 50  0000 L CNN
 F 1 "100n" H 1800 1350 50  0000 L CNN
-F 2 "c_0805" H 1800 1450 50  0001 C CNN
+F 2 "c_0603" H 1800 1450 50  0001 C CNN
 F 3 "" H 1800 1450 60  0001 C CNN
 F 4 "CAP FILM 0.1UF 63VDC RADIAL" H 1800 1650 60  0001 L CNN "Field4"
@@
 F 0 "C33" H 1950 7300 50  0000 L CNN
 F 1 "100n" H 1900 7125 50  0000 L CNN
-F 2 "c_0805" H 2100 7225 50  0001 C CNN
+F 2 "c_0603" H 2100 7225 50  0001 C CNN
 F 3 "" H 2100 7225 60  0001 C CNN
 F 4 "CAP FILM 0.1UF 63VDC RADIAL" H 2100 7425 60  0001 L CNN "Field4"
@@
 F 0 "R7" H 1725 7400 50  0000 C CNN
 F 1 "10k" V 1780 7225 50  0000 C CNN
-F 2 "r_0805" V 1880 7225 50  0001 C CNN
+F 2 "r_0603" V 1880 7225 50  0001 C CNN
 F 3 "" H 1775 7225 60  0001 C CNN
 F 4 "RES 10K OHM 1/8W 5% CF AXIAL" H 1775 7325 60  0001 L CNN "Field4"
@@
 F 0 "C32" H 1925 6225 50  0000 L CNN
 F 1 "100n" H 1925 6025 50  0000 L CNN
-F 2 "c_0805" H 1925 6125 50  0001 C CNN
+F 2 "c_0603" H 1925 6125 50  0001 C CNN
 F 3 "" H 1925 6125 60  0001 C CNN
 F 4 "CAP FILM 0.1UF 63VDC RADIAL" H 1925 6325 60  0001 L CNN "Field4"
@@
 F 0 "C30" H 800 6225 50  0000 L CNN
 F 1 "100n" H 800 6025 50  0000 L CNN
-F 2 "c_0805" H 800 6125 50  0001 C CNN
+F 2 "c_0603" H 800 6125 50  0001 C CNN
 F 3 "" H 800 6125 60  0001 C CNN
 F 4 "CAP FILM 0.1UF 63VDC RADIAL" H 800 6325 60  0001 L CNN "Field4"
@@
 F 0 "R22" H 5925 4050 50  0000 C CNN
 F 1 "10k" V 6005 3900 50  0000 C CNN
-F 2 "r_0805" V 6105 3900 50  0001 C CNN
+F 2 "r_0603" V 6105 3900 50  0001 C CNN
 F 3 "" H 6000 3900 60  0001 C CNN
 F 4 "RES 10K OHM 1/8W 5% CF AXIAL" H 6000 4000 60  0001 L CNN "Field4"
@@
 F 0 "R21" H 5725 4050 50  0000 C CNN
 F 1 "10k" V 5805 3900 50  0000 C CNN
-F 2 "r_0805" V 5905 3900 50  0001 C CNN
+F 2 "r_0603" V 5905 3900 50  0001 C CNN
 F 3 "" H 5800 3900 60  0001 C CNN
 F 4 "RES 10K OHM 1/8W 5% CF AXIAL" H 5800 4000 60  0001 L CNN "Field4"
@@
 F 0 "C28" H 3250 1550 50  0000 L CNN
 F 1 "100n" H 3250 1350 50  0000 L CNN
-F 2 "c_0805" H 3250 1450 50  0001 C CNN
+F 2 "c_0603" H 3250 1450 50  0001 C CNN
 F 3 "" H 3250 1450 60  0001 C CNN
 F 4 "CAP FILM 0.1UF 63VDC RADIAL" H 3250 1650 60  0001 L CNN "Field4"

Commit message: uControl_v2 progress : Pump 3d added
Parts:
- B10, B11, B12, B8, B9: footprint I/O -> I_O; symbol I/O -> I_O
Changed lines of the file:
@@
-EESchema Schematic File Version 2  date 17-Aug-13 4:16:42 PM
+EESchema Schematic File Version 2
 LIBS:Conn-raspberry
 LIBS:power
 LIBS:uControl
 LIBS:uControl_v2-cache
-EELAYER 27 0
+EELAYER 24 0
 EELAYER END
 $Descr A4 11693 8268
@@
 Blank
 $Comp
-L I/O B8
+L I_O B8
 U 1 1 520E3AF6
 P 4275 2250
 F 0 "B8" H 4355 2250 40  0000 L CNN
 F 1 "PC0" H 4275 2305 30  0001 C CNN
-F 2 "I/O" H 4275 2250 60  0001 C CNN
+F 2 "I_O" H 4275 2250 60  0001 C CNN
 F 3 "" H 4275 2250 60  0000 C CNN
 	1    4275 2250
@@
 $EndComp
 $Comp
-L I/O B9
+L I_O B9
 U 1 1 520E3DD3
 P 4275 2350
 F 0 "B9" H 4355 2350 40  0000 L CNN
 F 1 "PC1" H 4275 2405 30  0001 C CNN
-F 2 "I/O" H 4275 2350 60  0001 C CNN
+F 2 "I_O" H 4275 2350 60  0001 C CNN
 F 3 "" H 4275 2350 60  0000 C CNN
 	1    4275 2350
@@
 $EndComp
 $Comp
-L I/O B10
+L I_O B10
 U 1 1 520E3DD9
 P 4275 2850
 F 0 "B10" H 4355 2850 40  0000 L CNN
 F 1 "PC6" H 4275 2905 30  0001 C CNN
-F 2 "I/O" H 4275 2850 60  0001 C CNN
+F 2 "I_O" H 4275 2850 60  0001 C CNN
 F 3 "" H 4275 2850 60  0000 C CNN
 	1    4275 2850
@@
 $EndComp
 $Comp
-L I/O B11
+L I_O B11
 U 1 1 520E3ECF
 P 4275 2950
 F 0 "B11" H 4355 2950 40  0000 L CNN
 F 1 "PC7" H 4275 3005 30  0001 C CNN
-F 2 "I/O" H 4275 2950 60  0001 C CNN
+F 2 "I_O" H 4275 2950 60  0001 C CNN
 F 3 "" H 4275 2950 60  0000 C CNN
 	1    4275 2950
@@
 PC7
 $Comp
-L I/O B12
+L I_O B12
 U 1 1 520E5284
 P 4275 4050
 F 0 "B12" H 4355 4050 40  0000 L CNN
 F 1 "PB0" H 4275 4105 30  0001 C CNN
-F 2 "I/O" H 4275 4050 60  0001 C CNN
+F 2 "I_O" H 4275 4050 60  0001 C CNN
 F 3 "" H 4275 4050 60  0000 C CNN
 	1    4275 4050
