File: KiCad/uControl_v2/uControl_v2_B.sch (KiCad schematic (older format))
At the start: 28 parts, among them P1 AREF, P4 ICSP, P5 FTDI, SW1 Reset, SW2 INT0, SW3 INT1, U7 ATMEGA328-AU-ND, X1 16MHz

Commit message: uControl_v2 - laying out the parts on the board
Parts:
- removed B4: PB0, I_O, symbol I_O
- added C30, C32, C33: 100n, c_0603, symbol C
- added R7: 10k, r_0603, symbol R_10K
- added SD1: SD_CARD_MICRO, SD_Micro_seeed, symbol SD_CARD_MICRO
- added SHIELD1: ARDUINO_SHIELD, ARDUINO_SHIELD_2_040pins, symbol ARDUINO_SHIELD
- added U9: TXB0104D, TXB0104D, symbol TXB0104D
- P1: footprint ShortLink2 -> Header_3
Connections:
- net labels added: PD7_SD, SD_CS_3V3, SPI_CLK_3V3, SPI_MISO_3V3, SPI_MOSI_3V3
- net labels removed: PD7
- wire segments 131 -> 164
- no-connect marks 1 -> 41
Other:
- note added: "CS SDCard (ex Pump PD7_IO_X)"
- note added: "Micro SD Card"
- note removed: "Blank (ex Pump PD7_IO_X)"
