File: KiCad/uControl_v2/uControl_pwr.sch (KiCad schematic (older format))
At the start: 23 parts, among them P24 12V, U3 NCP1117ST50T3G, U4 NCP1117ST33T3G

Commit message: uControl2 : phew, discovered a short betn 5V0 and 12V. Updated. Some parts placement
Parts:
- U3: footprint SOT223 -> NCP1117ST50
- U4: footprint SOT223 -> NCP1117ST33
Connections:
- net labels removed: +5V
- wire segments 51 -> 47
Changed lines of the file:
@@
 	1725 950  1725 1050
 Wire Wire Line
-	2450 1050 2450 1550
+	2450 700  2450 1550
 Connection ~ 2450 1050
 Connection ~ 3850 1050
@@
 	1400 1150 1800 1150
 Connection ~ 3575 1950
-Connection ~ 4625 1050
 Wire Wire Line
 	3850 1950 3850 1800
 Wire Wire Line
-	3850 1050 3850 1525
-Wire Wire Line
-	4625 1050 4625 900
+	3850 975  3850 1525
 Wire Wire Line
 	2450 1950 3850 1950
@@
 	3025 1600 3025 1950
 Connection ~ 3025 1950
-Wire Wire Line
-	3425 1200 3575 1200
 Connection ~ 3575 1050
 Wire Wire Line
@@
 	3575 1050 3575 1525
 Wire Wire Line
-	6400 700  2300 700
-Wire Wire Line
-	2300 700  2300 1050
-Connection ~ 2300 1050
+	6400 700  2450 700
 Wire Wire Line
 	2450 2650 2450 2450
@@
 	1800 3525 2625 3525
 Connection ~ 3575 3525
-Wire Wire Line
-	3575 3675 3425 3675
 Connection ~ 3025 4425
 Wire Wire Line
@@
 U 1 1 50E2C000
 P 3025 3675
-F 0 "U4" H 2875 3675 60  0000 C CNN
-F 1 "NCP1117ST33T3G" H 3025 3975 60  0000 C CNN
-F 2 "SOT223" H 3025 4075 60  0001 C CNN
+F 0 "U4" H 2800 4050 40  0000 C CNN
+F 1 "NCP1117ST33T3G" H 3025 3975 40  0000 C CNN
+F 2 "NCP1117ST33" H 3025 4075 60  0001 C CNN
 F 3 "" H 3025 3675 60  0001 C CNN
 F 4 "IC REG LDO 3.3V 1A DPAK-3" H 3025 3775 60  0001 L CNN "Field4"
@@
 U 1 1 50E2BF58
 P 3025 1200
-F 0 "U3" H 2875 1200 60  0000 C CNN
-F 1 "NCP1117ST50T3G" H 3025 1500 60  0000 C CNN
-F 2 "SOT223" H 3025 1600 60  0001 C CNN
+F 0 "U3" H 2800 1550 40  0000 C CNN
+F 1 "NCP1117ST50T3G" H 3025 1475 40  0000 C CNN
+F 2 "NCP1117ST50" H 3025 1600 60  0001 C CNN
 F 3 "" H 3025 1200 60  0001 C CNN
 F 4 "IC REG LDO 5V 1A DPAK-3" H 3025 1300 60  0001 L CNN "Field4"
@@
 Text Label 7400 3575 0    40   ~ 0
 SCK
-Text Label 2300 1050 0    40   ~ 0
+Text Label 2525 1050 0    40   ~ 0
 12V
 Text Label 6200 2650 0    40   ~ 0
@@
 5V0
 $Comp
-L +5V #PWR022
-U 1 1 4FC61A10
-P 4625 900
-F 0 "#PWR022" H 4625 990 20  0001 C CNN
-F 1 "+5V" H 4625 990 30  0000 C CNN
-F 2 "" H 4625 900 60  0001 C CNN
-F 3 "" H 4625 900 60  0001 C CNN
-	1    4625 900
-	-1   0    0    -1
-$EndComp
-$Comp
-L GND #PWR023
+L GND #PWR022
 U 1 1 4FC61A0D
 P 4625 2750
-F 0 "#PWR023" H 4625 2750 30  0001 C CNN
+F 0 "#PWR022" H 4625 2750 30  0001 C CNN
 F 1 "GND" H 4625 2680 30  0001 C CNN
 F 2 "" H 4625 2750 60  0001 C CNN
@@
 $EndComp
 $Comp
-L GND #PWR024
+L GND #PWR023
 U 1 1 4FC61A09
 P 3575 2050
-F 0 "#PWR024" H 3575 2050 30  0001 C CNN
+F 0 "#PWR023" H 3575 2050 30  0001 C CNN
 F 1 "GND" H 3575 1980 30  0001 C CNN
 F 2 "" H 3575 2050 60  0001 C CNN
@@
 	1    0    0    -1
 $EndComp
-Connection ~ 3575 1200
-Connection ~ 3575 3675
+$Comp
+L PWR_FLAG #FLG024
+U 1 1 5213B593
+P 3850 975
+F 0 "#FLG024" H 3850 1245 30  0001 C CNN
+F 1 "PWR_FLAG" H 3850 1205 30  0000 C CNN
+F 2 "" H 3850 975 60  0001 C CNN
+F 3 "" H 3850 975 60  0001 C CNN
+	1    3850 975
+	1    0    0    -1
+$EndComp
 $EndSCHEMATC

Commit message: uControl_v2 : working on getting PiPower 3D in to the board to allow proper placement.
Connections:
- wire segments 47 -> 46
Other:
- moved on the sheet: C18, C19, C20, D4, P24, U3

Commit message: uControl_v2 : Ready to stary layout once RasPi and Gage orientation is finalized
Parts:
- added P13: PWR_IN, symbol CONN_2
- P24: value 12V -> PWR_IN
Connections:
- wire segments 46 -> 48
Other:
- moved on the sheet: D4
Changed lines of the file:
@@
 Wire Wire Line
 	7625 4200 7625 4250
-Connection ~ 1725 1400
-Wire Wire Line
-	1725 825  1725 1400
+Connection ~ 1500 1400
+Wire Wire Line
+	1500 825  1500 1400
 Wire Wire Line
 	2450 1050 2450 1900
@@
 	3575 2125 3575 2400
 Wire Wire Line
-	1400 1600 1800 1600
-Wire Wire Line
-	1400 1500 1800 1500
+	1400 1600 1500 1600
+Wire Wire Line
+	1400 1500 1500 1500
 Connection ~ 3575 2300
 Wire Wire Line
@@
 	3850 1325 3850 1875
 Wire Wire Line
-	1800 2300 6400 2300
+	1200 2300 6400 2300
 Wire Wire Line
 	2450 2300 2450 2150
 Connection ~ 4625 2300
 Wire Wire Line
-	1400 1400 1825 1400
-Wire Wire Line
-	1800 1500 1800 2300
+	1400 1400 1975 1400
+Wire Wire Line
+	1500 1500 1500 2300
 Wire Wire Line
 	3025 1950 3025 2300
@@
 Connection ~ 3575 1400
 Wire Wire Line
-	2225 1400 2625 1400
+	2375 1400 2625 1400
 Wire Wire Line
 	7625 3575 7400 3575
@@
 U 1 1 50E2B59E
 P 1100 1500
-F 0 "P24" H 1100 1700 60  0000 C CNN
-F 1 "12V" H 1100 1250 60  0000 C CNN
+F 0 "P24" H 800 1700 40  0000 C CNN
+F 1 "PWR_IN" H 1050 1700 40  0000 C CNN
 F 2 "JACK_ALIM" H 1100 1350 60  0001 C CNN
 F 3 "" H 1100 1500 60  0001 C CNN
@@
 L D_1N4001 D4
 U 1 1 50E2A12F
-P 2025 1400
-F 0 "D4" H 2025 1500 40  0000 C CNN
-F 1 "1N4007" H 2025 1300 40  0000 C CNN
-F 2 "diode-DO214AC" H 2025 1400 40  0001 C CNN
-F 3 "" H 2025 1400 60  0001 C CNN
-F 4 "DIODE GEN PURPOSE 50V 1A DO41" H 2025 1600 60  0001 L CNN "Field4"
-F 5 "50V, 1A" H 2025 1700 60  0001 L CNN "Field5"
-F 6 "DO-204AL, DO-41, Axial" H 2025 1800 60  0001 L CNN "Field6"
-F 7 "Fairchild Semiconductor" H 2025 1900 60  0001 L CNN "Field7"
-F 8 "1N4001" H 2025 2000 60  0001 L CNN "Field8"
-F 9 "Digikey" H 2025 2100 60  0001 L CNN "Field9"
-F 10 "1N4001FSCT-ND" H 2025 2200 60  0001 L CNN "Field10"
-F 11 "http://www.digikey.com/product-detail/en/1N4001/1N4001FSCT-ND/1532742" H 2025 2300 60  0001 L CNN "Field11"
-	1    2025 1400
+P 2175 1400
+F 0 "D4" H 2175 1500 40  0000 C CNN
+F 1 "1N4007" H 2175 1300 40  0000 C CNN
+F 2 "diode-DO214AC" H 2175 1400 40  0001 C CNN
+F 3 "" H 2175 1400 60  0001 C CNN
+F 4 "DIODE GEN PURPOSE 50V 1A DO41" H 2175 1600 60  0001 L CNN "Field4"
+F 5 "50V, 1A" H 2175 1700 60  0001 L CNN "Field5"
+F 6 "DO-204AL, DO-41, Axial" H 2175 1800 60  0001 L CNN "Field6"
+F 7 "Fairchild Semiconductor" H 2175 1900 60  0001 L CNN "Field7"
+F 8 "1N4001" H 2175 2000 60  0001 L CNN "Field8"
+F 9 "Digikey" H 2175 2100 60  0001 L CNN "Field9"
+F 10 "1N4001FSCT-ND" H 2175 2200 60  0001 L CNN "Field10"
+F 11 "http://www.digikey.com/product-detail/en/1N4001/1N4001FSCT-ND/1532742" H 2175 2300 60  0001 L CNN "Field11"
+	1    2175 1400
 	1    0    0    -1
 $EndComp
@@
 Text Notes 750  1750 0    30   Italic 6
 BARREL\nPOWER\nSOCKET
-Text Label 1450 1400 0    40   ~ 0
+Text Label 1725 1400 0    40   ~ 0
 PWR_IN
 $Comp
@@
 L PWR_FLAG #FLG016
 U 1 1 4FC9DE21
-P 1725 825
-F 0 "#FLG016" H 1725 1095 30  0001 C CNN
-F 1 "PWR_FLAG" H 1725 1055 30  0000 C CNN
-F 2 "" H 1725 825 60  0001 C CNN
-F 3 "" H 1725 825 60  0001 C CNN
-	1    1725 825
+P 1500 825
+F 0 "#FLG016" H 1500 1095 30  0001 C CNN
+F 1 "PWR_FLAG" H 1500 1055 30  0000 C CNN
+F 2 "" H 1500 825 60  0001 C CNN
+F 3 "" H 1500 825 60  0001 C CNN
+	1    1500 825
 	1    0    0    -1
 $EndComp
@@
 $EndComp
 Connection ~ 3850 2300
-Connection ~ 1800 1600
+Connection ~ 1500 1600
 Connection ~ 2450 2300
 Wire Wire Line
-	1725 900  6400 900
-Connection ~ 1725 900
+	1500 900  6400 900
+Connection ~ 1500 900
 Text HLabel 6400 900  2    40   BiDi ~ 0
 PWR_IN
 Text Label 6150 900  0    40   ~ 0
 PWR_IN
+$Comp
+L CONN_2 P13
+U 1 1 521B769C
+P 850 2200
+F 0 "P13" V 800 2200 40  0000 C CNN
+F 1 "PWR_IN" V 900 2200 40  0000 C CNN
+F 2 "" H 850 2200 60  0000 C CNN
+F 3 "" H 850 2200 60  0000 C CNN
+	1    850  2200
+	-1   0    0    -1
+$EndComp
+Connection ~ 1500 2300
+Wire Wire Line
+	1200 2100 1675 2100
+Wire Wire Line
+	1675 2100 1675 1400
+Connection ~ 1675 1400
 $EndSCHEMATC

Commit message: uControl_v2 : working on track layout. half way through.
Parts:
- P13: footprint (none) -> Header_2
Changed lines of the file:
@@
 F 0 "P13" V 800 2200 40  0000 C CNN
 F 1 "PWR_IN" V 900 2200 40  0000 C CNN
-F 2 "" H 850 2200 60  0000 C CNN
+F 2 "Header_2" H 850 2200 60  0001 C CNN
 F 3 "" H 850 2200 60  0000 C CNN
 	1    850  2200
