File: KiCad/uControl_v3/uControl_rtc.sch (KiCad schematic (older format))
At the start: 8 parts, among them U5 DS3231N

Commit message: uC_v3 work in progress
Parts:
- C23: footprint c_0603 -> c_0805
- R11: footprint r_0603 -> r_0805
Changed lines of the file:
@@
 $Descr A4 11693 8268
 encoding utf-8
-Sheet 4 6
+Sheet 4 5
 Title "uControl"
 Date "28 sep 2013"
@@
 F 0 "R11" H 7050 2150 50  0000 C CNN
 F 1 "10k" V 7155 2000 50  0000 C CNN
-F 2 "r_0603" V 7255 2000 50  0001 C CNN
+F 2 "r_0805" V 7255 2000 50  0001 C CNN
 F 3 "" H 7150 2000 60  0001 C CNN
 F 4 "RES 10K OHM 1/8W 5% CF AXIAL" H 7150 2100 60  0001 L CNN "Field4"
@@
 F 0 "C23" H 4175 2875 50  0000 L CNN
 F 1 "100n" H 4175 2675 50  0000 L CNN
-F 2 "c_0603" H 4175 2775 50  0001 C CNN
+F 2 "c_0805" H 4175 2775 50  0001 C CNN
 F 3 "" H 4175 2775 60  0001 C CNN
 F 4 "CAP FILM 0.1UF 63VDC RADIAL" H 4175 2975 60  0001 L CNN "Field4"
@@
 BAT
 $Comp
-L +BATT #PWR021
+L +BATT #PWR019
 U 1 1 4EC101F0
 P 5300 1850
-F 0 "#PWR021" H 5300 1800 20  0001 C CNN
+F 0 "#PWR019" H 5300 1800 20  0001 C CNN
 F 1 "+BATT" H 5300 1950 30  0000 C CNN
 F 2 "" H 5300 1850 60  0001 C CNN

Commit message: uCv3 some schematic cleanup based on BoM check.
Parts:
- C23: value 100n -> 100nF
Changed lines of the file:
@@
 P 4175 2775
 F 0 "C23" H 4175 2875 50  0000 L CNN
-F 1 "100n" H 4175 2675 50  0000 L CNN
+F 1 "100nF" V 4250 2450 50  0000 L CNN
 F 2 "c_0805" H 4175 2775 50  0001 C CNN
 F 3 "" H 4175 2775 60  0001 C CNN
